Commit message: begin grasp demo

File: src/bulldog/bulldog_description/urdf/bulldog_gazebo_robot.xacro (robot description, xacro)
@@ -5,5 +5,5 @@
   <xacro:arg name="ur5_enabled" default="false" />
   <xacro:arg name="kinect_enabled" default="false" />
-  <xacro:arg name="dual_ur5_enabled" default="true"/>
+  <xacro:arg name="dual_ur5_enabled" default="false"/>
   <xacro:arg name="robotiq_grippers_enabled" default="true"/>
   <xacro:include filename="$(find bulldog_description)/urdf/bulldog/bulldog_gazebo.urdf.xacro" />

File: src/bulldog_simulator/bulldog_gazebo/urdf/bulldog.gazebo.xacro (robot description, xacro)
@@ -21,8 +21,14 @@
 ARISING IN ANY WAY OUT OF THE USE OF THIS SOFTWARE, EVEN IF ADVISED OF THE POSSIBILITY OF SUCH DAMAGE.
 -->
-<robot name="bulldog_robot_gazebo" xmlns:xacro="http://ros.org/wiki/xacro">
+<robot name="bulldog_gazebo_robot" xmlns:xacro="http://ros.org/wiki/xacro">
   <xacro:include filename="$(find bulldog_gazebo)/urdf/accessories/kinect_camera.gazebo.xacro"/>
   <xacro:include filename="$(find bulldog_gazebo)/urdf/accessories/realsense_d415_camera.gazebo.xacro"/>
-  <xacro:macro name="bulldog_robot_gazebo">
+  <xacro:macro name="bulldog_gazebo_config">
+    <!-- ROS control -->
+    <gazebo>
+      <plugin name="gazebo_ros_control" filename="libgazebo_ros_control.so">
+        <robotNamespace>/</robotNamespace>
+      </plugin>
+    </gazebo>
     <!-- imu -->
     <gazebo>
@@ -77,4 +83,49 @@
       </gazebo>
     </xacro:if>
+    <xacro:if value="$(arg dual_ur5_enabled)">
+      <gazebo>
+        <plugin name="gazebo_grasp_fix" filename="libgazebo_grasp_fix.so">
+            <arm>
+              <arm_name>left_arm </arm_name>
+              <palm_link> left_arm_wrist_3_link </palm_link>
+              <gripper_link> left_gripper_finger_1_link_0 </gripper_link>
+              <gripper_link> left_gripper_finger_1_link_1 </gripper_link>
+              <gripper_link> left_gripper_finger_1_link_2 </gripper_link>
+              <gripper_link> left_gripper_finger_1_link_3 </gripper_link>
+              <gripper_link> left_gripper_finger_2_link_0 </gripper_link>
+              <gripper_link> left_gripper_finger_2_link_1 </gripper_link>
+              <gripper_link> left_gripper_finger_2_link_2 </gripper_link>
+              <gripper_link> left_gripper_finger_2_link_3 </gripper_link>
+              <gripper_link> left_gripper_finger_middle_link_0 </gripper_link>
+              <gripper_link> left_gripper_finger_middle_link_1 </gripper_link>
+              <gripper_link> left_gripper_finger_middle_link_2 </gripper_link>
+              <gripper_link> left_gripper_finger_middle_link_3 </gripper_link>
+            </arm>
+            <arm>
+              <arm_name>right_arm </arm_name>
+              <palm_link> right_arm_wrist_3_link  </palm_link>
+              <gripper_link> right_gripper_finger_1_link_0 </gripper_link>
+              <gripper_link> right_gripper_finger_1_link_1 </gripper_link>
+              <gripper_link> right_gripper_finger_1_link_2 </gripper_link>
+              <gripper_link> right_gripper_finger_1_link_3 </gripper_link>
+              <gripper_link> right_gripper_finger_2_link_0 </gripper_link>
+              <gripper_link> right_gripper_finger_2_link_1 </gripper_link>
+              <gripper_link> right_gripper_finger_2_link_2 </gripper_link>
+              <gripper_link> right_gripper_finger_2_link_3 </gripper_link>
+              <gripper_link> right_gripper_finger_middle_link_0 </gripper_link>
+              <gripper_link> right_gripper_finger_middle_link_1 </gripper_link>
+              <gripper_link> right_gripper_finger_middle_link_2 </gripper_link>
+              <gripper_link> right_gripper_finger_middle_link_3 </gripper_link>
+            </arm>
+          <forces_angle_tolerance>100</forces_angle_tolerance>
+          <update_rate>4</update_rate>
+          <grip_count_threshold>4</grip_count_threshold>
+          <max_grip_count>8</max_grip_count>
+          <release_tolerance>0.005</release_tolerance>
+          <disable_collisions_on_attach>false</disable_collisions_on_attach>
+          <contact_topic>__default_topic__</contact_topic>
+        </plugin>
+      </gazebo>
+    </xacro:if>
     <!-- robotiq grippers -->
     <xacro:if value="$(arg robotiq_grippers_enabled)">

File: src/bulldog_simulator/bulldog_gazebo/urdf/description.gazebo.xacro (robot description, xacro)
@@ -26,60 +26,9 @@
   <xacro:arg name="kinect_enabled" default="false" />
   <xacro:arg name="realsense_enabled" default="false" />
-  <xacro:arg name="dual_ur5_enabled" default="true" />
+  <xacro:arg name="dual_ur5_enabled" default="false" />
   <xacro:arg name="robotiq_grippers_enabled" default="true" />
   <xacro:include filename="$(find bulldog_description)/urdf/bulldog/bulldog.urdf.xacro" />
   <xacro:include filename="$(find bulldog_gazebo)/urdf/bulldog.gazebo.xacro" />
-  <!-- Gazebo plugin for ROS Control -->
-  <gazebo>
-    <plugin name="gazebo_ros_control" filename="libgazebo_ros_control.so">
-      <robotNamespace>/</robotNamespace>
-    </plugin>
-  </gazebo>
-  <xacro:if value="$(arg dual_ur5_enabled)">
-    <gazebo>
-      <plugin name="gazebo_grasp_fix" filename="libgazebo_grasp_fix.so">
-          <arm>
-            <arm_name>left_arm </arm_name>
-            <palm_link> left_arm_wrist_3_link </palm_link>
-            <gripper_link> left_gripper_finger_1_link_0 </gripper_link>
-            <gripper_link> left_gripper_finger_1_link_1 </gripper_link>
-            <gripper_link> left_gripper_finger_1_link_2 </gripper_link>
-            <gripper_link> left_gripper_finger_1_link_3 </gripper_link>
-            <gripper_link> left_gripper_finger_2_link_0 </gripper_link>
-            <gripper_link> left_gripper_finger_2_link_1 </gripper_link>
-            <gripper_link> left_gripper_finger_2_link_2 </gripper_link>
-            <gripper_link> left_gripper_finger_2_link_3 </gripper_link>
-            <gripper_link> left_gripper_finger_middle_link_0 </gripper_link>
-            <gripper_link> left_gripper_finger_middle_link_1 </gripper_link>
-            <gripper_link> left_gripper_finger_middle_link_2 </gripper_link>
-            <gripper_link> left_gripper_finger_middle_link_3 </gripper_link>
-          </arm>
-          <arm>
-            <arm_name>right_arm </arm_name>
-            <palm_link> right_arm_wrist_3_link  </palm_link>
-            <gripper_link> right_gripper_finger_1_link_0 </gripper_link>
-            <gripper_link> right_gripper_finger_1_link_1 </gripper_link>
-            <gripper_link> right_gripper_finger_1_link_2 </gripper_link>
-            <gripper_link> right_gripper_finger_1_link_3 </gripper_link>
-            <gripper_link> right_gripper_finger_2_link_0 </gripper_link>
-            <gripper_link> right_gripper_finger_2_link_1 </gripper_link>
-            <gripper_link> right_gripper_finger_2_link_2 </gripper_link>
-            <gripper_link> right_gripper_finger_2_link_3 </gripper_link>
-            <gripper_link> right_gripper_finger_middle_link_0 </gripper_link>
-            <gripper_link> right_gripper_finger_middle_link_1 </gripper_link>
-            <gripper_link> right_gripper_finger_middle_link_2 </gripper_link>
-            <gripper_link> right_gripper_finger_middle_link_3 </gripper_link>
-          </arm>
-        <forces_angle_tolerance>100</forces_angle_tolerance>
-        <update_rate>4</update_rate>
-        <grip_count_threshold>4</grip_count_threshold>
-        <max_grip_count>8</max_grip_count>
-        <release_tolerance>0.005</release_tolerance>
-        <disable_collisions_on_attach>false</disable_collisions_on_attach>
-        <contact_topic>__default_topic__</contact_topic>
-      </plugin>
-    </gazebo>
-  </xacro:if>
+  <xacro:bulldog_gazebo_config />
   <xacro:bulldog_robot />
-  <xacro:bulldog_robot_gazebo />
 </robot>
