Commit message: update urdf and srdf

File: src/bulldog/bulldog_description/urdf/bulldog/bulldog_gazebo.urdf.xacro (robot description, xacro)
@@ -8,4 +8,5 @@
   <xacro:include filename="$(find robotiq_s_model_visualization)/cfg/s-model_articulated_macro.xacro" />
   <xacro:include filename="$(find bulldog_description)/urdf/sensors/kinect_camera.urdf.xacro" />
+  <xacro:include filename="$(find realsense2_camera)/urdf/_d415.urdf.xacro"/>
   <xacro:property name="wheel_length" value="0.142" />
   <xacro:property name="wheel_radius" value="0.183" />
@@ -84,16 +85,25 @@
         <origin xyz="0 -0.15945 0.09069" rpy="-0.785 0 ${pi}" />
         </joint>
-        <xacro:s-model_articulated prefix="l_"/>
+        <xacro:s-model_articulated prefix="left_gripper_"/>
         <joint name="left_arm_gripper" type="fixed">
             <parent link="left_arm_ee_link" />
-            <child link="l_palm" />
+            <child link="left_gripper_palm" />
             <origin xyz="0 0 0" rpy="0 0 -1.57" />
         </joint>
-        <xacro:s-model_articulated prefix="r_"/>
+        <!-- realsense d415 -->
+        <!-- <sensor_d415 parent="base_link">
+          <origin xyz="0 0 0" rpy="0 0 0"/>
+        </sensor_d415> -->
+        <xacro:s-model_articulated prefix="right_gripper_"/>
         <joint name="right_arm_gripper" type="fixed">
             <parent link="right_arm_ee_link" />
-            <child link="r_palm" />
+            <child link="right_gripper_palm" />
             <origin xyz="0 0 0" rpy="0 0 -1.57" />
         </joint>
+        <!-- realsense d415 -->
+        <!-- <link name="base_link" />
+        <sensor_d415 parent="base_link">
+          <origin xyz="0 0 0" rpy="0 0 0"/>
+        </sensor_d415> -->
     </xacro:if>
     <!-- laser -->

Commit message: fix bugs for realsense simulation

File: src/bulldog/bulldog_description/urdf/bulldog/bulldog_gazebo.urdf.xacro (robot description, xacro)
@@ -110,5 +110,5 @@
     <!-- kinect -->
     <xacro:if value="$(arg kinect_enabled)">
-      <xacro:kinect_camera />
+      <xacro:kinect_camera prefix="kinect" parent="installation_plate_link" />
     </xacro:if>
     <!-- realsense d415 -->

File: src/bulldog/bulldog_description/urdf/sensors/kinect_camera.urdf.xacro (robot description, xacro)
@@ -48,7 +48,4 @@
       <child link="${prefix}_link" />
     </joint>
-    <gazebo reference="${prefix}_link">
-      <material>Gazebo/Grey</material>
-    </gazebo>
   </xacro:macro>
 </robot>

File: src/bulldog_simulator/bulldog_gazebo/urdf/accessories/kinect_camera.gazebo.xacro (robot description, xacro)
@@ -2,4 +2,9 @@
 <root xmlns:xacro="http://ros.org/wiki/xacro">
   <xacro:macro name="kinect_camera_gazebo" params="prefix">
+    <!-- material -->
+    <gazebo reference="${prefix}_link">
+      <material>Gazebo/Grey</material>
+    </gazebo>
+    <!-- optical joint and link -->
     <joint name="${prefix}_optical_joint" type="fixed">
       <origin xyz="0 0 0" rpy="-1.5708 0 -1.5708"/>
@@ -8,4 +13,5 @@
     </joint>
     <link name="${prefix}_frame_optical"/>
+    <!-- depth camera -->
     <gazebo reference="${prefix}_link">
       <sensor type="depth" name="${prefix}">

File: src/bulldog_simulator/bulldog_gazebo/urdf/accessories/realsense_d415_camera.gazebo.xacro (robot description, xacro)
@@ -2,4 +2,8 @@
 <root xmlns:xacro="http://ros.org/wiki/xacro">
   <xacro:macro name="sensor_d415_gazebo" params="prefix">
+    <!-- material -->
+    <gazebo reference="${prefix}camera_link">
+      <material>Gazebo/Grey</material>
+    </gazebo>
     <!-- color sensor -->
     <gazebo reference="${prefix}camera_depth_frame">

Commit message: upload HARDWARE.md

File: src/bulldog/bulldog_description/urdf/bulldog/bulldog_gazebo.urdf.xacro (robot description, xacro)
@@ -93,5 +93,5 @@
             <parent link="left_arm_ee_link" />
             <child link="left_gripper_palm" />
-            <origin xyz="0 0 0" rpy="0 0 -1.57" />
+            <origin xyz="0 0 0" rpy="0 -2.3562 -1.57" />
         </joint>
         <xacro:robotiq-3f-gripper_articulated prefix="right_gripper_"/>
@@ -99,5 +99,5 @@
             <parent link="right_arm_ee_link" />
             <child link="right_gripper_palm" />
-            <origin xyz="0 0 0" rpy="0 0 -1.57" />
+            <origin xyz="0 0 0" rpy="0 2.3562 -1.57" />
         </joint>
     </xacro:if>
