Commit message: rename materials.urdf

File: src/bulldog/bulldog_description/urdf/bulldog/bulldog.urdf.xacro (robot description, xacro)
@@ -2,5 +2,5 @@
 <robot name="bulldog_robot" xmlns:xacro="http://ros.org/wiki/xacro">
   <xacro:include filename="$(find bulldog_description)/urdf/bulldog/wheel.urdf.xacro" />
-  <xacro:include filename="$(find bulldog_description)/urdf/bulldog/materials.xacro" />
+  <xacro:include filename="$(find bulldog_description)/urdf/bulldog/materials.urdf.xacro" />
   <xacro:include filename="$(find ur_description)/urdf/ur5.urdf.xacro" />
   <xacro:include filename="$(find lms1xx)/urdf/sick_lms1xx.urdf.xacro" />

File: src/bulldog/bulldog_description/urdf/bulldog/materials.urdf.xacro (robot description, xacro)
@@ -1,4 +1,4 @@
 <?xml version="1.0"?>
-<robot>
+<robot name="bulldog_material" xmlns:xacro="http://ros.org/wiki/xacro">
   <material name="black">
     <color rgba="0 0 0 1.0"/>

File: src/bulldog/bulldog_description/urdf/bulldog/wheel.urdf.xacro (robot description, xacro)
@@ -2,47 +2,47 @@
 <robot name="bulldog_wheel" xmlns:xacro="http://ros.org/wiki/xacro">
   <xacro:macro name="bulldog_wheel" params="wheel_prefix *joint_pose">
-  <link name="${wheel_prefix}_wheel_link">
-    <inertial>
-      <mass value="3" />
-      <origin xyz="0 0 0" />
-      <inertia  ixx="0.025" ixy="0" ixz="0" iyy="0.025" iyz="0" izz="0.045" />
-    </inertial>
-    <visual>
-      <origin xyz="0 0 0" rpy="0 0 0" />
-      <geometry>
-        <mesh filename="package://bulldog_description/meshes/wheel.stl" />
-      </geometry>
-      <material name="dark_grey" />
-    </visual>
-    <collision>
-      <origin xyz="0 0 0" rpy="${pi / 2} 0 0" />
-      <geometry>
-        <cylinder length="${wheel_length}" radius="${wheel_radius}" />
-      </geometry>
-    </collision>
-  </link>
-  <gazebo reference="${wheel_prefix}_wheel_link">
-    <mu1 value="1.0"/>
-    <mu2 value="1.0"/>
-    <kp value="10000000.0" />
-    <kd value="1.0" />
-    <fdir1 value="1 0 0"/>
-    <material>Gazebo/DarkGrey</material>
-  </gazebo>
-  <joint name="${wheel_prefix}_wheel_joint" type="continuous">
-    <parent link="base_link"/>
-    <child link="${wheel_prefix}_wheel_link"/>
-    <xacro:insert_block name="joint_pose"/>
-    <axis xyz="0 1 0" rpy="0 0 0" />
-  </joint>
-  <transmission name="${wheel_prefix}_wheel_trans" type="SimpleTransmission">
-    <type>transmission_interface/SimpleTransmission</type>
-    <actuator name="${wheel_prefix}_wheel_motor">
-      <mechanicalReduction>1</mechanicalReduction>
-    </actuator>
-    <joint name="${wheel_prefix}_wheel_joint">
-      <hardwareInterface>VelocityJointInterface</hardwareInterface>
+    <link name="${wheel_prefix}_wheel_link">
+      <inertial>
+        <mass value="3" />
+        <origin xyz="0 0 0" />
+        <inertia  ixx="0.025" ixy="0" ixz="0" iyy="0.025" iyz="0" izz="0.045" />
+      </inertial>
+      <visual>
+        <origin xyz="0 0 0" rpy="0 0 0" />
+        <geometry>
+          <mesh filename="package://bulldog_description/meshes/wheel.stl" />
+        </geometry>
+        <material name="dark_grey" />
+      </visual>
+      <collision>
+        <origin xyz="0 0 0" rpy="${pi / 2} 0 0" />
+        <geometry>
+          <cylinder length="${wheel_length}" radius="${wheel_radius}" />
+        </geometry>
+      </collision>
+    </link>
+    <gazebo reference="${wheel_prefix}_wheel_link">
+      <mu1 value="1.0"/>
+      <mu2 value="1.0"/>
+      <kp value="10000000.0" />
+      <kd value="1.0" />
+      <fdir1 value="1 0 0"/>
+      <material>Gazebo/DarkGrey</material>
+    </gazebo>
+    <joint name="${wheel_prefix}_wheel_joint" type="continuous">
+      <parent link="base_link"/>
+      <child link="${wheel_prefix}_wheel_link"/>
+      <xacro:insert_block name="joint_pose"/>
+      <axis xyz="0 1 0" rpy="0 0 0" />
     </joint>
-  </transmission>
+    <transmission name="${wheel_prefix}_wheel_trans" type="SimpleTransmission">
+      <type>transmission_interface/SimpleTransmission</type>
+      <actuator name="${wheel_prefix}_wheel_motor">
+        <mechanicalReduction>1</mechanicalReduction>
+      </actuator>
+      <joint name="${wheel_prefix}_wheel_joint">
+        <hardwareInterface>VelocityJointInterface</hardwareInterface>
+      </joint>
+    </transmission>
   </xacro:macro>
 </robot>

Commit message: kinect and realsense

File: src/bulldog/bulldog_description/urdf/bulldog/bulldog.urdf.xacro (robot description, xacro)
@@ -8,4 +8,5 @@
   <xacro:include filename="$(find robotiq_s_model_visualization)/cfg/robotiq_hand_macro.urdf.xacro" />
   <xacro:include filename="$(find bulldog_description)/urdf/sensors/kinect_camera.urdf.xacro" />
+  <xacro:include filename="$(find realsense2_camera)/urdf/_d415.urdf.xacro" />
   <xacro:property name="wheel_length" value="0.142" />
   <xacro:property name="wheel_radius" value="0.183" />
@@ -84,10 +85,16 @@
         <origin xyz="0 -0.15945 0.09069" rpy="-0.785 0 ${pi}" />
       </joint>
-      <xacro:robotiq_hand prefix="l_" parent="left_arm_ee_link" reflect="-1">
+      <xacro:robotiq_hand prefix="left_gripper_" parent="left_arm_ee_link" reflect="-1">
         <origin rpy="0 0 -1.57" xyz="0 0 0"/>
       </xacro:robotiq_hand>
-      <xacro:robotiq_hand prefix="r_" parent="right_arm_ee_link" reflect="-1">
+      <xacro:sensor_d415 prefix="left_gripper_sensor_d415_" parent="left_gripper_palm">
+          <origin xyz="0 0 -0.065" rpy="${pi} 0 ${pi / 2}"/>
+        </xacro:sensor_d415>
+      <xacro:robotiq_hand prefix="right_gripper_" parent="right_arm_ee_link" reflect="-1">
         <origin rpy="0 0 -1.57" xyz="0 0 0"/>
       </xacro:robotiq_hand>
+      <xacro:sensor_d415 prefix="right_gripper_sensor_d415_" parent="right_gripper_palm">
+          <origin xyz="0 0 -0.065" rpy="${pi} 0 ${pi / 2}"/>
+        </xacro:sensor_d415>
     </xacro:if>
     <!-- laser -->
@@ -103,5 +110,5 @@
     <!-- kinect -->
     <xacro:if value="$(arg kinect_enabled)">
-      <xacro:kinect_camera />
+      <xacro:kinect_camera prefix="kinect" parent="installation_plate_link" />
     </xacro:if>
   </xacro:macro>

File: src/bulldog/bulldog_description/urdf/bulldog/bulldog_gazebo.urdf.xacro (robot description, xacro)
@@ -11,7 +11,7 @@
   <xacro:property name="wheel_length" value="0.142" />
   <xacro:property name="wheel_radius" value="0.183" />
-  <property name="base_x_size" value="0.85" />
-  <property name="base_y_size" value="0.42" />
-  <property name="base_z_size" value="0.325" />
+  <xacro:property name="base_x_size" value="0.85" />
+  <xacro:property name="base_y_size" value="0.42" />
+  <xacro:property name="base_z_size" value="0.325" />
   <xacro:macro name="bulldog_gazebo_robot">
     <!-- base -->

File: src/bulldog/bulldog_description/urdf/sensors/kinect_camera.urdf.xacro (robot description, xacro)
@@ -26,9 +26,8 @@
 -->
 <robot xmlns:xacro="http://ros.org/wiki/xacro" name="kinect_camera">
-  <xacro:macro name="kinect_camera" params="camera_link_name:=kinect_link
-                                            plate_link_name:=installation_plate_link">
+  <xacro:macro name="kinect_camera" params="prefix parent">
     <!-- Create kinect reference frame -->
     <!-- Add mesh for kinect -->
-    <link name="${camera_link_name}">
+    <link name="${prefix}_link">
       <origin xyz="0 0 0" rpy="0 0 0"/>
       <visual>
@@ -44,10 +43,10 @@
       </collision>
     </link>
-    <joint name="${camera_link_name}_joint" type="fixed">
+    <joint name="${prefix}_joint" type="fixed">
       <origin xyz="0.13 0 0.135" rpy=" 0 0.15 0" />
-      <parent link="${plate_link_name}" />
-      <child link="${camera_link_name}" />
+      <parent link="${parent}" />
+      <child link="${prefix}_link" />
     </joint>
-    <gazebo reference="${camera_link_name}">
+    <gazebo reference="${prefix}_link">
       <material>Gazebo/Black</material>
     </gazebo>

File: src/bulldog_simulator/bulldog_gazebo/urdf/bulldog.gazebo.xacro (robot description, xacro)
@@ -88,82 +88,82 @@
               <kp_position>5.0</kp_position>
               <kd_position>0.5</kd_position>
-             </plugin>
+            </plugin>
         </gazebo>
-        <gazebo reference="l_palm">
+        <gazebo reference="left_gripper">
             <material>Gazebo/Black</material>
         </gazebo>
-        <gazebo reference="r_palm">
+        <gazebo reference="right_gripper">
             <material>Gazebo/Black</material>
         </gazebo>
-        <gazebo reference="l_finger_1_link_0">
+        <gazebo reference="left_gripper_finger_1_link_0">
             <material>Gazebo/Black</material>
         </gazebo>
-        <gazebo reference="r_finger_1_link_0">
+        <gazebo reference="right_gripper_finger_1_link_0">
             <material>Gazebo/Black</material>
         </gazebo>
-        <gazebo reference="l_finger_1_link_1">
+        <gazebo reference="left_gripper_finger_1_link_1">
             <material>Gazebo/Black</material>
         </gazebo>
-        <gazebo reference="r_finger_1_link_1">
+        <gazebo reference="right_gripper_finger_1_link_1">
             <material>Gazebo/Black</material>
         </gazebo>
-        <gazebo reference="l_finger_1_link_2">
+        <gazebo reference="left_gripper_finger_1_link_2">
             <material>Gazebo/Black</material>
         </gazebo>
-        <gazebo reference="r_finger_1_link_2">
+        <gazebo reference="right_gripper_finger_1_link_2">
             <material>Gazebo/Black</material>
         </gazebo>
-        <gazebo reference="l_finger_1_link_3">
+        <gazebo reference="left_gripper_finger_1_link_3">
             <material>Gazebo/Grey</material>
         </gazebo>
-        <gazebo reference="r_finger_1_link_3">
+        <gazebo reference="right_gripper_finger_1_link_3">
             <material>Gazebo/Grey</material>
         </gazebo>
-        <gazebo reference="l_finger_2_link_0">
+        <gazebo reference="left_gripper_finger_2_link_0">
             <material>Gazebo/Black</material>
         </gazebo>
-        <gazebo reference="r_finger_2_link_0">
+        <gazebo reference="right_gripper_finger_2_link_0">
             <material>Gazebo/Black</material>
         </gazebo>
-        <gazebo reference="l_finger_2_link_1">
+        <gazebo reference="left_gripper_finger_2_link_1">
             <material>Gazebo/Black</material>
         </gazebo>
-        <gazebo reference="r_finger_2_link_1">
+        <gazebo reference="right_gripper_finger_2_link_1">
             <material>Gazebo/Black</material>
         </gazebo>
-        <gazebo reference="l_finger_2_link_2">
+        <gazebo reference="left_gripper_finger_2_link_2">
             <material>Gazebo/Black</material>
         </gazebo>
-        <gazebo reference="r_finger_2_link_2">
+        <gazebo reference="right_gripper_finger_2_link_2">
             <material>Gazebo/Black</material>
         </gazebo>
-        <gazebo reference="l_finger_2_link_3">
+        <gazebo reference="left_gripper_finger_2_link_3">
             <material>Gazebo/Grey</material>
         </gazebo>
-        <gazebo reference="r_finger_2_link_3">
+        <gazebo reference="right_gripper_finger_2_link_3">
             <material>Gazebo/Grey</material>
         </gazebo>
-        <gazebo reference="l_finger_middle_link_0">
+        <gazebo reference="left_gripper_finger_middle_link_0">
             <material>Gazebo/Black</material>
         </gazebo>
-        <gazebo reference="r_finger_middle_link_0">
+        <gazebo reference="right_gripper_finger_middle_link_0">
             <material>Gazebo/Black</material>
         </gazebo>
-        <gazebo reference="l_finger_middle_link_1">
+        <gazebo reference="left_gripper_finger_middle_link_1">
             <material>Gazebo/Black</material>
         </gazebo>
-        <gazebo reference="r_finger_middle_link_1">
+        <gazebo reference="right_gripper_finger_middle_link_1">
             <material>Gazebo/Black</material>
         </gazebo>
-        <gazebo reference="l_finger_middle_link_2">
+        <gazebo reference="left_gripper_finger_middle_link_2">
             <material>Gazebo/Black</material>
         </gazebo>
-        <gazebo reference="r_finger_middle_link_2">
+        <gazebo reference="right_gripper_finger_middle_link_2">
             <material>Gazebo/Black</material>
         </gazebo>
-        <gazebo reference="l_finger_middle_link_3">
+        <gazebo reference="left_gripper_finger_middle_link_3">
             <material>Gazebo/Grey</material>
         </gazebo>
-        <gazebo reference="r_finger_middle_link_3">
+        <gazebo reference="right_gripper_finger_middle_link_3">
             <material>Gazebo/Grey</material>
         </gazebo>
@@ -171,5 +171,5 @@
     <!-- kinect -->
     <xacro:if value="$(arg kinect_enabled)">
-      <xacro:kinect_camera_gazebo prefix="camera"/>
+      <xacro:kinect_camera_gazebo prefix="kinect"/>
     </xacro:if>
   </xacro:macro>

File: src/bulldog_simulator/bulldog_gazebo/urdf/description.gazebo.xacro (robot description, xacro)
@@ -25,6 +25,7 @@
   <xacro:arg name="ur5_enabled" default="false" />
   <xacro:arg name="kinect_enabled" default="false" />
-  <xacro:arg name="dual_ur5_enabled" default="true"/>
-  <xacro:arg name="robotiq_grippers_enabled" default="true"/>
+  <xacro:arg name="realsense_enabled" default="false" />
+  <xacro:arg name="dual_ur5_enabled" default="true" />
+  <xacro:arg name="robotiq_grippers_enabled" default="true" />
   <xacro:include filename="$(find bulldog_description)/urdf/bulldog/bulldog.urdf.xacro" />
   <xacro:include filename="$(find bulldog_gazebo)/urdf/bulldog.gazebo.xacro" />
@@ -35,47 +36,49 @@
     </plugin>
   </gazebo>
-  <gazebo>
-    <plugin name="gazebo_grasp_fix" filename="libgazebo_grasp_fix.so">
-        <arm>
-           <arm_name>left_arm </arm_name>
-           <palm_link> left_arm_wrist_3_link </palm_link>
-           <gripper_link> l_finger_1_link_0 </gripper_link>
-           <gripper_link> l_finger_1_link_1 </gripper_link>
-           <gripper_link> l_finger_1_link_2 </gripper_link>
-           <gripper_link> l_finger_1_link_3 </gripper_link>
-           <gripper_link> l_finger_2_link_0 </gripper_link>
-           <gripper_link> l_finger_2_link_1 </gripper_link>
-           <gripper_link> l_finger_2_link_2 </gripper_link>
-           <gripper_link> l_finger_2_link_3 </gripper_link>
-           <gripper_link> l_finger_middle_link_0 </gripper_link>
-           <gripper_link> l_finger_middle_link_1 </gripper_link>
-           <gripper_link> l_finger_middle_link_2 </gripper_link>
-           <gripper_link> l_finger_middle_link_3 </gripper_link>
-        </arm>
-        <arm>
-           <arm_name>right_arm </arm_name>
-           <palm_link> right_arm_wrist_3_link  </palm_link>
-           <gripper_link> r_finger_1_link_0 </gripper_link>
-           <gripper_link> r_finger_1_link_1 </gripper_link>
-           <gripper_link> r_finger_1_link_2 </gripper_link>
-           <gripper_link> r_finger_1_link_3 </gripper_link>
-           <gripper_link> r_finger_2_link_0 </gripper_link>
-           <gripper_link> r_finger_2_link_1 </gripper_link>
-           <gripper_link> r_finger_2_link_2 </gripper_link>
-           <gripper_link> r_finger_2_link_3 </gripper_link>
-           <gripper_link> r_finger_middle_link_0 </gripper_link>
-           <gripper_link> r_finger_middle_link_1 </gripper_link>
-           <gripper_link> r_finger_middle_link_2 </gripper_link>
-           <gripper_link> r_finger_middle_link_3 </gripper_link>
-        </arm>
-       <forces_angle_tolerance>100</forces_angle_tolerance>
-       <update_rate>4</update_rate>
-       <grip_count_threshold>4</grip_count_threshold>
-       <max_grip_count>8</max_grip_count>
-       <release_tolerance>0.005</release_tolerance>
-       <disable_collisions_on_attach>false</disable_collisions_on_attach>
-       <contact_topic>__default_topic__</contact_topic>
-    </plugin>
-  </gazebo>
+  <xacro:if value="$(arg dual_ur5_enabled)">
+    <gazebo>
+      <plugin name="gazebo_grasp_fix" filename="libgazebo_grasp_fix.so">
+          <arm>
+            <arm_name>left_arm </arm_name>
+            <palm_link> left_arm_wrist_3_link </palm_link>
+            <gripper_link> left_gripper_finger_1_link_0 </gripper_link>
+            <gripper_link> left_gripper_finger_1_link_1 </gripper_link>
+            <gripper_link> left_gripper_finger_1_link_2 </gripper_link>
+            <gripper_link> left_gripper_finger_1_link_3 </gripper_link>
+            <gripper_link> left_gripper_finger_2_link_0 </gripper_link>
+            <gripper_link> left_gripper_finger_2_link_1 </gripper_link>
+            <gripper_link> left_gripper_finger_2_link_2 </gripper_link>
+            <gripper_link> left_gripper_finger_2_link_3 </gripper_link>
+            <gripper_link> left_gripper_finger_middle_link_0 </gripper_link>
+            <gripper_link> left_gripper_finger_middle_link_1 </gripper_link>
+            <gripper_link> left_gripper_finger_middle_link_2 </gripper_link>
+            <gripper_link> left_gripper_finger_middle_link_3 </gripper_link>
+          </arm>
+          <arm>
+            <arm_name>right_arm </arm_name>
+            <palm_link> right_arm_wrist_3_link  </palm_link>
+            <gripper_link> right_gripper_finger_1_link_0 </gripper_link>
+            <gripper_link> right_gripper_finger_1_link_1 </gripper_link>
+            <gripper_link> right_gripper_finger_1_link_2 </gripper_link>
+            <gripper_link> right_gripper_finger_1_link_3 </gripper_link>
+            <gripper_link> right_gripper_finger_2_link_0 </gripper_link>
+            <gripper_link> right_gripper_finger_2_link_1 </gripper_link>
+            <gripper_link> right_gripper_finger_2_link_2 </gripper_link>
+            <gripper_link> right_gripper_finger_2_link_3 </gripper_link>
+            <gripper_link> right_gripper_finger_middle_link_0 </gripper_link>
+            <gripper_link> right_gripper_finger_middle_link_1 </gripper_link>
+            <gripper_link> right_gripper_finger_middle_link_2 </gripper_link>
+            <gripper_link> right_gripper_finger_middle_link_3 </gripper_link>
+          </arm>
+        <forces_angle_tolerance>100</forces_angle_tolerance>
+        <update_rate>4</update_rate>
+        <grip_count_threshold>4</grip_count_threshold>
+        <max_grip_count>8</max_grip_count>
+        <release_tolerance>0.005</release_tolerance>
+        <disable_collisions_on_attach>false</disable_collisions_on_attach>
+        <contact_topic>__default_topic__</contact_topic>
+      </plugin>
+    </gazebo>
+  </xacro:if>
   <xacro:bulldog_robot />
   <xacro:bulldog_robot_gazebo />

File: src/robotiq/robotiq_s_model_visualization/cfg/robotiq_hand_macro.urdf.xacro (robot description, xacro)
@@ -6,5 +6,5 @@
 there are multiple hands then a prefix followed by an "_" is needed.
 -->
-<robot xmlns:xacro="http://www.ros.org/wiki/xacro" name="robotiq_hand">
+<robot xmlns:xacro="http://ros.org/wiki/xacro" name="robotiq_hand">
   <xacro:macro name="robotiq_finger" params="prefix">
     <!-- Link list -->
