Commit message: realsense simulation

File: src/bulldog/bulldog_description/urdf/bulldog/bulldog.urdf.xacro (robot description, xacro)
@@ -85,16 +85,12 @@
         <origin xyz="0 -0.15945 0.09069" rpy="-0.785 0 ${pi}" />
       </joint>
+      <!-- If you modify the name of the grippers, remember to change the *prefix* in line
+           780 and 782 accordingly of $(find robotiq_s_model_articulated_gazebo_plugins)/src/RobotiqHandPlugin.cpp. -->
       <xacro:robotiq_hand prefix="left_gripper_" parent="left_arm_ee_link" reflect="-1">
         <origin rpy="0 0 -1.57" xyz="0 0 0"/>
       </xacro:robotiq_hand>
-      <xacro:sensor_d415 prefix="left_gripper_sensor_d415_" parent="left_gripper_palm">
-          <origin xyz="0 0 -0.065" rpy="${pi} 0 ${pi / 2}"/>
-        </xacro:sensor_d415>
       <xacro:robotiq_hand prefix="right_gripper_" parent="right_arm_ee_link" reflect="-1">
         <origin rpy="0 0 -1.57" xyz="0 0 0"/>
       </xacro:robotiq_hand>
-      <xacro:sensor_d415 prefix="right_gripper_sensor_d415_" parent="right_gripper_palm">
-          <origin xyz="0 0 -0.065" rpy="${pi} 0 ${pi / 2}"/>
-        </xacro:sensor_d415>
     </xacro:if>
     <!-- laser -->
@@ -112,4 +108,13 @@
       <xacro:kinect_camera prefix="kinect" parent="installation_plate_link" />
     </xacro:if>
+    <!-- realsense d415 -->
+    <xacro:if value="$(arg realsense_enabled)">
+      <xacro:sensor_d415 prefix="left_gripper_sensor_d415_" parent="left_gripper_palm">
+        <origin xyz="0 0 -0.065" rpy="${pi} 0 ${pi / 2}"/>
+      </xacro:sensor_d415>
+      <xacro:sensor_d415 prefix="right_gripper_sensor_d415_" parent="right_gripper_palm">
+          <origin xyz="0 0 -0.065" rpy="${pi} 0 ${pi / 2}"/>
+        </xacro:sensor_d415>
+    </xacro:if>
   </xacro:macro>
 </robot>

File: src/bulldog/bulldog_description/urdf/bulldog/bulldog_gazebo.urdf.xacro (robot description, xacro)
@@ -91,7 +91,4 @@
             <origin xyz="0 0 0" rpy="0 0 -1.57" />
         </joint>
-        <xacro:sensor_d415 prefix="left_gripper_sensor_d415_" parent="left_gripper_palm">
-          <origin xyz="0 0 -0.065" rpy="${pi} 0 ${pi / 2}"/>
-        </xacro:sensor_d415>
         <xacro:s-model_articulated prefix="right_gripper_"/>
         <joint name="right_arm_gripper" type="fixed">
@@ -100,7 +97,4 @@
             <origin xyz="0 0 0" rpy="0 0 -1.57" />
         </joint>
-        <xacro:sensor_d415 prefix="right_gripper_sensor_d415_" parent="right_gripper_palm">
-          <origin xyz="0 0 -0.065" rpy="${pi} 0 ${pi / 2}"/>
-        </xacro:sensor_d415>
     </xacro:if>
     <!-- laser -->
@@ -118,4 +112,13 @@
       <xacro:kinect_camera />
     </xacro:if>
+    <!-- realsense d415 -->
+    <xacro:if value="$(arg realsense_enabled)">
+      <xacro:sensor_d415 prefix="left_gripper_sensor_d415_" parent="left_gripper_palm">
+        <origin xyz="0 0 -0.065" rpy="${pi} 0 ${pi / 2}"/>
+      </xacro:sensor_d415>
+      <xacro:sensor_d415 prefix="right_gripper_sensor_d415_" parent="right_gripper_palm">
+          <origin xyz="0 0 -0.065" rpy="${pi} 0 ${pi / 2}"/>
+      </xacro:sensor_d415>
+    </xacro:if>
   </xacro:macro>
 </robot>

File: src/bulldog/bulldog_description/urdf/sensors/kinect_camera.urdf.xacro (robot description, xacro)
@@ -49,5 +49,5 @@
     </joint>
     <gazebo reference="${prefix}_link">
-      <material>Gazebo/Black</material>
+      <material>Gazebo/Grey</material>
     </gazebo>
   </xacro:macro>

File: src/bulldog_simulator/bulldog_gazebo/urdf/accessories/kinect_camera.gazebo.xacro (robot description, xacro)
@@ -11,5 +11,5 @@
       <sensor type="depth" name="${prefix}">
         <always_on>true</always_on>
-        <update_rate>20.0</update_rate>
+        <update_rate>30.0</update_rate>
         <camera>
           <horizontal_fov>${60.0 * pi / 180.0}</horizontal_fov>
@@ -24,6 +24,6 @@
           </clip>
         </camera>
-        <plugin name="kinect_${prefix}_controller" filename="libgazebo_ros_openni_kinect.so">
-          <cameraName>${prefix}</cameraName>
+        <plugin name="${prefix}_controller" filename="libgazebo_ros_openni_kinect.so">
+          <cameraName>${prefix}_camera</cameraName>
           <alwaysOn>true</alwaysOn>
           <updateRate>10</updateRate>

File: src/bulldog_simulator/bulldog_gazebo/urdf/bulldog.gazebo.xacro (robot description, xacro)
@@ -23,4 +23,5 @@
 <robot name="bulldog_robot_gazebo" xmlns:xacro="http://ros.org/wiki/xacro">
   <xacro:include filename="$(find bulldog_gazebo)/urdf/accessories/kinect_camera.gazebo.xacro"/>
+  <xacro:include filename="$(find bulldog_gazebo)/urdf/accessories/realsense_d415_camera.gazebo.xacro"/>
   <xacro:macro name="bulldog_robot_gazebo">
     <!-- imu -->
@@ -53,25 +54,27 @@
     <!-- ur5 arm -->
     <!--Remove when https://github.com/ros-industrial/universal_robot/pull/168 is resolved -->
-    <gazebo reference="ur5_arm_shoulder_link">
-      <selfCollide>true</selfCollide>
-    </gazebo>
-    <gazebo reference="ur5_arm_upper_arm_link">
-      <selfCollide>true</selfCollide>
-    </gazebo>
-    <gazebo reference="ur5_arm_forearm_link">
-      <selfCollide>true</selfCollide>
-    </gazebo>
-    <gazebo reference="ur5_arm_wrist_1_link">
-      <selfCollide>true</selfCollide>
-    </gazebo>
-    <gazebo reference="ur5_arm_wrist_3_link">
-      <selfCollide>true</selfCollide>
-    </gazebo>
-    <gazebo reference="ur5_arm_wrist_2_link">
-      <selfCollide>true</selfCollide>
-    </gazebo>
-    <gazebo reference="ur5_arm_ee_link">
-      <selfCollide>true</selfCollide>
-    </gazebo>
+    <xacro:if value="$(arg ur5_enabled)">
+      <gazebo reference="ur5_arm_shoulder_link">
+        <selfCollide>true</selfCollide>
+      </gazebo>
+      <gazebo reference="ur5_arm_upper_arm_link">
+        <selfCollide>true</selfCollide>
+      </gazebo>
+      <gazebo reference="ur5_arm_forearm_link">
+        <selfCollide>true</selfCollide>
+      </gazebo>
+      <gazebo reference="ur5_arm_wrist_1_link">
+        <selfCollide>true</selfCollide>
+      </gazebo>
+      <gazebo reference="ur5_arm_wrist_3_link">
+        <selfCollide>true</selfCollide>
+      </gazebo>
+      <gazebo reference="ur5_arm_wrist_2_link">
+        <selfCollide>true</selfCollide>
+      </gazebo>
+      <gazebo reference="ur5_arm_ee_link">
+        <selfCollide>true</selfCollide>
+      </gazebo>
+    </xacro:if>
     <!-- robotiq grippers -->
     <xacro:if value="$(arg robotiq_grippers_enabled)">
@@ -173,4 +176,9 @@
       <xacro:kinect_camera_gazebo prefix="kinect"/>
     </xacro:if>
+    <!-- realsense -->
+    <xacro:if value="$(arg realsense_enabled)">
+      <xacro:sensor_d415_gazebo prefix="left_gripper_sensor_d415_"/>
+      <xacro:sensor_d415_gazebo prefix="right_gripper_sensor_d415_"/>
+    </xacro:if>
   </xacro:macro>
 </robot>

Commit message: conform bulldog gazebo and moveit configuration

File: src/bulldog/bulldog_description/urdf/bulldog/bulldog.urdf.xacro (robot description, xacro)
@@ -111,5 +111,5 @@
     <xacro:if value="$(arg realsense_enabled)">
       <xacro:sensor_d415 prefix="left_gripper_sensor_d415_" parent="left_gripper_palm">
-        <origin xyz="0 0 -0.065" rpy="${pi} 0 ${pi / 2}"/>
+        <origin xyz="0 0 0.065" rpy="0 0 ${pi / 2}"/>
       </xacro:sensor_d415>
       <xacro:sensor_d415 prefix="right_gripper_sensor_d415_" parent="right_gripper_palm">

File: src/bulldog/bulldog_description/urdf/bulldog/bulldog_gazebo.urdf.xacro (robot description, xacro)
@@ -115,5 +115,5 @@
     <xacro:if value="$(arg realsense_enabled)">
       <xacro:sensor_d415 prefix="left_gripper_sensor_d415_" parent="left_gripper_palm">
-        <origin xyz="0 0 -0.065" rpy="${pi} 0 ${pi / 2}"/>
+        <origin xyz="0 0 0.065" rpy="0 0 ${pi / 2}"/>
       </xacro:sensor_d415>
       <xacro:sensor_d415 prefix="right_gripper_sensor_d415_" parent="right_gripper_palm">

File: src/bulldog_simulator/bulldog_gazebo/urdf/bulldog.gazebo.xacro (robot description, xacro)
@@ -97,5 +97,5 @@
               <gripper_link> left_gripper_finger_2_link_2 </gripper_link>
               <gripper_link> left_gripper_finger_2_link_3 </gripper_link>
-              <gripper_link> left_gripper_finger_middle_link_0 </gripper_link>
+              <!-- <gripper_link> left_gripper_finger_middle_link_0 </gripper_link> -->
               <gripper_link> left_gripper_finger_middle_link_1 </gripper_link>
               <gripper_link> left_gripper_finger_middle_link_2 </gripper_link>
@@ -113,5 +113,5 @@
               <gripper_link> right_gripper_finger_2_link_2 </gripper_link>
               <gripper_link> right_gripper_finger_2_link_3 </gripper_link>
-              <gripper_link> right_gripper_finger_middle_link_0 </gripper_link>
+              <!-- <gripper_link> right_gripper_finger_middle_link_0 </gripper_link> -->
               <gripper_link> right_gripper_finger_middle_link_1 </gripper_link>
               <gripper_link> right_gripper_finger_middle_link_2 </gripper_link>
@@ -198,10 +198,10 @@
             <material>Gazebo/Grey</material>
         </gazebo>
-        <gazebo reference="left_gripper_finger_middle_link_0">
+        <!-- <gazebo reference="left_gripper_finger_middle_link_0">
             <material>Gazebo/Black</material>
         </gazebo>
         <gazebo reference="right_gripper_finger_middle_link_0">
             <material>Gazebo/Black</material>
-        </gazebo>
+        </gazebo> -->
         <gazebo reference="left_gripper_finger_middle_link_1">
             <material>Gazebo/Black</material>

Commit message: manipulating grippers

File: src/bulldog/bulldog_description/urdf/bulldog/bulldog.urdf.xacro (robot description, xacro)
@@ -111,5 +111,5 @@
     <xacro:if value="$(arg realsense_enabled)">
       <xacro:sensor_d415 prefix="left_gripper_sensor_d415_" parent="left_gripper_palm">
-        <origin xyz="0 0 0.065" rpy="0 0 ${pi / 2}"/>
+        <origin xyz="0 0 -0.065" rpy="${pi} 0 ${pi / 2}"/>
       </xacro:sensor_d415>
       <xacro:sensor_d415 prefix="right_gripper_sensor_d415_" parent="right_gripper_palm">

File: src/bulldog/bulldog_description/urdf/bulldog/bulldog_gazebo.urdf.xacro (robot description, xacro)
@@ -115,5 +115,5 @@
     <xacro:if value="$(arg realsense_enabled)">
       <xacro:sensor_d415 prefix="left_gripper_sensor_d415_" parent="left_gripper_palm">
-        <origin xyz="0 0 0.065" rpy="0 0 ${pi / 2}"/>
+        <origin xyz="0 0 -0.065" rpy="${pi} 0 ${pi / 2}"/>
       </xacro:sensor_d415>
       <xacro:sensor_d415 prefix="right_gripper_sensor_d415_" parent="right_gripper_palm">

File: src/bulldog_simulator/bulldog_gazebo/urdf/bulldog.gazebo.xacro (robot description, xacro)
@@ -97,5 +97,5 @@
               <gripper_link> left_gripper_finger_2_link_2 </gripper_link>
               <gripper_link> left_gripper_finger_2_link_3 </gripper_link>
-              <!-- <gripper_link> left_gripper_finger_middle_link_0 </gripper_link> -->
+              <gripper_link> left_gripper_finger_middle_link_0 </gripper_link>
               <gripper_link> left_gripper_finger_middle_link_1 </gripper_link>
               <gripper_link> left_gripper_finger_middle_link_2 </gripper_link>
@@ -113,5 +113,5 @@
               <gripper_link> right_gripper_finger_2_link_2 </gripper_link>
               <gripper_link> right_gripper_finger_2_link_3 </gripper_link>
-              <!-- <gripper_link> right_gripper_finger_middle_link_0 </gripper_link> -->
+              <gripper_link> right_gripper_finger_middle_link_0 </gripper_link>
               <gripper_link> right_gripper_finger_middle_link_1 </gripper_link>
               <gripper_link> right_gripper_finger_middle_link_2 </gripper_link>
@@ -198,10 +198,10 @@
             <material>Gazebo/Grey</material>
         </gazebo>
-        <!-- <gazebo reference="left_gripper_finger_middle_link_0">
+        <gazebo reference="left_gripper_finger_middle_link_0">
             <material>Gazebo/Black</material>
         </gazebo>
         <gazebo reference="right_gripper_finger_middle_link_0">
             <material>Gazebo/Black</material>
-        </gazebo> -->
+        </gazebo>
         <gazebo reference="left_gripper_finger_middle_link_1">
             <material>Gazebo/Black</material>

File: src/bulldog_simulator/bulldog_gazebo/urdf/description.gazebo.xacro (robot description, xacro)
@@ -28,7 +28,7 @@
   <xacro:arg name="dual_ur5_enabled" default="true" />
   <xacro:arg name="robotiq_grippers_enabled" default="true" />
-  <xacro:include filename="$(find bulldog_description)/urdf/bulldog/bulldog_gazebo.urdf.xacro" />
+  <xacro:include filename="$(find bulldog_description)/urdf/bulldog/bulldog.urdf.xacro" />
   <xacro:include filename="$(find bulldog_gazebo)/urdf/bulldog.gazebo.xacro" />
   <xacro:bulldog_gazebo_config />
-  <xacro:bulldog_gazebo_robot />
+  <xacro:bulldog_robot />
 </robot>

File: src/robotiq/robotiq_s_model_visualization/cfg/robotiq_hand_macro.urdf.xacro (robot description, xacro)
@@ -16,7 +16,10 @@
           <mesh filename="package://robotiq_s_model_visualization/meshes/s-model_articulated/visual/link_0.STL" />
         </geometry>
-        <material name="green">
+        <!-- <material name="green">
           <color rgba="0 1 0 1"/>
-        </material>
+        </material> -->
+        <material name="gray">
+					<color rgba="0.2 0.2 0.2 1"/>
+				</material>
       </visual>
       <collision>
@@ -46,5 +49,6 @@
           <mesh filename="package://robotiq_s_model_visualization/meshes/s-model_articulated/visual/link_1.STL" />
         </geometry>
-        <material name="green"/>
+        <!-- <material name="green"/> -->
+				<material name="gray"/>
       </visual>
       <collision>
@@ -79,5 +83,6 @@
           <mesh filename="package://robotiq_s_model_visualization/meshes/s-model_articulated/visual/link_2.STL" />
         </geometry>
-        <material name="green"/>
+        <!-- <material name="green"/> -->
+				<material name="gray"/>
       </visual>
       <collision>
@@ -110,5 +115,6 @@
           <mesh filename="package://robotiq_s_model_visualization/meshes/s-model_articulated/visual/link_3.STL" />
         </geometry>
-        <material name="green"/>
+        <!-- <material name="green"/> -->
+				<material name="gray"/>
       </visual>
       <collision>
@@ -136,5 +142,5 @@
     <!-- Link proximal actuating hinge -->
     <link name="${prefix}link_proximal_actuating_hinge">
-      <visual>
+      <!-- <visual>
         <origin rpy="0 0 0" xyz="0.01429 0 0"/>
         <geometry>
@@ -147,5 +153,5 @@
           <box size="0.02858 .0075 .002"/>
         </geometry>
-      </collision>
+      </collision> -->
       <inertial>
         <origin rpy="0 0 0" xyz="0.0012 -0.00162 -0.00161"/>
@@ -165,5 +171,5 @@
     <!-- Link paraproximal actuating hinge -->
     <link name="${prefix}link_paraproximal_actuating_hinge">
-      <visual>
+      <!-- <visual>
         <origin rpy="0 0 0" xyz="0.01143 0 0"/>
         <geometry>
@@ -176,5 +182,5 @@
           <box size="0.02286 .0075 .002"/>
         </geometry>
-      </collision>
+      </collision> -->
       <inertial>
         <origin rpy="0 0 0" xyz="0.0064 0 0"/>
@@ -195,5 +201,5 @@
     <!-- Link proximal actuating bar -->
     <link name="${prefix}link_proximal_actuating_bar">
-      <visual>
+      <!-- <visual>
         <origin rpy="0 0 0" xyz="0.026789 0 0"/>
         <geometry>
@@ -206,5 +212,5 @@
           <box size="0.05398 .0075 .002"/>
         </geometry>
-      </collision>
+      </collision> -->
       <inertial>
         <origin rpy="0 0 0" xyz="0.02699 -0.00122 0"/>
@@ -224,5 +230,5 @@
     <!-- Link paraproximal bar -->
     <link name="${prefix}link_paraproximal_bar">
-      <visual>
+      <!-- <visual>
         <origin rpy="0 0 0" xyz="0.02885 0 0"/>
         <geometry>
@@ -235,5 +241,5 @@
           <box size="0.05770 .0075 .002"/>
         </geometry>
-      </collision>
+      </collision> -->
       <inertial>
         <origin rpy="0 0 0" xyz="0.02858 -0.00129 0"/>
@@ -253,16 +259,16 @@
     <!-- Link median actuating hinge -->
     <link name="${prefix}link_median_actuating_hinge">
-      <visual>
+      <!-- <visual>
         <origin rpy="0 0 0" xyz="0 0 0"/>
         <geometry>
+          <box size="0.0 0.0 0.0"/>
+        </geometry>
+      </visual>
+      <collision>
+        <origin rpy="0 0 0" xyz="0 0 0"/>
+         <geometry>
           <box size=".02 .02 .002"/>
         </geometry>
-      </visual>
-      <collision>
-        <origin rpy="0 0 0" xyz="0 0 0"/>
-         <geometry>
-          <box size=".02 .02 .002"/>
-        </geometry>
-      </collision>
+      </collision> -->
       <inertial>
         <origin rpy="0 0 0" xyz="0.0092 0.00514 0"/>
@@ -282,16 +288,16 @@
     <!-- Link median bar -->
     <link name="${prefix}link_median_bar">
-      <visual>
+      <!-- <visual>
         <origin rpy="0 0 0" xyz="0.01905 0 0"/>
         <geometry>
+          <box size="0.0 0.0 0.0"/>
+        </geometry>
+      </visual>
+      <collision>
+        <origin rpy="0 0 0" xyz="0.01905 0 0"/>
+         <geometry>
           <box size="0.0381 .0075 .002"/>
         </geometry>
-      </visual>
-      <collision>
-        <origin rpy="0 0 0" xyz="0.01905 0 0"/>
-         <geometry>
-          <box size="0.0381 .0075 .002"/>
-        </geometry>
-      </collision>
+      </collision> -->
       <inertial>
         <origin rpy="0 0 0" xyz="0.01905 -0.00107 0"/>
@@ -311,5 +317,5 @@
     <!-- Link paramedian hinge -->
     <link name="${prefix}link_paramedian_hinge">
-      <visual>
+      <!-- <visual>
         <origin rpy="0 0 0" xyz="0 0 0"/>
         <geometry>
@@ -322,5 +328,5 @@
           <box size=".02 .02 .002"/>
         </geometry>
-      </collision>
+      </collision> -->
       <inertial>
         <origin rpy="0 0 0" xyz="-0.01025 0.00046 0"/>
@@ -340,5 +346,5 @@
     <!-- Link median bar underactuated -->
     <link name="${prefix}link_median_bar_underactuated">
-      <visual>
+      <!-- <visual>
         <origin rpy="0 0 0" xyz="0.01905 0 0"/>
         <geometry>
@@ -351,5 +357,5 @@
           <box size="0.0381 .0075 .002"/>
         </geometry>
-      </collision>
+      </collision> -->
       <inertial>
         <origin rpy="0 0 0" xyz="0.01905 -0.00107 0"/>
@@ -369,5 +375,5 @@
     <!-- Link paradistal hinge -->
     <link name="${prefix}link_paradistal_hinge">
-      <visual>
+      <!-- <visual>
         <origin rpy="0 0 0" xyz="0 0 0"/>
         <geometry>
@@ -380,5 +386,5 @@
           <box size=".02 0.02 .002"/>
         </geometry>
-      </collision>
+      </collision> -->
       <inertial>
         <origin rpy="0 0 0" xyz="0.00548 0 0"/>
@@ -650,6 +656,9 @@
             <mesh filename="package://robotiq_s_model_visualization/meshes/s-model_articulated/visual/palm.STL" />
           </geometry>
-          <material name="green">
+          <!-- <material name="green">
             <color rgba="0 1 0 1"/>
+          </material> -->
+          <material name="gray">
+            <color rgba="0.2 0.2 0.2 1"/>
           </material>
         </visual>
@@ -658,5 +667,6 @@
           <origin rpy="0 0 0" xyz="0 0 0"/>
           <geometry>
-            <box size="0.1 0.1 0.1"/>
+            <!-- <box size="0.1 0.1 0.1"/> -->
+  					<mesh filename="package://robotiq_s_model_visualization/meshes/s-model_articulated/collision/palm.STL" />
           </geometry>
           <material name="yellow">
@@ -674,4 +684,9 @@
         <mu2>1.1</mu2>
       </gazebo>
+  		<link name="${prefix}tool0"/>
+      <gazebo reference="${prefix}tool0">
+        <mu1>1.1</mu1>
+        <mu2>1.1</mu2>
+      </gazebo>
     <!-- End of link list -->
     <!-- Joint list -->
@@ -714,4 +729,12 @@
       <implicitSpringDamper>1</implicitSpringDamper>
     </gazebo>
+    <joint name="${prefix}palm_tool0" type="fixed">
+			<parent link="${prefix}palm"/>
+			<child link="${prefix}tool0"/>
+			<origin xyz="0.0 0.0875 0.0" rpy="0 0 1.5707"/>
+		</joint>
+    <gazebo reference="${prefix}palm_finger_middle_joint">
+      <implicitSpringDamper>1</implicitSpringDamper>
+    </gazebo>
     <!-- end of joint list -->
   </xacro:macro>

Commit message: grasp demo works basically!

File: src/bulldog/bulldog_description/urdf/bulldog/bulldog.urdf.xacro (robot description, xacro)
@@ -111,5 +111,5 @@
     <xacro:if value="$(arg realsense_enabled)">
       <xacro:sensor_d415 prefix="left_gripper_sensor_d415_" parent="left_gripper_palm">
-        <origin xyz="0 0 -0.065" rpy="${pi} 0 ${pi / 2}"/>
+        <origin xyz="0 0 0.065" rpy="0 0 ${pi / 2}"/>
       </xacro:sensor_d415>
       <xacro:sensor_d415 prefix="right_gripper_sensor_d415_" parent="right_gripper_palm">

Commit message: simplify robotiq gripper model

File: src/bulldog/bulldog_description/urdf/bulldog/bulldog.urdf.xacro (robot description, xacro)
@@ -6,5 +6,5 @@
   <xacro:include filename="$(find ur_description)/urdf/ur5.urdf.xacro" />
   <xacro:include filename="$(find lms1xx)/urdf/sick_lms1xx.urdf.xacro" />
-  <xacro:include filename="$(find robotiq_3f_gripper_visualization)/cfg/robotiq_hand_macro.urdf.xacro" />
+  <xacro:include filename="$(find robotiq_3f_gripper_visualization)/cfg/robotiq-3f-gripper_articulated_macro.xacro" />
   <xacro:include filename="$(find bulldog_description)/urdf/sensors/kinect_camera.urdf.xacro" />
   <xacro:include filename="$(find realsense2_description)/urdf/_d415.urdf.xacro" />
@@ -87,10 +87,16 @@
       <!-- If you modify the name of the grippers, remember to change the *prefix* in line
            780 and 782 accordingly of $(find robotiq_s_model_articulated_gazebo_plugins)/src/RobotiqHandPlugin.cpp. -->
-      <xacro:robotiq_hand prefix="left_gripper_" parent="left_arm_ee_link" reflect="-1">
-        <origin rpy="0 0 -1.57" xyz="0 0 0"/>
-      </xacro:robotiq_hand>
-      <xacro:robotiq_hand prefix="right_gripper_" parent="right_arm_ee_link" reflect="-1">
-        <origin rpy="0 0 -1.57" xyz="0 0 0"/>
-      </xacro:robotiq_hand>
+        <xacro:robotiq-3f-gripper_articulated prefix="left_gripper_"/>
+        <joint name="left_arm_gripper_joint" type="fixed">
+            <parent link="left_arm_ee_link" />
+            <child link="left_gripper_palm" />
+            <origin xyz="0 0 0" rpy="0 0 -1.57" />
+        </joint>
+        <xacro:robotiq-3f-gripper_articulated prefix="right_gripper_"/>
+        <joint name="right_arm_gripper_joint" type="fixed">
+            <parent link="right_arm_ee_link" />
+            <child link="right_gripper_palm" />
+            <origin xyz="0 0 0" rpy="0 0 -1.57" />
+        </joint>
     </xacro:if>
     <!-- laser -->

File: src/bulldog_simulator/bulldog_gazebo/urdf/bulldog.gazebo.xacro (robot description, xacro)
@@ -147,8 +147,8 @@
             </plugin>
         </gazebo>
-        <gazebo reference="left_gripper">
-            <material>Gazebo/Black</material>
-        </gazebo>
-        <gazebo reference="right_gripper">
+        <gazebo reference="left_gripper_palm">
+            <material>Gazebo/Black</material>
+        </gazebo>
+        <gazebo reference="right_gripper_palm">
             <material>Gazebo/Black</material>
         </gazebo>
