Commit message: begin grasping test

File: src/bulldog/bulldog_description/urdf/bulldog/bulldog.urdf.xacro (robot description, xacro)
@@ -6,5 +6,5 @@
   <xacro:include filename="$(find ur_description)/urdf/ur5.urdf.xacro" />
   <xacro:include filename="$(find lms1xx)/urdf/sick_lms1xx.urdf.xacro" />
-  <xacro:include filename="$(find robotiq_3f_gripper_visualization)/cfg/robotiq-3f-gripper_articulated_macro.xacro" />
+  <xacro:include filename="$(find robotiq_3f_gripper_visualization)/cfg/robotiq_hand_macro.urdf.xacro" />
   <xacro:include filename="$(find bulldog_description)/urdf/sensors/kinect_camera.urdf.xacro" />
   <xacro:include filename="$(find realsense2_description)/urdf/_d415.urdf.xacro" />
@@ -87,16 +87,10 @@
       <!-- If you modify the name of the grippers, remember to change the *prefix* in line
            780 and 782 accordingly of $(find robotiq_s_model_articulated_gazebo_plugins)/src/RobotiqHandPlugin.cpp. -->
-        <xacro:robotiq-3f-gripper_articulated prefix="left_gripper_"/>
-        <joint name="left_arm_gripper_joint" type="fixed">
-            <parent link="left_arm_ee_link" />
-            <child link="left_gripper_palm" />
-            <origin xyz="0 0 0" rpy="0 0 -1.57" />
-        </joint>
-        <xacro:robotiq-3f-gripper_articulated prefix="right_gripper_"/>
-        <joint name="right_arm_gripper_joint" type="fixed">
-            <parent link="right_arm_ee_link" />
-            <child link="right_gripper_palm" />
-            <origin xyz="0 0 0" rpy="0 0 -1.57" />
-        </joint>
+      <xacro:robotiq_hand prefix="left_gripper_" parent="left_arm_ee_link" reflect="-1">
+        <origin rpy="0 0 -1.57" xyz="0 0 0"/>
+      </xacro:robotiq_hand>
+      <xacro:robotiq_hand prefix="right_gripper_" parent="right_arm_ee_link" reflect="-1">
+        <origin rpy="0 0 -1.57" xyz="0 0 0"/>
+      </xacro:robotiq_hand>
     </xacro:if>
     <!-- laser -->

File: src/robotiq/robotiq_3f_gripper_visualization/cfg/robotiq_hand_macro.urdf.xacro (robot description, xacro)
@@ -259,10 +259,10 @@
         </geometry>
       </visual>
-      <collision>
+      <!-- <collision>
         <origin rpy="0 0 0" xyz="0 0 0"/>
          <geometry>
           <box size=".02 .02 .002"/>
         </geometry>
-      </collision>
+      </collision> -->
       <inertial>
         <origin rpy="0 0 0" xyz="0.0092 0.00514 0"/>
@@ -317,10 +317,10 @@
         </geometry>
       </visual>
-      <collision>
+      <!-- <collision>
         <origin rpy="0 0 0" xyz="0 0 0"/>
          <geometry>
           <box size=".02 .02 .002"/>
         </geometry>
-      </collision>
+      </collision> -->
       <inertial>
         <origin rpy="0 0 0" xyz="-0.01025 0.00046 0"/>
@@ -375,10 +375,10 @@
         </geometry>
       </visual>
-      <collision>
+      <!--  <collision>
         <origin rpy="0 0 0" xyz="0 0 0"/>
          <geometry>
           <box size=".02 0.02 .002"/>
         </geometry>
-      </collision>
+      </collision> -->
       <inertial>
         <origin rpy="0 0 0" xyz="0.00548 0 0"/>

Commit message: fine tune robotiq 3 finger gripper orientation in URDF

File: src/bulldog/bulldog_description/urdf/bulldog/bulldog.urdf.xacro (robot description, xacro)
@@ -73,5 +73,6 @@
     <!-- dual ur5 arms -->
     <xacro:if value="$(arg dual_ur5_enabled)">
-      <xacro:ur5_robot prefix="left_arm_" joint_limited="true"/>
+      <xacro:ur5_robot prefix="left_arm_" joint_limited="true"
+        transmission_hw_interface="hardware_interface/PositionJointInterface" />
       <joint name="left_arm_base" type="fixed">
         <parent link="installation_plate_link" />
@@ -79,5 +80,6 @@
         <origin xyz="0 0.15945 0.09069" rpy="-0.785 0 0" />
       </joint>
-      <xacro:ur5_robot prefix="right_arm_" joint_limited="true"/>
+      <xacro:ur5_robot prefix="right_arm_" joint_limited="true"
+        transmission_hw_interface="hardware_interface/PositionJointInterface" />
       <joint name="right_arm_base" type="fixed">
         <parent link="installation_plate_link" />
@@ -88,8 +90,8 @@
            780 and 782 accordingly of $(find robotiq_s_model_articulated_gazebo_plugins)/src/RobotiqHandPlugin.cpp. -->
       <xacro:robotiq_hand prefix="left_gripper_" parent="left_arm_ee_link" reflect="-1">
-        <origin rpy="0 0 -1.57" xyz="0 0 0"/>
+        <origin rpy="0 -2.3562 -1.5708" xyz="0 0 0"/>
       </xacro:robotiq_hand>
       <xacro:robotiq_hand prefix="right_gripper_" parent="right_arm_ee_link" reflect="-1">
-        <origin rpy="0 0 -1.57" xyz="0 0 0"/>
+        <origin rpy="0 -2.3562 -1.5708" xyz="0 0 0"/>
       </xacro:robotiq_hand>
     </xacro:if>

File: src/bulldog/bulldog_description/urdf/bulldog/bulldog_gazebo.urdf.xacro (robot description, xacro)
@@ -73,5 +73,6 @@
     <!-- dual ur5 arms -->
     <xacro:if value="$(arg dual_ur5_enabled)">
-        <xacro:ur5_robot prefix="left_arm_" joint_limited="true"/>
+        <xacro:ur5_robot prefix="left_arm_" joint_limited="true"
+          transmission_hw_interface="hardware_interface/PositionJointInterface" />
         <joint name="left_arm_base" type="fixed">
         <parent link="installation_plate_link" />
@@ -79,5 +80,6 @@
         <origin xyz="0 0.15945 0.09069" rpy="-0.785 0 0" />
         </joint>
-        <xacro:ur5_robot prefix="right_arm_" joint_limited="true"/>
+        <xacro:ur5_robot prefix="right_arm_" joint_limited="true"
+          transmission_hw_interface="hardware_interface/PositionJointInterface" />
         <joint name="right_arm_base" type="fixed">
         <parent link="installation_plate_link" />

Commit message: fine tune right robotiq gripper URDF

File: src/bulldog/bulldog_description/urdf/bulldog/bulldog.urdf.xacro (robot description, xacro)
@@ -93,5 +93,5 @@
       </xacro:robotiq_hand>
       <xacro:robotiq_hand prefix="right_gripper_" parent="right_arm_ee_link" reflect="-1">
-        <origin rpy="0 -2.3562 -1.5708" xyz="0 0 0"/>
+        <origin rpy="0 2.3562 -1.5708" xyz="0 0 0"/>
       </xacro:robotiq_hand>
     </xacro:if>

Commit message: debugging wheel drivers

File: src/bulldog/bulldog_description/urdf/bulldog/bulldog.urdf.xacro (robot description, xacro)
@@ -8,5 +8,5 @@
   <xacro:include filename="$(find robotiq_3f_gripper_visualization)/cfg/robotiq_hand_macro.urdf.xacro" />
   <xacro:include filename="$(find bulldog_description)/urdf/sensors/kinect_camera.urdf.xacro" />
-  <xacro:include filename="$(find realsense2_description)/urdf/_d415.urdf.xacro" />
+  <xacro:include filename="$(find realsense2_camera)/urdf/_d415.urdf.xacro" />
   <xacro:property name="wheel_length" value="0.142" />
   <xacro:property name="wheel_radius" value="0.183" />
@@ -88,8 +88,8 @@
            780 and 782 accordingly of $(find robotiq_s_model_articulated_gazebo_plugins)/src/RobotiqHandPlugin.cpp. -->
       <xacro:robotiq_hand prefix="left_gripper_" parent="left_arm_ee_link" reflect="-1">
-        <origin rpy="0 0 -1.57" xyz="0 0 0"/>
+        <origin rpy="0 -2.3562 -1.5708" xyz="0 0 0"/>
       </xacro:robotiq_hand>
       <xacro:robotiq_hand prefix="right_gripper_" parent="right_arm_ee_link" reflect="-1">
-        <origin rpy="0 0 -1.57" xyz="0 0 0"/>
+        <origin rpy="0 -2.3562 -1.5708" xyz="0 0 0"/>
       </xacro:robotiq_hand>
     </xacro:if>

Commit message: update bulldog_description

File: src/bulldog/bulldog_description/urdf/bulldog/bulldog.urdf.xacro (robot description, xacro)
@@ -73,5 +73,6 @@
     <!-- dual ur5 arms -->
     <xacro:if value="$(arg dual_ur5_enabled)">
-      <xacro:ur5_robot prefix="left_arm_" joint_limited="true"/>
+      <xacro:ur5_robot prefix="left_arm_" joint_limited="true"
+        transmission_hw_interface="hardware_interface/PositionJointInterface" />
       <joint name="left_arm_base" type="fixed">
         <parent link="installation_plate_link" />
@@ -79,5 +80,6 @@
         <origin xyz="0 0.15945 0.09069" rpy="-0.785 0 0" />
       </joint>
-      <xacro:ur5_robot prefix="right_arm_" joint_limited="true"/>
+      <xacro:ur5_robot prefix="right_arm_" joint_limited="true"
+        transmission_hw_interface="hardware_interface/PositionJointInterface" />
       <joint name="right_arm_base" type="fixed">
         <parent link="installation_plate_link" />
@@ -88,8 +90,8 @@
            780 and 782 accordingly of $(find robotiq_s_model_articulated_gazebo_plugins)/src/RobotiqHandPlugin.cpp. -->
       <xacro:robotiq_hand prefix="left_gripper_" parent="left_arm_ee_link" reflect="-1">
-        <origin rpy="0 0 -1.57" xyz="0 0 0"/>
+        <origin rpy="0 -2.3562 -1.5708" xyz="0 0 0"/>
       </xacro:robotiq_hand>
       <xacro:robotiq_hand prefix="right_gripper_" parent="right_arm_ee_link" reflect="-1">
-        <origin rpy="0 0 -1.57" xyz="0 0 0"/>
+        <origin rpy="0 2.3562 -1.5708" xyz="0 0 0"/>
       </xacro:robotiq_hand>
     </xacro:if>

File: src/bulldog/bulldog_description/urdf/bulldog/bulldog_gazebo.urdf.xacro (robot description, xacro)
@@ -73,5 +73,6 @@
     <!-- dual ur5 arms -->
     <xacro:if value="$(arg dual_ur5_enabled)">
-        <xacro:ur5_robot prefix="left_arm_" joint_limited="true"/>
+        <xacro:ur5_robot prefix="left_arm_" joint_limited="true"
+          transmission_hw_interface="hardware_interface/PositionJointInterface" />
         <joint name="left_arm_base" type="fixed">
         <parent link="installation_plate_link" />
@@ -79,5 +80,6 @@
         <origin xyz="0 0.15945 0.09069" rpy="-0.785 0 0" />
         </joint>
-        <xacro:ur5_robot prefix="right_arm_" joint_limited="true"/>
+        <xacro:ur5_robot prefix="right_arm_" joint_limited="true"
+          transmission_hw_interface="hardware_interface/PositionJointInterface" />
         <joint name="right_arm_base" type="fixed">
         <parent link="installation_plate_link" />
@@ -91,5 +93,5 @@
             <parent link="left_arm_ee_link" />
             <child link="left_gripper_palm" />
-            <origin xyz="0 0 0" rpy="0 0 -1.57" />
+            <origin xyz="0 0 0" rpy="0 -2.3562 -1.57" />
         </joint>
         <xacro:robotiq-3f-gripper_articulated prefix="right_gripper_"/>
@@ -97,5 +99,5 @@
             <parent link="right_arm_ee_link" />
             <child link="right_gripper_palm" />
-            <origin xyz="0 0 0" rpy="0 0 -1.57" />
+            <origin xyz="0 0 0" rpy="0 2.3562 -1.57" />
         </joint>
     </xacro:if>

Commit message: realsense d435 white material

File: src/bulldog/bulldog_description/urdf/bulldog/bulldog.urdf.xacro (robot description, xacro)
@@ -111,5 +111,5 @@
       <xacro:kinect_camera prefix="kinect" parent="installation_plate_link" />
     </xacro:if>
-    <!-- realsense d415 -->
+    <!-- realsense d435 -->
     <xacro:if value="$(arg realsense_enabled)">
       <xacro:realsense_support prefix="left_gripper_sensor_support_"
@@ -117,5 +117,5 @@
         <origin xyz="0 -0.050 0" rpy="${pi / 2} 0 ${pi}" />
       </xacro:realsense_support>
-      <xacro:sensor_d435 prefix="left_gripper_sensor_d415_"
+      <xacro:sensor_d435 prefix="left_gripper_sensor_d435_"
         parent="left_gripper_sensor_support_mounted_link">
         <origin xyz="0 0 0" rpy="0 0 0"/>
@@ -125,5 +125,5 @@
         <origin xyz="0 -0.050 0" rpy="${-pi / 2} 0 0" />
       </xacro:realsense_support>
-      <xacro:sensor_d435 prefix="right_gripper_sensor_d415_"
+      <xacro:sensor_d435 prefix="right_gripper_sensor_d435_"
         parent="right_gripper_sensor_support_mounted_link">
         <origin xyz="0 0 0" rpy="0 0 0"/>

File: src/bulldog_simulator/bulldog_gazebo/urdf/accessories/realsense_camera.gazebo.xacro (robot description, xacro)
@@ -1,8 +1,8 @@
 <?xml version="1.0"?>
 <root xmlns:xacro="http://ros.org/wiki/xacro">
-  <xacro:macro name="sensor_d415_gazebo" params="prefix">
+  <xacro:macro name="sensor_d435_gazebo" params="prefix">
     <!-- material -->
     <gazebo reference="${prefix}camera_link">
-      <material>Gazebo/Grey</material>
+      <material>Gazebo/White</material>
     </gazebo>
     <!-- color sensor -->

File: src/bulldog_simulator/bulldog_gazebo/urdf/bulldog.gazebo.xacro (robot description, xacro)
@@ -23,5 +23,5 @@
 <robot name="bulldog_robot" xmlns:xacro="http://ros.org/wiki/xacro">
   <xacro:include filename="$(find bulldog_gazebo)/urdf/accessories/kinect_camera.gazebo.xacro"/>
-  <xacro:include filename="$(find bulldog_gazebo)/urdf/accessories/realsense_d415_camera.gazebo.xacro"/>
+  <xacro:include filename="$(find bulldog_gazebo)/urdf/accessories/realsense_camera.gazebo.xacro"/>
   <xacro:macro name="bulldog_gazebo_config">
     <!-- ROS control -->
@@ -236,6 +236,6 @@
     <!-- realsense -->
     <xacro:if value="$(arg realsense_enabled)">
-      <xacro:sensor_d415_gazebo prefix="left_gripper_sensor_d415_"/>
-      <xacro:sensor_d415_gazebo prefix="right_gripper_sensor_d415_"/>
+      <xacro:sensor_d435_gazebo prefix="left_gripper_sensor_d435_"/>
+      <xacro:sensor_d435_gazebo prefix="right_gripper_sensor_d435_"/>
     </xacro:if>
   </xacro:macro>
