Commit message: revert to d415

File: src/bulldog/bulldog_description/urdf/accessories/realsense_support.urdf.xacro (robot description, xacro)
@@ -29,5 +29,5 @@
     </link>
     <joint name="${prefix}mounted_joint" type="fixed">
-        <origin xyz="0 0.0785 0.00875" rpy="0 ${-pi / 2} ${-pi / 2}" />
+        <origin xyz="0 0.0795 0.00875" rpy="0 ${-pi / 2} ${-pi / 2}" />
         <parent link="${prefix}support_link" />
         <child link="${prefix}mounted_link" />

File: src/bulldog/bulldog_description/urdf/bulldog/bulldog.urdf.xacro (robot description, xacro)
@@ -9,5 +9,5 @@
   <xacro:include filename="$(find robotiq_3f_gripper_visualization)/cfg/robotiq_hand_macro.urdf.xacro" />
   <xacro:include filename="$(find bulldog_description)/urdf/sensors/kinect_camera.urdf.xacro" />
-  <xacro:include filename="$(find realsense2_description)/urdf/_d435.urdf.xacro" />
+  <xacro:include filename="$(find realsense2_description)/urdf/_d415.urdf.xacro" />
   <xacro:property name="wheel_length" value="0.142" />
   <xacro:property name="wheel_radius" value="0.183" />
@@ -111,5 +111,5 @@
       <xacro:kinect_camera prefix="kinect" parent="installation_plate_link" />
     </xacro:if>
-    <!-- realsense d435 -->
+    <!-- realsense d415 -->
     <xacro:if value="$(arg realsense_enabled)">
       <xacro:realsense_support prefix="left_gripper_sensor_support_"
@@ -117,16 +117,16 @@
         <origin xyz="0 -0.050 0" rpy="${pi / 2} 0 ${pi}" />
       </xacro:realsense_support>
-      <xacro:sensor_d435 prefix="left_gripper_sensor_d435_"
+      <xacro:sensor_d415 prefix="left_gripper_sensor_d415_"
         parent="left_gripper_sensor_support_mounted_link">
         <origin xyz="0 0 0" rpy="0 0 0"/>
-      </xacro:sensor_d435>
+      </xacro:sensor_d415>
       <xacro:realsense_support prefix="right_gripper_sensor_support_"
         installation_link="right_gripper_palm">
         <origin xyz="0 -0.050 0" rpy="${-pi / 2} 0 0" />
       </xacro:realsense_support>
-      <xacro:sensor_d435 prefix="right_gripper_sensor_d435_"
+      <xacro:sensor_d415 prefix="right_gripper_sensor_d415_"
         parent="right_gripper_sensor_support_mounted_link">
         <origin xyz="0 0 0" rpy="0 0 0"/>
-      </xacro:sensor_d435>
+      </xacro:sensor_d415>
     </xacro:if>
   </xacro:macro>

File: src/bulldog_simulator/bulldog_gazebo/urdf/accessories/realsense_camera.gazebo.xacro (robot description, xacro)
@@ -1,5 +1,5 @@
 <?xml version="1.0"?>
 <root xmlns:xacro="http://ros.org/wiki/xacro">
-  <xacro:macro name="sensor_d435_gazebo" params="prefix">
+  <xacro:macro name="sensor_d415_gazebo" params="prefix">
     <!-- material -->
     <gazebo reference="${prefix}camera_link">

File: src/bulldog_simulator/bulldog_gazebo/urdf/bulldog.gazebo.xacro (robot description, xacro)
@@ -236,6 +236,6 @@
     <!-- realsense -->
     <xacro:if value="$(arg realsense_enabled)">
-      <xacro:sensor_d435_gazebo prefix="left_gripper_sensor_d435_"/>
-      <xacro:sensor_d435_gazebo prefix="right_gripper_sensor_d435_"/>
+      <xacro:sensor_d415_gazebo prefix="left_gripper_sensor_d415_"/>
+      <xacro:sensor_d415_gazebo prefix="right_gripper_sensor_d415_"/>
     </xacro:if>
   </xacro:macro>
