Commit message: modify bulldog urdf

File: src/bulldog/bulldog_description/urdf/accessories/plates.urdf.xacro (robot description, xacro)
@@ -36,5 +36,5 @@
       <parent link="installation_plate_link"/>
       <child link="laser_plate_link"/>
-      <origin xyz="0.3 0 -0.1" rpy="${M_PI} 0 0" />
+      <origin xyz="0.3 0 -0.1" rpy="${pi} 0 0" />
     </joint>
   </xacro:macro>

File: src/bulldog/bulldog_description/urdf/bulldog/bulldog.urdf.xacro (robot description, xacro)
@@ -6,140 +6,127 @@
   <xacro:include filename="$(find lms1xx)/urdf/sick_lms1xx.urdf.xacro" />
   <xacro:include filename="$(find robotiq_s_model_visualization)/cfg/robotiq_hand_macro.urdf.xacro" />
-  <!--xacro:include filename="$(find bulldog_description)/urdf/sensors/kinect_camera.urdf.xacro" /-->
+  <xacro:include filename="$(find bulldog_description)/urdf/sensors/kinect_camera.urdf.xacro" />
   <!--xacro:include filename="$(find bulldog_description)/urdf/accessories/yuntai.urdf.xacro" /-->
-  <property name="M_PI" value="3.141592654"/>
   <xacro:property name="wheel_length" value="0.142" />
   <xacro:property name="wheel_radius" value="0.183" />
-  <property name="base_x_size" value="0.85" />
-  <property name="base_y_size" value="0.42" />
-  <property name="base_z_size" value="0.325" />
+  <xacro:property name="base_x_size" value="0.85" />
+  <xacro:property name="base_y_size" value="0.42" />
+  <xacro:property name="base_z_size" value="0.325" />
   <xacro:macro name="bulldog_robot">
-  <link name="base_link">
-    <visual>
+    <!-- base -->
+    <link name="base_link">
+      <visual>
+        <origin xyz="0 0 0" rpy="0 0 0" />
+        <geometry>
+          <mesh filename="package://bulldog_description/meshes/base_link.stl" />
+        </geometry>
+        <material name="flat_black" />
+      </visual>
+      <collision>
+        <origin xyz="0 0 ${base_z_size/2.0}" rpy="0 0 0" />
+        <geometry>
+          <box size="${base_x_size} ${base_y_size} ${base_z_size}"/>
+        </geometry>
+      </collision>
+    </link>
+    <gazebo reference="base_link">
+      <material>Gazebo/FlatBlack</material>
+    </gazebo>
+    <!-- inertial -->
+    <link name="inertial_link">
+      <inertial>
+        <mass value="40" />
+        <origin xyz="0 0 0.1" />
+        <inertia ixx="0.7" ixy="-0.03" ixz="-0.15" iyy="2" iyz="-0.01" izz="4" />
+      </inertial>
+    </link>
+    <joint name="inertial_joint" type="fixed">
       <origin xyz="0 0 0" rpy="0 0 0" />
-      <geometry>
-        <mesh filename="package://bulldog_description/meshes/base_link.stl" />
-      </geometry>
-      <material name="flat_black" />
-    </visual>
-    <collision>
-      <origin xyz="0 0 ${base_z_size/2.0}" rpy="0 0 0" />
-      <geometry>
-        <box size="${base_x_size} ${base_y_size} ${base_z_size}"/>
-      </geometry>
-    </collision>
-  </link>
-  <gazebo reference="base_link">
-    <material>Gazebo/FlatBlack</material>
-  </gazebo>
-  <link name="inertial_link">
-    <inertial>
-      <mass value="40" />
-      <origin xyz="0 0 0.1" />
-      <inertia ixx="0.7" ixy="-0.03" ixz="-0.15" iyy="2" iyz="-0.01" izz="4" />
-    </inertial>
-  </link>
-  <joint name="inertial_joint" type="fixed">
-    <origin xyz="0 0 0" rpy="0 0 0" />
-    <parent link="base_link" />
-    <child link="inertial_link" />
-  </joint>
-  <link name="top_plate_link">
-    <visual>
+      <parent link="base_link" />
+      <child link="inertial_link" />
+    </joint>
+    <!-- top plate -->
+    <link name="top_plate_link">
+      <visual>
+        <origin xyz="0 0 0" rpy="0 0 0" />
+        <geometry>
+          <mesh filename="package://bulldog_description/meshes/top_plate.stl" />
+        </geometry>
+        <material name="grey" />
+      </visual>
+    </link>
+    <gazebo reference="top_plate_link">
+      <material>Gazebo/Grey</material>
+    </gazebo>
+    <joint name="top_plate_joint" type="fixed">
+      <origin xyz="0.07937 0 0.253" rpy="0 0 0" />
+      <parent link="base_link" />
+      <child link="top_plate_link" />
+    </joint>
+    <!-- imu -->
+    <link name="imu_link"/>
+    <joint name="imu_joint" type="fixed">
       <origin xyz="0 0 0" rpy="0 0 0" />
-      <geometry>
-        <mesh filename="package://bulldog_description/meshes/top_plate.stl" />
-      </geometry>
-      <material name="grey" />
-    </visual>
-  </link>
-  <gazebo reference="top_plate_link">
-    <material>Gazebo/Grey</material>
-  </gazebo>
-  <joint name="top_plate_joint" type="fixed">
-    <origin xyz="0.07937 0 0.253" rpy="0 0 0" />
-    <parent link="base_link" />
-    <child link="top_plate_link" />
-  </joint>
-  <link name="imu_link"/>
-  <joint name="imu_joint" type="fixed">
-    <origin xyz="0 0 0" rpy="0 0 0" />
-    <parent link="base_link" />
-    <child link="imu_link" />
-  </joint>
-  <gazebo reference="imu_link" />
-  <xacro:bulldog_wheel wheel_prefix="front_left">
-    <origin xyz="0.27937 0.285 0.0435" rpy="0 0 0" />
-  </xacro:bulldog_wheel>
-  <xacro:bulldog_wheel wheel_prefix="front_right">
-    <origin xyz="0.27937 -0.285 0.0435" rpy="0 0 0" />
-  </xacro:bulldog_wheel>
-  <xacro:bulldog_wheel wheel_prefix="rear_left">
-    <origin xyz="-0.27937 0.285 0.0435" rpy="0 0 0" />
-  </xacro:bulldog_wheel>
-  <xacro:bulldog_wheel wheel_prefix="rear_right">
-    <origin xyz="-0.27937 -0.285 0.0435" rpy="0 0 0" />
-  </xacro:bulldog_wheel>
-  <!--xacro:if value="$(optenv BULLDOG_DUAL_UR5_ENABLED true)"-->
-    <!--xacro:installation_plate /-->
-    <xacro:ur5_robot prefix="left_arm_" joint_limited="true"/>
-    <joint name="left_arm_base" type="fixed">
-      <parent link="installation_plate_link" />
-      <child link="left_arm_base_link" />
-      <origin xyz="0 0.15945 0.09069" rpy="-0.785 0 0" />
+      <parent link="base_link" />
+      <child link="imu_link" />
     </joint>
-    <xacro:ur5_robot prefix="right_arm_" joint_limited="true"/>
-    <joint name="right_arm_base" type="fixed">
-      <parent link="installation_plate_link" />
-      <child link="right_arm_base_link" />
-      <origin xyz="0 -0.15945 0.09069" rpy="-0.785 0 ${M_PI}" />
-    </joint>
-  <xacro:robotiq_hand prefix="l_" parent="left_arm_ee_link" reflect="-1">
-    <origin rpy="0 0 -1.57" xyz="0 0 0"/>
-  </xacro:robotiq_hand>
-  <xacro:robotiq_hand prefix="r_" parent="right_arm_ee_link" reflect="-1">
-    <origin rpy="0 0 -1.57" xyz="0 0 0"/>
-  </xacro:robotiq_hand>
-  <xacro:if value="$(arg laser_enabled)">
+    <gazebo reference="imu_link" />
+    <xacro:bulldog_wheel wheel_prefix="front_left">
+      <origin xyz="0.27937 0.285 0.0435" rpy="0 0 0" />
+    </xacro:bulldog_wheel>
+    <xacro:bulldog_wheel wheel_prefix="front_right">
+      <origin xyz="0.27937 -0.285 0.0435" rpy="0 0 0" />
+    </xacro:bulldog_wheel>
+    <xacro:bulldog_wheel wheel_prefix="rear_left">
+      <origin xyz="-0.27937 0.285 0.0435" rpy="0 0 0" />
+    </xacro:bulldog_wheel>
+    <xacro:bulldog_wheel wheel_prefix="rear_right">
+      <origin xyz="-0.27937 -0.285 0.0435" rpy="0 0 0" />
+    </xacro:bulldog_wheel>
+    <!-- installation plate -->
     <xacro:installation_plate />
-    <xacro:laser_plate />
-    <sick_lms1xx frame="laser" topic="scan"/>
-    <joint name="laser_mount_joint" type="fixed">
-      <origin xyz="0.015 0 0.044" rpy="${M_PI} 0 0" />
-      <parent link="laser_plate_link" />
-      <child link="laser" />
-    </joint>
-  </xacro:if>
-    <link name="camera_link">
-    <visual>
-      <origin xyz="0 0 0" rpy="0 0 0" />
-      <geometry>
-        <box size="0.065 0.25 0.065"/>
-      </geometry>
-      <mesh filename="package://bulldog_description/meshes/kinect.dae" />
-    </visual>
-    <collision>
-      <origin xyz="0 0 0" rpy="0 0 0" />
-      <geometry>
-        <!--box size="0.065 0.25 0.065"/-->
-        <box size = "0 0 0"/>
-      </geometry>
-    </collision>
-    </link>
-  <gazebo reference="camera_link">
-    <material>Gazebo/Black</material>
-  </gazebo>
-    <joint name="kinect_frame_joint" type="fixed">
+    <!-- dual ur5 arms -->
+    <xacro:if value="$(arg dual_ur5_enabled)">
+      <xacro:ur5_robot prefix="left_arm_" joint_limited="true"/>
+      <joint name="left_arm_base" type="fixed">
+        <parent link="installation_plate_link" />
+        <child link="left_arm_base_link" />
+        <origin xyz="0 0.15945 0.09069" rpy="-0.785 0 0" />
+      </joint>
+      <xacro:ur5_robot prefix="right_arm_" joint_limited="true"/>
+      <joint name="right_arm_base" type="fixed">
+        <parent link="installation_plate_link" />
+        <child link="right_arm_base_link" />
+        <origin xyz="0 -0.15945 0.09069" rpy="-0.785 0 ${pi}" />
+      </joint>
+      <xacro:robotiq_hand prefix="l_" parent="left_arm_ee_link" reflect="-1">
+        <origin rpy="0 0 -1.57" xyz="0 0 0"/>
+      </xacro:robotiq_hand>
+      <xacro:robotiq_hand prefix="r_" parent="right_arm_ee_link" reflect="-1">
+        <origin rpy="0 0 -1.57" xyz="0 0 0"/>
+      </xacro:robotiq_hand>
+    </xacro:if>
+    <!-- laser -->
+    <xacro:if value="$(arg laser_enabled)">
+      <xacro:laser_plate />
+      <sick_lms1xx frame="laser" topic="scan"/>
+      <joint name="laser_mount_joint" type="fixed">
+        <origin xyz="0.015 0 0.044" rpy="${pi} 0 0" />
+        <parent link="laser_plate_link" />
+        <child link="laser" />
+      </joint>
+    </xacro:if>
+    <!-- kinect -->
+    <xacro:if value="$(arg kinect_enabled)">
+      <xacro:kinect_camera prefix="camera" />
+      <gazebo reference="camera_link">
+        <material>Gazebo/Black</material>
+      </gazebo>
+      <joint name="kinect_frame_joint" type="fixed">
         <origin xyz="0.13 0 0.135" rpy=" 0 0.15 0" />
-      <parent link="installation_plate_link"/>
-      <child link="camera_link"/>
-    </joint>
-    <xacro:kinect_camera prefix="camera"/>
-  <!--joint name="yuntai_installation_plate_joint" type="fixed">
-    <origin xyz="0.05 0 0.135 " rpy="0 ${M_PI/2} 0" />
-    <parent link="installation_plate_link"/>
-    <child link="yuntai_base_link" />
-  </joint>
-  <xacro:yuntai_robot /-->
+        <parent link="installation_plate_link"/>
+        <child link="camera_link"/>
+      </joint>
+    </xacro:if>
   </xacro:macro>
 </robot>

File: src/bulldog/bulldog_description/urdf/bulldog/wheel.urdf.xacro (robot description, xacro)
@@ -16,5 +16,5 @@
     </visual>
     <collision>
-      <origin xyz="0 0 0" rpy="${M_PI/2} 0 0" />
+      <origin xyz="0 0 0" rpy="${pi / 2} 0 0" />
       <geometry>
         <cylinder length="${wheel_length}" radius="${wheel_radius}" />

File: src/bulldog/bulldog_description/urdf/sensors/kinect_camera.urdf.xacro (robot description, xacro)
@@ -29,8 +29,9 @@
     <!-- Create kinect reference frame -->
     <!-- Add mesh for kinect -->
-    <!--link name="${prefix}_link">
+    <link name="${prefix}_link">
       <origin xyz="0 0 0" rpy="0 0 0"/>
       <visual>
-        <origin xyz="0 0 0" rpy="0 0 ${M_PI/2}"/>
+        <origin xyz="0 0 0" rpy="0 0 ${pi / 2}"/>
+        <!-- <origin xyz="0 0 0" rpy="0 0 0"/> -->
         <geometry>
           <mesh filename="package://bulldog_description/meshes/kinect.dae" />
@@ -42,6 +43,6 @@
         </geometry>
       </collision>
-    </link-->
-    <link name="camera_link">
+    </link>
+    <!-- <link name="camera_link">
     <visual>
       <origin xyz="0 0 0" rpy="0 0 0" />
@@ -57,5 +58,5 @@
       </geometry>
     </collision>
-    </link>
+    </link> -->
   </xacro:macro>
 </robot>

File: src/bulldog_simulator/bulldog_gazebo/urdf/accessories/kinect_camera.gazebo.xacro (robot description, xacro)
@@ -1,47 +1,47 @@
 <?xml version="1.0"?>
 <root xmlns:xacro="http://ros.org/wiki/xacro">
-<xacro:macro name="kinect_camera_gazebo" params="prefix">
-  <joint name="${prefix}_optical_joint" type="fixed">
-    <origin xyz="0 0 0" rpy="-1.5708 0 -1.5708"/>
-    <parent link="${prefix}_link"/>
-    <child link="${prefix}_frame_optical"/>
-  </joint>
-  <link name="${prefix}_frame_optical"/>
-  <gazebo reference="${prefix}_link">
-    <sensor type="depth" name="${prefix}">
-      <always_on>true</always_on>
-      <update_rate>20.0</update_rate>
-      <camera>
-        <horizontal_fov>${60.0*M_PI/180.0}</horizontal_fov>
-        <image>
-          <format>R8G8B8</format>
-          <width>640</width>
-          <height>480</height>
-        </image>
-        <clip>
-          <near>0.05</near>
-          <far>8.0</far>
-        </clip>
-      </camera>
-      <plugin name="kinect_${prefix}_controller" filename="libgazebo_ros_openni_kinect.so">
-        <cameraName>${prefix}</cameraName>
-        <alwaysOn>true</alwaysOn>
-        <updateRate>10</updateRate>
-        <imageTopicName>rgb/image_raw</imageTopicName>
-        <depthImageTopicName>depth/image_raw</depthImageTopicName>
-        <pointCloudTopicName>depth/points</pointCloudTopicName>
-        <cameraInfoTopicName>rgb/camera_info</cameraInfoTopicName>
-        <depthImageCameraInfoTopicName>depth/camera_info</depthImageCameraInfoTopicName>
-        <frameName>${prefix}_frame_optical</frameName>
-        <baseline>0.1</baseline>
-        <distortion_k1>0.0</distortion_k1>
-        <distortion_k2>0.0</distortion_k2>
-        <distortion_k3>0.0</distortion_k3>
-        <distortion_t1>0.0</distortion_t1>
-        <distortion_t2>0.0</distortion_t2>
-        <pointCloudCutoff>0.4</pointCloudCutoff>
-      </plugin>
-    </sensor>
-  </gazebo>
-</xacro:macro>
+  <xacro:macro name="kinect_camera_gazebo" params="prefix">
+    <joint name="${prefix}_optical_joint" type="fixed">
+      <origin xyz="0 0 0" rpy="-1.5708 0 -1.5708"/>
+      <parent link="${prefix}_link"/>
+      <child link="${prefix}_frame_optical"/>
+    </joint>
+    <link name="${prefix}_frame_optical"/>
+    <gazebo reference="${prefix}_link">
+      <sensor type="depth" name="${prefix}">
+        <always_on>true</always_on>
+        <update_rate>20.0</update_rate>
+        <camera>
+          <horizontal_fov>${60.0 * pi / 180.0}</horizontal_fov>
+          <image>
+            <format>R8G8B8</format>
+            <width>640</width>
+            <height>480</height>
+          </image>
+          <clip>
+            <near>0.05</near>
+            <far>8.0</far>
+          </clip>
+        </camera>
+        <plugin name="kinect_${prefix}_controller" filename="libgazebo_ros_openni_kinect.so">
+          <cameraName>${prefix}</cameraName>
+          <alwaysOn>true</alwaysOn>
+          <updateRate>10</updateRate>
+          <imageTopicName>rgb/image_raw</imageTopicName>
+          <depthImageTopicName>depth/image_raw</depthImageTopicName>
+          <pointCloudTopicName>depth/points</pointCloudTopicName>
+          <cameraInfoTopicName>rgb/camera_info</cameraInfoTopicName>
+          <depthImageCameraInfoTopicName>depth/camera_info</depthImageCameraInfoTopicName>
+          <frameName>${prefix}_frame_optical</frameName>
+          <baseline>0.1</baseline>
+          <distortion_k1>0.0</distortion_k1>
+          <distortion_k2>0.0</distortion_k2>
+          <distortion_k3>0.0</distortion_k3>
+          <distortion_t1>0.0</distortion_t1>
+          <distortion_t2>0.0</distortion_t2>
+          <pointCloudCutoff>0.4</pointCloudCutoff>
+        </plugin>
+      </sensor>
+    </gazebo>
+  </xacro:macro>
 </root>

File: src/bulldog_simulator/bulldog_gazebo/urdf/bulldog.gazebo.xacro (robot description, xacro)
@@ -24,4 +24,5 @@
   <xacro:include filename="$(find bulldog_gazebo)/urdf/accessories/kinect_camera.gazebo.xacro"/>
   <xacro:macro name="bulldog_robot_gazebo">
+    <!-- imu -->
     <gazebo>
       <plugin name="imu_controller" filename="libhector_gazebo_ros_imu.so">
@@ -34,4 +35,5 @@
       </plugin>
     </gazebo>
+    <!-- gps -->
     <gazebo>
       <plugin name="gps_controller" filename="libhector_gazebo_ros_gps.so">
@@ -49,33 +51,35 @@
       </plugin>
     </gazebo>
-      <!--Remove when https://github.com/ros-industrial/universal_robot/pull/168 is resolved -->
-      <gazebo reference="ur5_arm_shoulder_link">
-        <selfCollide>true</selfCollide>
-      </gazebo>
-      <gazebo reference="ur5_arm_upper_arm_link">
-        <selfCollide>true</selfCollide>
-      </gazebo>
-      <gazebo reference="ur5_arm_forearm_link">
-        <selfCollide>true</selfCollide>
-      </gazebo>
-      <gazebo reference="ur5_arm_wrist_1_link">
-        <selfCollide>true</selfCollide>
-      </gazebo>
-      <gazebo reference="ur5_arm_wrist_3_link">
-       <selfCollide>true</selfCollide>
-      </gazebo>
-      <gazebo reference="ur5_arm_wrist_2_link">
-        <selfCollide>true</selfCollide>
-      </gazebo>
-      <gazebo reference="ur5_arm_ee_link">
-        <selfCollide>true</selfCollide>
-      </gazebo>
+    <!-- ur5 arm -->
+    <!--Remove when https://github.com/ros-industrial/universal_robot/pull/168 is resolved -->
+    <gazebo reference="ur5_arm_shoulder_link">
+      <selfCollide>true</selfCollide>
+    </gazebo>
+    <gazebo reference="ur5_arm_upper_arm_link">
+      <selfCollide>true</selfCollide>
+    </gazebo>
+    <gazebo reference="ur5_arm_forearm_link">
+      <selfCollide>true</selfCollide>
+    </gazebo>
+    <gazebo reference="ur5_arm_wrist_1_link">
+      <selfCollide>true</selfCollide>
+    </gazebo>
+    <gazebo reference="ur5_arm_wrist_3_link">
+      <selfCollide>true</selfCollide>
+    </gazebo>
+    <gazebo reference="ur5_arm_wrist_2_link">
+      <selfCollide>true</selfCollide>
+    </gazebo>
+    <gazebo reference="ur5_arm_ee_link">
+      <selfCollide>true</selfCollide>
+    </gazebo>
+    <!-- robotiq grippers -->
     <xacro:if value="$(arg robotiq_grippers_enabled)">
         <gazebo>
-	    <plugin name="robotiq_left_hand_plugin" filename="libRobotiqHandPlugin.so">
-	      <side>left</side>
-	      <kp_position>5.0</kp_position>
-	      <kd_position>0.5</kd_position>
-	     </plugin>
+          <plugin name="robotiq_left_hand_plugin" filename="libRobotiqHandPlugin.so">
+            <side>left</side>
+            <kp_position>5.0</kp_position>
+            <kd_position>0.5</kd_position>
+          </plugin>
         </gazebo>
          <gazebo>
@@ -92,78 +96,81 @@
             <material>Gazebo/Black</material>
         </gazebo>
- <gazebo reference="l_finger_1_link_0">
+        <gazebo reference="l_finger_1_link_0">
             <material>Gazebo/Black</material>
         </gazebo>
-<gazebo reference="r_finger_1_link_0">
+        <gazebo reference="r_finger_1_link_0">
             <material>Gazebo/Black</material>
         </gazebo>
-<gazebo reference="l_finger_1_link_1">
+        <gazebo reference="l_finger_1_link_1">
             <material>Gazebo/Black</material>
         </gazebo>
-<gazebo reference="r_finger_1_link_1">
+        <gazebo reference="r_finger_1_link_1">
             <material>Gazebo/Black</material>
         </gazebo>
-<gazebo reference="l_finger_1_link_2">
+        <gazebo reference="l_finger_1_link_2">
             <material>Gazebo/Black</material>
         </gazebo>
-<gazebo reference="r_finger_1_link_2">
+        <gazebo reference="r_finger_1_link_2">
             <material>Gazebo/Black</material>
         </gazebo>
-<gazebo reference="l_finger_1_link_3">
+        <gazebo reference="l_finger_1_link_3">
             <material>Gazebo/Grey</material>
         </gazebo>
-<gazebo reference="r_finger_1_link_3">
+        <gazebo reference="r_finger_1_link_3">
             <material>Gazebo/Grey</material>
         </gazebo>
-<gazebo reference="l_finger_2_link_0">
+        <gazebo reference="l_finger_2_link_0">
             <material>Gazebo/Black</material>
         </gazebo>
-<gazebo reference="r_finger_2_link_0">
+        <gazebo reference="r_finger_2_link_0">
             <material>Gazebo/Black</material>
         </gazebo>
-<gazebo reference="l_finger_2_link_1">
+        <gazebo reference="l_finger_2_link_1">
             <material>Gazebo/Black</material>
         </gazebo>
-<gazebo reference="r_finger_2_link_1">
+        <gazebo reference="r_finger_2_link_1">
             <material>Gazebo/Black</material>
         </gazebo>
-<gazebo reference="l_finger_2_link_2">
+        <gazebo reference="l_finger_2_link_2">
             <material>Gazebo/Black</material>
         </gazebo>
-<gazebo reference="r_finger_2_link_2">
+        <gazebo reference="r_finger_2_link_2">
             <material>Gazebo/Black</material>
         </gazebo>
-<gazebo reference="l_finger_2_link_3">
+        <gazebo reference="l_finger_2_link_3">
             <material>Gazebo/Grey</material>
         </gazebo>
-<gazebo reference="r_finger_2_link_3">
+        <gazebo reference="r_finger_2_link_3">
             <material>Gazebo/Grey</material>
         </gazebo>
-<gazebo reference="l_finger_middle_link_0">
+        <gazebo reference="l_finger_middle_link_0">
             <material>Gazebo/Black</material>
         </gazebo>
-<gazebo reference="r_finger_middle_link_0">
+        <gazebo reference="r_finger_middle_link_0">
             <material>Gazebo/Black</material>
         </gazebo>
-<gazebo reference="l_finger_middle_link_1">
+        <gazebo reference="l_finger_middle_link_1">
             <material>Gazebo/Black</material>
         </gazebo>
-<gazebo reference="r_finger_middle_link_1">
+        <gazebo reference="r_finger_middle_link_1">
             <material>Gazebo/Black</material>
         </gazebo>
-<gazebo reference="l_finger_middle_link_2">
+        <gazebo reference="l_finger_middle_link_2">
             <material>Gazebo/Black</material>
         </gazebo>
-<gazebo reference="r_finger_middle_link_2">
+        <gazebo reference="r_finger_middle_link_2">
             <material>Gazebo/Black</material>
         </gazebo>
-<gazebo reference="l_finger_middle_link_3">
+        <gazebo reference="l_finger_middle_link_3">
             <material>Gazebo/Grey</material>
         </gazebo>
-<gazebo reference="r_finger_middle_link_3">
+        <gazebo reference="r_finger_middle_link_3">
             <material>Gazebo/Grey</material>
         </gazebo>
     </xacro:if>
+    <!-- kinect -->
+    <xacro:if value="$(arg kinect_enabled)">
       <xacro:kinect_camera_gazebo prefix="camera"/>
+    </xacro:if>
   </xacro:macro>
 </robot>
