Commit message: modify bulldog urdf

File: src/bulldog_simulator/bulldog_gazebo/urdf/description.gazebo.xacro (robot description, xacro)
@@ -25,6 +25,6 @@
   <xacro:arg name="ur5_enabled" default="false" />
   <xacro:arg name="kinect_enabled" default="true" />
-  <xacro:arg name="dual_ur5_enabled" default="false"/>
-  <xacro:arg name="robotiq_grippers_enabled" default="false"/>
+  <xacro:arg name="dual_ur5_enabled" default="true"/>
+  <xacro:arg name="robotiq_grippers_enabled" default="true"/>
   <xacro:include filename="$(find bulldog_description)/urdf/bulldog/bulldog.urdf.xacro" />
   <xacro:include filename="$(find bulldog_description)/urdf/accessories/plates.urdf.xacro" />
@@ -49,5 +49,5 @@
            <gripper_link> l_finger_2_link_2 </gripper_link>
            <gripper_link> l_finger_2_link_3 </gripper_link>
-            <gripper_link> l_finger_middle_link_0 </gripper_link>
+           <gripper_link> l_finger_middle_link_0 </gripper_link>
            <gripper_link> l_finger_middle_link_1 </gripper_link>
            <gripper_link> l_finger_middle_link_2 </gripper_link>
@@ -65,5 +65,5 @@
            <gripper_link> r_finger_2_link_2 </gripper_link>
            <gripper_link> r_finger_2_link_3 </gripper_link>
-            <gripper_link> r_finger_middle_link_0 </gripper_link>
+           <gripper_link> r_finger_middle_link_0 </gripper_link>
            <gripper_link> r_finger_middle_link_1 </gripper_link>
            <gripper_link> r_finger_middle_link_2 </gripper_link>

Commit message: remove redundant files

File: src/bulldog/bulldog_description/urdf/accessories/plates.urdf.xacro (robot description, xacro)
@@ -1,4 +1,23 @@
 <?xml version="1.0"?>
-<robot name="bulldog_plates" xmlns:xacro="http://ros.org/wiki/xacro">
+<robot name="bulldog_plates" xmlns:xacro="http://www.ros.org/wiki/xacro">
+  <xacro:macro name="top_plate">
+    <link name="top_plate_link">
+      <visual>
+        <origin xyz="0 0 0" rpy="0 0 0" />
+        <geometry>
+          <mesh filename="package://bulldog_description/meshes/top_plate.stl" />
+        </geometry>
+        <material name="grey" />
+      </visual>
+    </link>
+    <joint name="top_plate_joint" type="fixed">
+      <origin xyz="0.07937 0 0.253" rpy="0 0 0" />
+      <parent link="base_link" />
+      <child link="top_plate_link" />
+    </joint>
+    <gazebo reference="top_plate_link">
+      <material>Gazebo/Grey</material>
+    </gazebo>
+  </xacro:macro>
   <xacro:macro name="installation_plate">
     <link name="installation_plate_link">
@@ -11,7 +30,4 @@
       </visual>
     </link>
-    <gazebo reference="installation_plate_link">
-      <material>Gazebo/Black</material>
-    </gazebo>
     <joint name="installation_plate_joint" type="fixed">
       <parent link="base_link"/>
@@ -19,4 +35,7 @@
       <origin xyz="0.197 0 0.314" rpy="0 0 0" />
     </joint>
+    <gazebo reference="installation_plate_link">
+      <material>Gazebo/Black</material>
+    </gazebo>
   </xacro:macro>
   <xacro:macro name="laser_plate">
@@ -30,7 +49,4 @@
       </visual>
     </link>
-    <gazebo reference="laser_plate_link">
-      <material>Gazebo/FlatBlack</material>
-    </gazebo>
     <joint name="laser_plate_joint" type="fixed">
       <parent link="installation_plate_link"/>
@@ -38,4 +54,7 @@
       <origin xyz="0.3 0 -0.1" rpy="${pi} 0 0" />
     </joint>
+    <gazebo reference="laser_plate_link">
+      <material>Gazebo/FlatBlack</material>
+    </gazebo>
   </xacro:macro>
 </robot>

File: src/bulldog/bulldog_description/urdf/bulldog/bulldog.urdf.xacro (robot description, xacro)
@@ -1,11 +1,11 @@
 <?xml version="1.0"?>
 <robot name="bulldog_robot" xmlns:xacro="http://ros.org/wiki/xacro">
-  <xacro:include filename="$(find bulldog_description)/urdf/bulldog/wheel.urdf.xacro" />
-  <xacro:include filename="$(find bulldog_description)/urdf/bulldog/materials.urdf.xacro" />
+  <xacro:include filename="$(find bulldog_description)/urdf/accessories/wheel.urdf.xacro" />
+  <xacro:include filename="$(find bulldog_description)/urdf/accessories/materials.urdf.xacro" />
+  <xacro:include filename="$(find bulldog_description)/urdf/accessories/plates.urdf.xacro" />
   <xacro:include filename="$(find ur_description)/urdf/ur5.urdf.xacro" />
   <xacro:include filename="$(find lms1xx)/urdf/sick_lms1xx.urdf.xacro" />
   <xacro:include filename="$(find robotiq_s_model_visualization)/cfg/robotiq_hand_macro.urdf.xacro" />
   <xacro:include filename="$(find bulldog_description)/urdf/sensors/kinect_camera.urdf.xacro" />
-  <!--xacro:include filename="$(find bulldog_description)/urdf/accessories/yuntai.urdf.xacro" /-->
   <xacro:property name="wheel_length" value="0.142" />
   <xacro:property name="wheel_radius" value="0.183" />
@@ -24,5 +24,5 @@
       </visual>
       <collision>
-        <origin xyz="0 0 ${base_z_size/2.0}" rpy="0 0 0" />
+        <origin xyz="0 0 ${base_z_size / 2.0}" rpy="0 0 0" />
         <geometry>
           <box size="${base_x_size} ${base_y_size} ${base_z_size}"/>
@@ -47,21 +47,5 @@
     </joint>
     <!-- top plate -->
-    <link name="top_plate_link">
-      <visual>
-        <origin xyz="0 0 0" rpy="0 0 0" />
-        <geometry>
-          <mesh filename="package://bulldog_description/meshes/top_plate.stl" />
-        </geometry>
-        <material name="grey" />
-      </visual>
-    </link>
-    <gazebo reference="top_plate_link">
-      <material>Gazebo/Grey</material>
-    </gazebo>
-    <joint name="top_plate_joint" type="fixed">
-      <origin xyz="0.07937 0 0.253" rpy="0 0 0" />
-      <parent link="base_link" />
-      <child link="top_plate_link" />
-    </joint>
+    <xacro:top_plate />
     <!-- imu -->
     <link name="imu_link"/>
@@ -119,13 +103,5 @@
     <!-- kinect -->
     <xacro:if value="$(arg kinect_enabled)">
-      <xacro:kinect_camera prefix="camera" />
-      <gazebo reference="camera_link">
-        <material>Gazebo/Black</material>
-      </gazebo>
-      <joint name="kinect_frame_joint" type="fixed">
-        <origin xyz="0.13 0 0.135" rpy=" 0 0.15 0" />
-        <parent link="installation_plate_link"/>
-        <child link="camera_link"/>
-      </joint>
+      <xacro:kinect_camera />
     </xacro:if>
   </xacro:macro>

File: src/bulldog/bulldog_description/urdf/bulldog/bulldog_gazebo.urdf.xacro (robot description, xacro)
@@ -1,12 +1,11 @@
 <?xml version="1.0"?>
 <robot name="bulldog_robot" xmlns:xacro="http://ros.org/wiki/xacro">
-  <xacro:include filename="$(find bulldog_description)/urdf/bulldog/wheel.urdf.xacro" />
-  <xacro:include filename="$(find bulldog_description)/urdf/bulldog/materials.xacro" />
+  <xacro:include filename="$(find bulldog_description)/urdf/accessories/wheel.urdf.xacro" />
+  <xacro:include filename="$(find bulldog_description)/urdf/accessories/materials.urdf.xacro" />
+  <xacro:include filename="$(find bulldog_description)/urdf/accessories/plates.urdf.xacro" />
   <xacro:include filename="$(find ur_description)/urdf/ur5.urdf.xacro" />
   <xacro:include filename="$(find lms1xx)/urdf/sick_lms1xx.urdf.xacro" />
   <xacro:include filename="$(find robotiq_s_model_visualization)/cfg/s-model_articulated_macro.xacro" />
-  <!--xacro:include filename="$(find bulldog_description)/urdf/sensors/kinect_camera.urdf.xacro" /-->
-  <!--xacro:include filename="$(find bulldog_description)/urdf/accessories/yuntai.urdf.xacro" /-->
-  <property name="M_PI" value="3.141592654"/>
+  <xacro:include filename="$(find bulldog_description)/urdf/sensors/kinect_camera.urdf.xacro" />
   <xacro:property name="wheel_length" value="0.142" />
   <xacro:property name="wheel_radius" value="0.183" />
@@ -14,138 +13,102 @@
   <property name="base_y_size" value="0.42" />
   <property name="base_z_size" value="0.325" />
-  <xacro:macro name="bulldog_robot">
-  <link name="base_link">
-    <visual>
+  <xacro:macro name="bulldog_gazebo_robot">
+    <!-- base -->
+    <link name="base_link">
+      <visual>
+        <origin xyz="0 0 0" rpy="0 0 0" />
+        <geometry>
+          <mesh filename="package://bulldog_description/meshes/base_link.stl" />
+        </geometry>
+        <material name="flat_black" />
+      </visual>
+      <collision>
+        <origin xyz="0 0 ${base_z_size / 2.0}" rpy="0 0 0" />
+        <geometry>
+          <box size="${base_x_size} ${base_y_size} ${base_z_size}"/>
+        </geometry>
+      </collision>
+    </link>
+    <gazebo reference="base_link">
+      <material>Gazebo/FlatBlack</material>
+    </gazebo>
+    <!-- inertial -->
+    <link name="inertial_link">
+      <inertial>
+        <mass value="40" />
+        <origin xyz="0 0 0.1" />
+        <inertia ixx="0.7" ixy="-0.03" ixz="-0.15" iyy="2" iyz="-0.01" izz="4" />
+      </inertial>
+    </link>
+    <joint name="inertial_joint" type="fixed">
       <origin xyz="0 0 0" rpy="0 0 0" />
-      <geometry>
-        <mesh filename="package://bulldog_description/meshes/base_link.stl" />
-      </geometry>
-      <material name="flat_black" />
-    </visual>
-    <collision>
-      <origin xyz="0 0 ${base_z_size/2.0}" rpy="0 0 0" />
-      <geometry>
-        <box size="${base_x_size} ${base_y_size} ${base_z_size}"/>
-      </geometry>
-    </collision>
-  </link>
-  <gazebo reference="base_link">
-    <material>Gazebo/FlatBlack</material>
-  </gazebo>
-  <link name="inertial_link">
-    <inertial>
-      <mass value="40" />
-      <origin xyz="0 0 0.1" />
-      <inertia ixx="0.7" ixy="-0.03" ixz="-0.15" iyy="2" iyz="-0.01" izz="4" />
-    </inertial>
-  </link>
-  <joint name="inertial_joint" type="fixed">
-    <origin xyz="0 0 0" rpy="0 0 0" />
-    <parent link="base_link" />
-    <child link="inertial_link" />
-  </joint>
-  <link name="top_plate_link">
-    <visual>
+      <parent link="base_link" />
+      <child link="inertial_link" />
+    </joint>
+    <!-- top plate -->
+    <xacro:top_plate />
+    <!-- imu -->
+    <link name="imu_link"/>
+    <joint name="imu_joint" type="fixed">
       <origin xyz="0 0 0" rpy="0 0 0" />
-      <geometry>
-        <mesh filename="package://bulldog_description/meshes/top_plate.stl" />
-      </geometry>
-      <material name="grey" />
-    </visual>
-  </link>
-  <gazebo reference="top_plate_link">
-    <material>Gazebo/Grey</material>
-  </gazebo>
-  <joint name="top_plate_joint" type="fixed">
-    <origin xyz="0.07937 0 0.253" rpy="0 0 0" />
-    <parent link="base_link" />
-    <child link="top_plate_link" />
-  </joint>
-  <link name="imu_link"/>
-  <joint name="imu_joint" type="fixed">
-    <origin xyz="0 0 0" rpy="0 0 0" />
-    <parent link="base_link" />
-    <child link="imu_link" />
-  </joint>
-  <gazebo reference="imu_link" />
-  <xacro:bulldog_wheel wheel_prefix="front_left">
-    <origin xyz="0.27937 0.285 0.0435" rpy="0 0 0" />
-  </xacro:bulldog_wheel>
-  <xacro:bulldog_wheel wheel_prefix="front_right">
-    <origin xyz="0.27937 -0.285 0.0435" rpy="0 0 0" />
-  </xacro:bulldog_wheel>
-  <xacro:bulldog_wheel wheel_prefix="rear_left">
-    <origin xyz="-0.27937 0.285 0.0435" rpy="0 0 0" />
-  </xacro:bulldog_wheel>
-  <xacro:bulldog_wheel wheel_prefix="rear_right">
-    <origin xyz="-0.27937 -0.285 0.0435" rpy="0 0 0" />
-  </xacro:bulldog_wheel>
-  <!--xacro:if value="$(optenv BULLDOG_DUAL_UR5_ENABLED true)"-->
-    <!--xacro:installation_plate /-->
-    <xacro:ur5_robot prefix="left_arm_" joint_limited="true"/>
-    <joint name="left_arm_base" type="fixed">
-      <parent link="installation_plate_link" />
-      <child link="left_arm_base_link" />
-      <origin xyz="0 0.15945 0.09069" rpy="-0.785 0 0" />
+      <parent link="base_link" />
+      <child link="imu_link" />
     </joint>
-    <xacro:ur5_robot prefix="right_arm_" joint_limited="true"/>
-    <joint name="right_arm_base" type="fixed">
-      <parent link="installation_plate_link" />
-      <child link="right_arm_base_link" />
-      <origin xyz="0 -0.15945 0.09069" rpy="-0.785 0 ${M_PI}" />
-    </joint>
-  <xacro:s-model_articulated prefix="l_"/>
-  <joint name="left_arm_gripper" type="fixed">
-    <parent link="left_arm_ee_link" />
-    <child link="l_palm" />
-    <origin xyz="0 0 0" rpy="0 0 -1.57" />
-  </joint>
-  <xacro:s-model_articulated prefix="r_"/>
-  <joint name="right_arm_gripper" type="fixed">
-    <parent link="right_arm_ee_link" />
-    <child link="r_palm" />
-    <origin xyz="0 0 0" rpy="0 0 -1.57" />
-  </joint>
-  <xacro:if value="$(arg laser_enabled)">
+    <gazebo reference="imu_link" />
+    <xacro:bulldog_wheel wheel_prefix="front_left">
+      <origin xyz="0.27937 0.285 0.0435" rpy="0 0 0" />
+    </xacro:bulldog_wheel>
+    <xacro:bulldog_wheel wheel_prefix="front_right">
+      <origin xyz="0.27937 -0.285 0.0435" rpy="0 0 0" />
+    </xacro:bulldog_wheel>
+    <xacro:bulldog_wheel wheel_prefix="rear_left">
+      <origin xyz="-0.27937 0.285 0.0435" rpy="0 0 0" />
+    </xacro:bulldog_wheel>
+    <xacro:bulldog_wheel wheel_prefix="rear_right">
+      <origin xyz="-0.27937 -0.285 0.0435" rpy="0 0 0" />
+    </xacro:bulldog_wheel>
+    <!-- installation plate -->
     <xacro:installation_plate />
-    <xacro:laser_plate />
-    <sick_lms1xx frame="laser" topic="scan"/>
-    <joint name="laser_mount_joint" type="fixed">
-      <origin xyz="0.015 0 0.044" rpy="${M_PI} 0 0" />
-      <parent link="laser_plate_link" />
-      <child link="laser" />
-    </joint>
-  </xacro:if>
-    <link name="camera_link">
-    <visual>
-      <origin xyz="0 0 0" rpy="0 0 0" />
-      <geometry>
-        <box size="0.065 0.25 0.065"/>
-      </geometry>
-      <material name="white" />
-    </visual>
-    <collision>
-      <origin xyz="0 0 0" rpy="0 0 0" />
-      <geometry>
-        <!--box size="0.065 0.25 0.065"/-->
-        <box size = "0 0 0"/>
-      </geometry>
-    </collision>
-    </link>
-  <gazebo reference="camera_link">
-    <material>Gazebo/White</material>
-  </gazebo>
-    <joint name="kinect_frame_joint" type="fixed">
-        <origin xyz="0.13 0 0.135" rpy=" 0 0.15 0" />
-      <parent link="installation_plate_link"/>
-      <child link="camera_link"/>
-    </joint>
-    <xacro:kinect_camera prefix="camera"/>
-  <!--joint name="yuntai_installation_plate_joint" type="fixed">
-    <origin xyz="0.05 0 0.135 " rpy="0 ${M_PI/2} 0" />
-    <parent link="installation_plate_link"/>
-    <child link="yuntai_base_link" />
-  </joint>
-  <xacro:yuntai_robot /-->
+    <!-- dual ur5 arms -->
+    <xacro:if value="$(arg dual_ur5_enabled)">
+        <xacro:ur5_robot prefix="left_arm_" joint_limited="true"/>
+        <joint name="left_arm_base" type="fixed">
+        <parent link="installation_plate_link" />
+        <child link="left_arm_base_link" />
+        <origin xyz="0 0.15945 0.09069" rpy="-0.785 0 0" />
+        </joint>
+        <xacro:ur5_robot prefix="right_arm_" joint_limited="true"/>
+        <joint name="right_arm_base" type="fixed">
+        <parent link="installation_plate_link" />
+        <child link="right_arm_base_link" />
+        <origin xyz="0 -0.15945 0.09069" rpy="-0.785 0 ${pi}" />
+        </joint>
+        <xacro:s-model_articulated prefix="l_"/>
+        <joint name="left_arm_gripper" type="fixed">
+            <parent link="left_arm_ee_link" />
+            <child link="l_palm" />
+            <origin xyz="0 0 0" rpy="0 0 -1.57" />
+        </joint>
+        <xacro:s-model_articulated prefix="r_"/>
+        <joint name="right_arm_gripper" type="fixed">
+            <parent link="right_arm_ee_link" />
+            <child link="r_palm" />
+            <origin xyz="0 0 0" rpy="0 0 -1.57" />
+        </joint>
+    </xacro:if>
+    <!-- laser -->
+    <xacro:if value="$(arg laser_enabled)">
+      <xacro:laser_plate />
+      <sick_lms1xx frame="laser" topic="scan"/>
+      <joint name="laser_mount_joint" type="fixed">
+        <origin xyz="0.015 0 0.044" rpy="${pi} 0 0" />
+        <parent link="laser_plate_link" />
+        <child link="laser" />
+      </joint>
+    </xacro:if>
+    <!-- kinect -->
+    <xacro:if value="$(arg kinect_enabled)">
+      <xacro:kinect_camera />
+    </xacro:if>
   </xacro:macro>
 </robot>

File: src/bulldog/bulldog_description/urdf/bulldog_gazebo_robot.xacro (robot description, xacro)
@@ -1,11 +1,11 @@
 <?xml version="1.0"?>
+<!-- Create a bulldog robot instantiation in gazebo -->
 <robot name="bulldog_robot" xmlns:xacro="http://ros.org/wiki/xacro">
   <xacro:arg name="laser_enabled" default="true" />
   <xacro:arg name="ur5_enabled" default="false" />
   <xacro:arg name="kinect_enabled" default="false" />
-  <xacro:arg name="dual_ur5_enabled" default="false"/>
-  <xacro:arg name="robotiq_grippers_enabled" default="false"/>
+  <xacro:arg name="dual_ur5_enabled" default="true"/>
+  <xacro:arg name="robotiq_grippers_enabled" default="true"/>
   <xacro:include filename="$(find bulldog_description)/urdf/bulldog/bulldog_gazebo.urdf.xacro" />
-  <xacro:include filename="$(find bulldog_description)/urdf/accessories/plates.urdf.xacro" />
-  <xacro:bulldog_robot />
+  <xacro:bulldog_gazebo_robot />
 </robot>

File: src/bulldog/bulldog_description/urdf/bulldog_robot.xacro (robot description, xacro)
@@ -1,11 +1,11 @@
 <?xml version="1.0"?>
+<!-- Create a bulldog robot instantiation -->
 <robot name="bulldog_robot" xmlns:xacro="http://ros.org/wiki/xacro">
   <xacro:arg name="laser_enabled" default="true" />
   <xacro:arg name="ur5_enabled" default="false" />
-  <xacro:arg name="kinect_enabled" default="true" />
-  <xacro:arg name="dual_ur5_enabled" default="false"/>
-  <xacro:arg name="robotiq_grippers_enabled" default="false"/>
+  <xacro:arg name="kinect_enabled" default="false" />
+  <xacro:arg name="dual_ur5_enabled" default="true"/>
+  <xacro:arg name="robotiq_grippers_enabled" default="true"/>
   <xacro:include filename="$(find bulldog_description)/urdf/bulldog/bulldog.urdf.xacro" />
-  <xacro:include filename="$(find bulldog_description)/urdf/accessories/plates.urdf.xacro" />
   <xacro:bulldog_robot />
 </robot>

File: src/bulldog/bulldog_description/urdf/sensors/kinect_camera.urdf.xacro (robot description, xacro)
@@ -26,12 +26,12 @@
 -->
 <robot xmlns:xacro="http://ros.org/wiki/xacro" name="kinect_camera">
-  <xacro:macro name="kinect_camera" params="prefix:=camera">
+  <xacro:macro name="kinect_camera" params="camera_link_name:=kinect_link
+                                            plate_link_name:=installation_plate_link">
     <!-- Create kinect reference frame -->
     <!-- Add mesh for kinect -->
-    <link name="${prefix}_link">
+    <link name="${camera_link_name}">
       <origin xyz="0 0 0" rpy="0 0 0"/>
       <visual>
         <origin xyz="0 0 0" rpy="0 0 ${pi / 2}"/>
-        <!-- <origin xyz="0 0 0" rpy="0 0 0"/> -->
         <geometry>
           <mesh filename="package://bulldog_description/meshes/kinect.dae" />
@@ -44,19 +44,12 @@
       </collision>
     </link>
-    <!-- <link name="camera_link">
-    <visual>
-      <origin xyz="0 0 0" rpy="0 0 0" />
-      <geometry>
-        <box size="0.065 0.25 0.065"/>
-      </geometry>
-      <mesh filename="package://bulldog_description/meshes/kinect.dae" />
-    </visual>
-    <collision>
-      <origin xyz="0 0 0" rpy="0 0 0" />
-      <geometry>
-        <box size="0.065 0.25 0.065"/>
-      </geometry>
-    </collision>
-    </link> -->
+    <joint name="${camera_link_name}_joint" type="fixed">
+      <origin xyz="0.13 0 0.135" rpy=" 0 0.15 0" />
+      <parent link="${plate_link_name}" />
+      <child link="${camera_link_name}" />
+    </joint>
+    <gazebo reference="${camera_link_name}">
+      <material>Gazebo/Black</material>
+    </gazebo>
   </xacro:macro>
 </robot>

File: src/bulldog_simulator/bulldog_gazebo/urdf/description.gazebo.xacro (robot description, xacro)
@@ -28,5 +28,4 @@
   <xacro:arg name="robotiq_grippers_enabled" default="true"/>
   <xacro:include filename="$(find bulldog_description)/urdf/bulldog/bulldog.urdf.xacro" />
-  <!-- <xacro:include filename="$(find bulldog_description)/urdf/accessories/plates.urdf.xacro" /> -->
   <xacro:include filename="$(find bulldog_gazebo)/urdf/bulldog.gazebo.xacro" />
   <!-- Gazebo plugin for ROS Control -->
