Commit message: merge urdf from server

File: src/bulldog/bulldog_description/urdf/sensors/kinect_camera.urdf.xacro (robot description, xacro)
@@ -26,11 +26,12 @@
 -->
 <robot xmlns:xacro="http://ros.org/wiki/xacro" name="kinect_camera">
-  <xacro:macro name="kinect_camera" params="prefix:=camera">
+  <xacro:macro name="kinect_camera" params="camera_link_name:=kinect_link
+                                            plate_link_name:=installation_plate_link">
     <!-- Create kinect reference frame -->
     <!-- Add mesh for kinect -->
-    <!--link name="${prefix}_link">
+    <link name="${camera_link_name}">
       <origin xyz="0 0 0" rpy="0 0 0"/>
       <visual>
-        <origin xyz="0 0 0" rpy="0 0 ${M_PI/2}"/>
+        <origin xyz="0 0 0" rpy="0 0 ${pi / 2}"/>
         <geometry>
           <mesh filename="package://bulldog_description/meshes/kinect.dae" />
@@ -42,20 +43,13 @@
         </geometry>
       </collision>
-    </link-->
-    <link name="camera_link">
-    <visual>
-      <origin xyz="0 0 0" rpy="0 0 0" />
-      <geometry>
-        <box size="0.065 0.25 0.065"/>
-      </geometry>
-      <mesh filename="package://bulldog_description/meshes/kinect.dae" />
-    </visual>
-    <collision>
-      <origin xyz="0 0 0" rpy="0 0 0" />
-      <geometry>
-        <box size="0.065 0.25 0.065"/>
-      </geometry>
-    </collision>
     </link>
+    <joint name="${camera_link_name}_joint" type="fixed">
+      <origin xyz="0.13 0 0.135" rpy=" 0 0.15 0" />
+      <parent link="${plate_link_name}" />
+      <child link="${camera_link_name}" />
+    </joint>
+    <gazebo reference="${camera_link_name}">
+      <material>Gazebo/Black</material>
+    </gazebo>
   </xacro:macro>
 </robot>

File: src/bulldog_simulator/bulldog_gazebo/urdf/description.gazebo.xacro (robot description, xacro)
@@ -24,9 +24,8 @@
   <xacro:arg name="laser_enabled" default="true" />
   <xacro:arg name="ur5_enabled" default="false" />
-  <xacro:arg name="kinect_enabled" default="true" />
-  <xacro:arg name="dual_ur5_enabled" default="false"/>
-  <xacro:arg name="robotiq_grippers_enabled" default="false"/>
+  <xacro:arg name="kinect_enabled" default="false" />
+  <xacro:arg name="dual_ur5_enabled" default="true"/>
+  <xacro:arg name="robotiq_grippers_enabled" default="true"/>
   <xacro:include filename="$(find bulldog_description)/urdf/bulldog/bulldog.urdf.xacro" />
-  <xacro:include filename="$(find bulldog_description)/urdf/accessories/plates.urdf.xacro" />
   <xacro:include filename="$(find bulldog_gazebo)/urdf/bulldog.gazebo.xacro" />
   <!-- Gazebo plugin for ROS Control -->
@@ -36,5 +35,5 @@
     </plugin>
   </gazebo>
-<gazebo>
+  <gazebo>
     <plugin name="gazebo_grasp_fix" filename="libgazebo_grasp_fix.so">
         <arm>
@@ -49,5 +48,5 @@
            <gripper_link> l_finger_2_link_2 </gripper_link>
            <gripper_link> l_finger_2_link_3 </gripper_link>
-            <gripper_link> l_finger_middle_link_0 </gripper_link>
+           <gripper_link> l_finger_middle_link_0 </gripper_link>
            <gripper_link> l_finger_middle_link_1 </gripper_link>
            <gripper_link> l_finger_middle_link_2 </gripper_link>
@@ -65,5 +64,5 @@
            <gripper_link> r_finger_2_link_2 </gripper_link>
            <gripper_link> r_finger_2_link_3 </gripper_link>
-            <gripper_link> r_finger_middle_link_0 </gripper_link>
+           <gripper_link> r_finger_middle_link_0 </gripper_link>
            <gripper_link> r_finger_middle_link_1 </gripper_link>
            <gripper_link> r_finger_middle_link_2 </gripper_link>

File: src/robotiq_85_gripper/robotiq_85_description/urdf/robotiq_85_gripper.urdf.xacro (robot description, xacro)
@@ -1,4 +1,4 @@
 <?xml version="1.0"?>
-<robot name="robotiq_85_gripper" xmlns:xacro="http://ros.org/wiki/xacro">
+<robot name="robotiq_85_gripper" xmlns:xacro="http://wiki.ros.org/xacro">
     <xacro:include filename="$(find robotiq_85_description)/urdf/robotiq_85_gripper.transmission.xacro" />
     <property name="pi" value="3.14159"/>

File: src/robotiq_85_gripper/robotiq_85_description/urdf/robotiq_85_gripper.xacro (robot description, xacro)
@@ -1,4 +1,4 @@
 <?xml version="1.0" ?>
-<robot name="robotiq_85_gripper" xmlns:xacro="http://ros.org/wiki/xacro">
+<robot name="robotiq_85_gripper" xmlns:xacro="http://wiki.ros.org/xacro">
     <xacro:include filename="$(find robotiq_85_description)/urdf/robotiq_85_gripper.urdf.xacro" />
     <gazebo>

File: src/robotiq_85_gripper/robotiq_85_description/urdf/robotiq_85_gripper_sim_base.urdf.xacro (robot description, xacro)
@@ -1,4 +1,4 @@
 <?xml version="1.0"?>
-<robot name="robotiq_85_gripper_sim_base" xmlns:xacro="http://ros.org/wiki/xacro">
+<robot name="robotiq_85_gripper_sim_base" xmlns:xacro="http://wiki.ros.org/xacro">
     <xacro:macro name="robotiq_85_gripper_sim_base" params="prefix">
         <link name="${prefix}gripper_root_link">

Commit message: add d415 into urdf

File: src/bulldog/bulldog_description/urdf/accessories/plates.urdf.xacro (robot description, xacro)
@@ -1,4 +1,4 @@
 <?xml version="1.0"?>
-<robot name="bulldog_plates" xmlns:xacro="http://www.ros.org/wiki/xacro">
+<robot name="bulldog_plates" xmlns:xacro="http://ros.org/wiki/xacro">
   <xacro:macro name="top_plate">
     <link name="top_plate_link">

File: src/bulldog/bulldog_description/urdf/bulldog/bulldog_gazebo.urdf.xacro (robot description, xacro)
@@ -8,5 +8,5 @@
   <xacro:include filename="$(find robotiq_s_model_visualization)/cfg/s-model_articulated_macro.xacro" />
   <xacro:include filename="$(find bulldog_description)/urdf/sensors/kinect_camera.urdf.xacro" />
-  <xacro:include filename="$(find realsense2_camera)/urdf/_d415.urdf.xacro"/>
+  <xacro:include filename="$(find realsense2_camera)/urdf/_d415.urdf.xacro" />
   <xacro:property name="wheel_length" value="0.142" />
   <xacro:property name="wheel_radius" value="0.183" />
@@ -91,8 +91,7 @@
             <origin xyz="0 0 0" rpy="0 0 -1.57" />
         </joint>
-        <!-- realsense d415 -->
-        <!-- <sensor_d415 parent="base_link">
-          <origin xyz="0 0 0" rpy="0 0 0"/>
-        </sensor_d415> -->
+        <xacro:sensor_d415 prefix="left_gripper_sensor_d415_" parent="left_gripper_palm">
+          <origin xyz="0 0 -0.065" rpy="${pi} 0 ${pi / 2}"/>
+        </xacro:sensor_d415>
         <xacro:s-model_articulated prefix="right_gripper_"/>
         <joint name="right_arm_gripper" type="fixed">
@@ -101,9 +100,7 @@
             <origin xyz="0 0 0" rpy="0 0 -1.57" />
         </joint>
-        <!-- realsense d415 -->
-        <!-- <link name="base_link" />
-        <sensor_d415 parent="base_link">
-          <origin xyz="0 0 0" rpy="0 0 0"/>
-        </sensor_d415> -->
+        <xacro:sensor_d415 prefix="right_gripper_sensor_d415_" parent="right_gripper_palm">
+          <origin xyz="0 0 -0.065" rpy="${pi} 0 ${pi / 2}"/>
+        </xacro:sensor_d415>
     </xacro:if>
     <!-- laser -->

Commit message: remove NAN from point cloud and forward installation_plate

File: src/bulldog/bulldog_description/urdf/accessories/plates.urdf.xacro (robot description, xacro)
@@ -12,5 +12,5 @@
     </link>
     <joint name="top_plate_joint" type="fixed">
-      <origin xyz="0.07937 0 0.253" rpy="0 0 0" />
+      <origin xyz="0.13437 0 0.253" rpy="0 0 0" /><!-- <origin xyz="0.07937 0 0.253" rpy="0 0 0" /> -->
       <parent link="base_link" />
       <child link="top_plate_link" />
@@ -33,5 +33,5 @@
       <parent link="base_link"/>
       <child link="installation_plate_link"/>
-      <origin xyz="0.197 0 0.314" rpy="0 0 0" />
+      <origin xyz="0.252 0 0.314" rpy="0 0 0" /><!-- <origin xyz="0.197 0 0.314" rpy="0 0 0" /> -->
     </joint>
     <gazebo reference="installation_plate_link">
@@ -52,5 +52,5 @@
       <parent link="installation_plate_link"/>
       <child link="laser_plate_link"/>
-      <origin xyz="0.3 0 -0.1" rpy="${pi} 0 0" />
+      <origin xyz="0.245 0 -0.1" rpy="${pi} 0 0" /><!-- <origin xyz="0.3 0 -0.1" rpy="${pi} 0 0" /> -->
     </joint>
     <gazebo reference="laser_plate_link">

Commit message: hardware grasping demo workgit status!

File: src/bulldog/bulldog_description/urdf/accessories/plates.urdf.xacro (robot description, xacro)
@@ -33,5 +33,6 @@
       <parent link="base_link"/>
       <child link="installation_plate_link"/>
-      <origin xyz="0.252 0 0.314" rpy="0 0 0" /><!-- <origin xyz="0.197 0 0.314" rpy="0 0 0" /> -->
+      <origin xyz="0.202 0 0.314" rpy="0 0 0" /><!-- <origin xyz="0.197 0 0.314" rpy="0 0 0" /> -->
+      <!-- <origin xyz="0.147 0 0.314" rpy="0 0 0" /> -->
     </joint>
     <gazebo reference="installation_plate_link">
@@ -52,5 +53,5 @@
       <parent link="installation_plate_link"/>
       <child link="laser_plate_link"/>
-      <origin xyz="0.245 0 -0.1" rpy="${pi} 0 0" /><!-- <origin xyz="0.3 0 -0.1" rpy="${pi} 0 0" /> -->
+      <origin xyz="0.3 0 -0.1" rpy="${pi} 0 0" /><!-- <origin xyz="0.3 0 -0.1" rpy="${pi} 0 0" /> -->
     </joint>
     <gazebo reference="laser_plate_link">

File: src/bulldog/bulldog_description/urdf/bulldog/bulldog.urdf.xacro (robot description, xacro)
@@ -90,8 +90,8 @@
            780 and 782 accordingly of $(find robotiq_s_model_articulated_gazebo_plugins)/src/RobotiqHandPlugin.cpp. -->
       <xacro:robotiq_hand prefix="left_gripper_" parent="left_arm_ee_link" reflect="-1">
-        <origin rpy="0 -2.3562 -1.5708" xyz="0 0 0"/>
+        <origin rpy="0 -2.3562 -1.5708" xyz="0.065 0 0"/>
       </xacro:robotiq_hand>
       <xacro:robotiq_hand prefix="right_gripper_" parent="right_arm_ee_link" reflect="-1">
-        <origin rpy="0 2.3562 -1.5708" xyz="0 0 0"/>
+        <origin rpy="0 2.3562 -1.5708" xyz="0.065 0 0"/>
       </xacro:robotiq_hand>
     </xacro:if>

Commit message: update bulldog_description

File: src/bulldog/bulldog_description/urdf/accessories/plates.urdf.xacro (robot description, xacro)
@@ -33,5 +33,5 @@
       <parent link="base_link"/>
       <child link="installation_plate_link"/>
-      <origin xyz="0.197 0 0.314" rpy="0 0 0" />
+      <origin xyz="0.147 0 0.314" rpy="0 0 0" />
     </joint>
     <gazebo reference="installation_plate_link">

File: src/bulldog/bulldog_description/urdf/bulldog/bulldog.urdf.xacro (robot description, xacro)
@@ -89,9 +89,9 @@
       <!-- If you modify the name of the grippers, remember to change the *prefix* in line
            780 and 782 accordingly of $(find robotiq_s_model_articulated_gazebo_plugins)/src/RobotiqHandPlugin.cpp. -->
-      <xacro:robotiq_hand prefix="left_gripper_" parent="left_arm_ee_link" reflect="-1">
-        <origin rpy="0 -2.3562 -1.5708" xyz="0 0 0"/>
+      <xacro:robotiq_hand prefix="left_gripper_" parent="left_arm_tool0" reflect="-1">
+        <origin rpy="1.5708 0 -2.3562" xyz="0 0 0.065"/>
       </xacro:robotiq_hand>
-      <xacro:robotiq_hand prefix="right_gripper_" parent="right_arm_ee_link" reflect="-1">
-        <origin rpy="0 2.3562 -1.5708" xyz="0 0 0"/>
+      <xacro:robotiq_hand prefix="right_gripper_" parent="right_arm_tool0" reflect="-1">
+        <origin rpy="1.5708 0 2.3562" xyz="0 0 0.065"/>
       </xacro:robotiq_hand>
     </xacro:if>

Commit message: add realsense supports

File: src/bulldog/bulldog_description/urdf/accessories/plates.urdf.xacro (robot description, xacro)
@@ -1,4 +1,4 @@
 <?xml version="1.0"?>
-<robot name="bulldog_plates" xmlns:xacro="http://ros.org/wiki/xacro">
+<robot name="plates" xmlns:xacro="http://ros.org/wiki/xacro">
   <xacro:macro name="top_plate">
     <link name="top_plate_link">
@@ -12,5 +12,5 @@
     </link>
     <joint name="top_plate_joint" type="fixed">
-      <origin xyz="0.13437 0 0.253" rpy="0 0 0" /><!-- <origin xyz="0.07937 0 0.253" rpy="0 0 0" /> -->
+      <origin xyz="0.07937 0 0.253" rpy="0 0 0" />
       <parent link="base_link" />
       <child link="top_plate_link" />
@@ -33,6 +33,5 @@
       <parent link="base_link"/>
       <child link="installation_plate_link"/>
-      <origin xyz="0.202 0 0.314" rpy="0 0 0" /><!-- <origin xyz="0.197 0 0.314" rpy="0 0 0" /> -->
-      <!-- <origin xyz="0.147 0 0.314" rpy="0 0 0" /> -->
+      <origin xyz="0.147 0 0.314" rpy="0 0 0" />
     </joint>
     <gazebo reference="installation_plate_link">
@@ -53,5 +52,5 @@
       <parent link="installation_plate_link"/>
       <child link="laser_plate_link"/>
-      <origin xyz="0.3 0 -0.1" rpy="${pi} 0 0" /><!-- <origin xyz="0.3 0 -0.1" rpy="${pi} 0 0" /> -->
+      <origin xyz="0.3 0 -0.1" rpy="${pi} 0 0" />
     </joint>
     <gazebo reference="laser_plate_link">

File: src/bulldog/bulldog_description/urdf/bulldog/bulldog.urdf.xacro (robot description, xacro)
@@ -4,4 +4,5 @@
   <xacro:include filename="$(find bulldog_description)/urdf/accessories/materials.urdf.xacro" />
   <xacro:include filename="$(find bulldog_description)/urdf/accessories/plates.urdf.xacro" />
+  <xacro:include filename="$(find bulldog_description)/urdf/accessories/realsense_support.urdf.xacro" />
   <xacro:include filename="$(find ur_description)/urdf/ur5.urdf.xacro" />
   <xacro:include filename="$(find lms1xx)/urdf/sick_lms1xx.urdf.xacro" />
@@ -89,9 +90,9 @@
       <!-- If you modify the name of the grippers, remember to change the *prefix* in line
            780 and 782 accordingly of $(find robotiq_s_model_articulated_gazebo_plugins)/src/RobotiqHandPlugin.cpp. -->
-      <xacro:robotiq_hand prefix="left_gripper_" parent="left_arm_ee_link" reflect="-1">
-        <origin rpy="0 -2.3562 -1.5708" xyz="0.065 0 0"/>
+      <xacro:robotiq_hand prefix="left_gripper_" parent="left_arm_tool0" reflect="-1">
+        <origin rpy="${pi / 2} 0 ${-pi * 3 / 4}" xyz="0 0 0.065"/>
       </xacro:robotiq_hand>
-      <xacro:robotiq_hand prefix="right_gripper_" parent="right_arm_ee_link" reflect="-1">
-        <origin rpy="0 2.3562 -1.5708" xyz="0.065 0 0"/>
+      <xacro:robotiq_hand prefix="right_gripper_" parent="right_arm_tool0" reflect="-1">
+        <origin rpy="${pi / 2} 0 ${pi * 3 / 4}" xyz="0 0 0.065"/>
       </xacro:robotiq_hand>
     </xacro:if>
@@ -112,10 +113,20 @@
     <!-- realsense d415 -->
     <xacro:if value="$(arg realsense_enabled)">
-      <xacro:sensor_d415 prefix="left_gripper_sensor_d415_" parent="left_gripper_palm">
-        <origin xyz="0 0 0.065" rpy="0 0 ${pi / 2}"/>
+      <xacro:realsense_support prefix="left_gripper_sensor_support_"
+        installation_link="left_gripper_palm">
+        <origin xyz="0 -0.050 0" rpy="${pi / 2} 0 ${pi}" />
+      </xacro:realsense_support>
+      <xacro:sensor_d415 prefix="left_gripper_sensor_d415_"
+        parent="left_gripper_sensor_support_mounted_link">
+        <origin xyz="0 0 0" rpy="0 0 0"/>
       </xacro:sensor_d415>
-      <xacro:sensor_d415 prefix="right_gripper_sensor_d415_" parent="right_gripper_palm">
-          <origin xyz="0 0 -0.065" rpy="${pi} 0 ${pi / 2}"/>
-        </xacro:sensor_d415>
+      <xacro:realsense_support prefix="right_gripper_sensor_support_"
+        installation_link="right_gripper_palm">
+        <origin xyz="0 -0.050 0" rpy="${-pi / 2} 0 0" />
+      </xacro:realsense_support>
+      <xacro:sensor_d415 prefix="right_gripper_sensor_d415_"
+        parent="right_gripper_sensor_support_mounted_link">
+        <origin xyz="0 0 0" rpy="0 0 0"/>
+      </xacro:sensor_d415>
     </xacro:if>
   </xacro:macro>

File: src/bulldog_simulator/bulldog_gazebo/urdf/accessories/realsense_camera.gazebo.xacro (robot description, xacro)
@@ -4,5 +4,5 @@
     <!-- material -->
     <gazebo reference="${prefix}camera_link">
-      <material>Gazebo/Grey</material>
+      <material>Gazebo/White</material>
     </gazebo>
     <!-- color sensor -->
@@ -151,5 +151,5 @@
           <depthImageTopicName>/${prefix}camera/depth/image_rect_raw</depthImageTopicName>
           <depthImageCameraInfoTopicName>/${prefix}camera/depth/camera_info</depthImageCameraInfoTopicName>
-          <pointCloudTopicName>/${prefix}camera/depth_registered/points</pointCloudTopicName>
+          <pointCloudTopicName>/${prefix}camera/depth/color/points</pointCloudTopicName>
           <frameName>${prefix}camera_depth_optical_frame</frameName>
           <pointCloudCutoff>0.4</pointCloudCutoff>

File: src/bulldog_simulator/bulldog_gazebo/urdf/bulldog.gazebo.xacro (robot description, xacro)
@@ -23,5 +23,5 @@
 <robot name="bulldog_robot" xmlns:xacro="http://ros.org/wiki/xacro">
   <xacro:include filename="$(find bulldog_gazebo)/urdf/accessories/kinect_camera.gazebo.xacro"/>
-  <xacro:include filename="$(find bulldog_gazebo)/urdf/accessories/realsense_d415_camera.gazebo.xacro"/>
+  <xacro:include filename="$(find bulldog_gazebo)/urdf/accessories/realsense_camera.gazebo.xacro"/>
   <xacro:macro name="bulldog_gazebo_config">
     <!-- ROS control -->
@@ -95,6 +95,6 @@
             <kp_position>5.0</kp_position>
             <kd_position>0.5</kd_position>
-            <topic_command>left_hand/command</topic_command>
-            <topic_state>left_hand/state</topic_state>
+            <topic_command>left_gripper/command</topic_command>
+            <topic_state>left_gripper/state</topic_state>
           </plugin>
         </gazebo>
@@ -104,6 +104,6 @@
               <kp_position>5.0</kp_position>
               <kd_position>0.5</kd_position>
-              <topic_command>right_hand/command</topic_command>
-              <topic_state>right_hand/state</topic_state>
+              <topic_command>right_gripper/command</topic_command>
+              <topic_state>right_gripper/state</topic_state>
             </plugin>
         </gazebo>

Commit message: debugging laser scan position

File: src/bulldog/bulldog_description/urdf/accessories/plates.urdf.xacro (robot description, xacro)
@@ -52,5 +52,6 @@
       <parent link="installation_plate_link"/>
       <child link="laser_plate_link"/>
-      <origin xyz="0.3 0 -0.1" rpy="${pi} 0 0" />
+      <origin xyz="0.35 0 -0.0476" rpy="${pi} 0 0" />
+      <!-- <origin xyz="0.3 0 -0.1" rpy="${pi} 0 0" /> -->
     </joint>
     <gazebo reference="laser_plate_link">

File: src/bulldog_simulator/bulldog_gazebo/urdf/bulldog.gazebo.xacro (robot description, xacro)
@@ -40,6 +40,10 @@
         <bodyName>base_link</bodyName>
         <topicName>imu/data</topicName>
-        <serviceName>imu_service</serviceName>
-        <gaussianNoise>0.0</gaussianNoise>
+        <accelDrift>0.005 0.005 0.005</accelDrift>
+        <accelGaussianNoise>0.005 0.005 0.005</accelGaussianNoise>
+        <rateDrift>0.005 0.005 0.005 </rateDrift>
+        <rateGaussianNoise>0.005 0.005 0.005 </rateGaussianNoise>
+        <headingDrift>0.005</headingDrift>
+        <headingGaussianNoise>0.005</headingGaussianNoise>
       </plugin>
     </gazebo>

Commit message: debugging laser plate position

File: src/bulldog/bulldog_description/urdf/accessories/plates.urdf.xacro (robot description, xacro)
@@ -53,5 +53,4 @@
       <child link="laser_plate_link"/>
       <origin xyz="0.35 0 -0.0476" rpy="${pi} 0 0" />
-      <!-- <origin xyz="0.3 0 -0.1" rpy="${pi} 0 0" /> -->
     </joint>
     <gazebo reference="laser_plate_link">
