Commit message: begin to merger server branch

File: src/bulldog/bulldog_description/urdf/accessories/wheel.urdf.xacro (robot description, xacro)
@@ -42,5 +42,5 @@
       </actuator>
       <joint name="${wheel_prefix}_wheel_joint">
-        <hardwareInterface>hardware_interface/VelocityJointInterface</hardwareInterface>
+        <hardwareInterface>VelocityJointInterface</hardwareInterface>
       </joint>
     </transmission>

File: src/bulldog/bulldog_description/urdf/bulldog/bulldog.urdf.xacro (robot description, xacro)
@@ -6,6 +6,7 @@
   <xacro:include filename="$(find ur_description)/urdf/ur5.urdf.xacro" />
   <xacro:include filename="$(find lms1xx)/urdf/sick_lms1xx.urdf.xacro" />
-  <xacro:include filename="$(find robotiq_s_model_visualization)/cfg/robotiq_hand_macro.urdf.xacro" />
+  <xacro:include filename="$(find robotiq_3f_gripper_visualization)/cfg/robotiq_hand_macro.urdf.xacro" />
   <xacro:include filename="$(find bulldog_description)/urdf/sensors/kinect_camera.urdf.xacro" />
+  <xacro:include filename="$(find realsense2_camera)/urdf/_d415.urdf.xacro" />
   <xacro:property name="wheel_length" value="0.142" />
   <xacro:property name="wheel_radius" value="0.183" />
@@ -84,8 +85,10 @@
         <origin xyz="0 -0.15945 0.09069" rpy="-0.785 0 ${pi}" />
       </joint>
-      <xacro:robotiq_hand prefix="l_" parent="left_arm_ee_link" reflect="-1">
+      <!-- If you modify the name of the grippers, remember to change the *prefix* in line
+           780 and 782 accordingly of $(find robotiq_s_model_articulated_gazebo_plugins)/src/RobotiqHandPlugin.cpp. -->
+      <xacro:robotiq_hand prefix="left_gripper_" parent="left_arm_ee_link" reflect="-1">
         <origin rpy="0 0 -1.57" xyz="0 0 0"/>
       </xacro:robotiq_hand>
-      <xacro:robotiq_hand prefix="r_" parent="right_arm_ee_link" reflect="-1">
+      <xacro:robotiq_hand prefix="right_gripper_" parent="right_arm_ee_link" reflect="-1">
         <origin rpy="0 0 -1.57" xyz="0 0 0"/>
       </xacro:robotiq_hand>
@@ -103,5 +106,14 @@
     <!-- kinect -->
     <xacro:if value="$(arg kinect_enabled)">
-      <xacro:kinect_camera />
+      <xacro:kinect_camera prefix="kinect" parent="installation_plate_link" />
+    </xacro:if>
+    <!-- realsense d415 -->
+    <xacro:if value="$(arg realsense_enabled)">
+      <xacro:sensor_d415 prefix="left_gripper_sensor_d415_" parent="left_gripper_palm">
+        <origin xyz="0 0 -0.065" rpy="${pi} 0 ${pi / 2}"/>
+      </xacro:sensor_d415>
+      <xacro:sensor_d415 prefix="right_gripper_sensor_d415_" parent="right_gripper_palm">
+          <origin xyz="0 0 -0.065" rpy="${pi} 0 ${pi / 2}"/>
+        </xacro:sensor_d415>
     </xacro:if>
   </xacro:macro>

File: src/bulldog/bulldog_description/urdf/bulldog/bulldog_gazebo.urdf.xacro (robot description, xacro)
@@ -6,11 +6,12 @@
   <xacro:include filename="$(find ur_description)/urdf/ur5.urdf.xacro" />
   <xacro:include filename="$(find lms1xx)/urdf/sick_lms1xx.urdf.xacro" />
-  <xacro:include filename="$(find robotiq_s_model_visualization)/cfg/s-model_articulated_macro.xacro" />
+  <xacro:include filename="$(find robotiq_3f_gripper_visualization)/cfg/robotiq-3f-gripper_articulated_macro.xacro" />
   <xacro:include filename="$(find bulldog_description)/urdf/sensors/kinect_camera.urdf.xacro" />
+  <xacro:include filename="$(find realsense2_camera)/urdf/_d415.urdf.xacro" />
   <xacro:property name="wheel_length" value="0.142" />
   <xacro:property name="wheel_radius" value="0.183" />
-  <property name="base_x_size" value="0.85" />
-  <property name="base_y_size" value="0.42" />
-  <property name="base_z_size" value="0.325" />
+  <xacro:property name="base_x_size" value="0.85" />
+  <xacro:property name="base_y_size" value="0.42" />
+  <xacro:property name="base_z_size" value="0.325" />
   <xacro:macro name="bulldog_gazebo_robot">
     <!-- base -->
@@ -84,14 +85,14 @@
         <origin xyz="0 -0.15945 0.09069" rpy="-0.785 0 ${pi}" />
         </joint>
-        <xacro:s-model_articulated prefix="l_"/>
+        <xacro:robotiq-3f-gripper_articulated prefix="left_gripper_"/>
         <joint name="left_arm_gripper" type="fixed">
             <parent link="left_arm_ee_link" />
-            <child link="l_palm" />
+            <child link="left_gripper_palm" />
             <origin xyz="0 0 0" rpy="0 0 -1.57" />
         </joint>
-        <xacro:s-model_articulated prefix="r_"/>
+        <xacro:robotiq-3f-gripper_articulated prefix="right_gripper_"/>
         <joint name="right_arm_gripper" type="fixed">
             <parent link="right_arm_ee_link" />
-            <child link="r_palm" />
+            <child link="right_gripper_palm" />
             <origin xyz="0 0 0" rpy="0 0 -1.57" />
         </joint>
@@ -109,5 +110,14 @@
     <!-- kinect -->
     <xacro:if value="$(arg kinect_enabled)">
-      <xacro:kinect_camera />
+      <xacro:kinect_camera prefix="kinect" parent="installation_plate_link" />
+    </xacro:if>
+    <!-- realsense d415 -->
+    <xacro:if value="$(arg realsense_enabled)">
+      <xacro:sensor_d415 prefix="left_gripper_sensor_d415_" parent="left_gripper_palm">
+        <origin xyz="0 0 -0.065" rpy="${pi} 0 ${pi / 2}"/>
+      </xacro:sensor_d415>
+      <xacro:sensor_d415 prefix="right_gripper_sensor_d415_" parent="right_gripper_palm">
+          <origin xyz="0 0 -0.065" rpy="${pi} 0 ${pi / 2}"/>
+      </xacro:sensor_d415>
     </xacro:if>
   </xacro:macro>

File: src/bulldog/bulldog_description/urdf/bulldog_gazebo_robot.xacro (robot description, xacro)
@@ -5,4 +5,5 @@
   <xacro:arg name="ur5_enabled" default="false" />
   <xacro:arg name="kinect_enabled" default="false" />
+  <xacro:arg name="realsense_enabled" default="true" />
   <xacro:arg name="dual_ur5_enabled" default="true"/>
   <xacro:arg name="robotiq_grippers_enabled" default="true"/>

File: src/bulldog/bulldog_description/urdf/bulldog_robot.xacro (robot description, xacro)
@@ -5,4 +5,5 @@
   <xacro:arg name="ur5_enabled" default="false" />
   <xacro:arg name="kinect_enabled" default="false" />
+  <xacro:arg name="realsense_enabled" default="true" />
   <xacro:arg name="dual_ur5_enabled" default="true"/>
   <xacro:arg name="robotiq_grippers_enabled" default="true"/>

File: src/bulldog/bulldog_description/urdf/sensors/kinect_camera.urdf.xacro (robot description, xacro)
@@ -26,9 +26,8 @@
 -->
 <robot xmlns:xacro="http://ros.org/wiki/xacro" name="kinect_camera">
-  <xacro:macro name="kinect_camera" params="camera_link_name:=kinect_link
-                                            plate_link_name:=installation_plate_link">
+  <xacro:macro name="kinect_camera" params="prefix parent">
     <!-- Create kinect reference frame -->
     <!-- Add mesh for kinect -->
-    <link name="${camera_link_name}">
+    <link name="${prefix}_link">
       <origin xyz="0 0 0" rpy="0 0 0"/>
       <visual>
@@ -44,12 +43,9 @@
       </collision>
     </link>
-    <joint name="${camera_link_name}_joint" type="fixed">
+    <joint name="${prefix}_joint" type="fixed">
       <origin xyz="0.13 0 0.135" rpy=" 0 0.15 0" />
-      <parent link="${plate_link_name}" />
-      <child link="${camera_link_name}" />
+      <parent link="${parent}" />
+      <child link="${prefix}_link" />
     </joint>
-    <gazebo reference="${camera_link_name}">
-      <material>Gazebo/Black</material>
-    </gazebo>
   </xacro:macro>
 </robot>

File: src/bulldog_simulator/bulldog_gazebo/urdf/accessories/kinect_camera.gazebo.xacro (robot description, xacro)
@@ -2,4 +2,9 @@
 <root xmlns:xacro="http://ros.org/wiki/xacro">
   <xacro:macro name="kinect_camera_gazebo" params="prefix">
+    <!-- material -->
+    <gazebo reference="${prefix}_link">
+      <material>Gazebo/Grey</material>
+    </gazebo>
+    <!-- optical joint and link -->
     <joint name="${prefix}_optical_joint" type="fixed">
       <origin xyz="0 0 0" rpy="-1.5708 0 -1.5708"/>
@@ -8,8 +13,9 @@
     </joint>
     <link name="${prefix}_frame_optical"/>
+    <!-- depth camera -->
     <gazebo reference="${prefix}_link">
       <sensor type="depth" name="${prefix}">
         <always_on>true</always_on>
-        <update_rate>20.0</update_rate>
+        <update_rate>30.0</update_rate>
         <camera>
           <horizontal_fov>${60.0 * pi / 180.0}</horizontal_fov>
@@ -24,6 +30,6 @@
           </clip>
         </camera>
-        <plugin name="kinect_${prefix}_controller" filename="libgazebo_ros_openni_kinect.so">
-          <cameraName>${prefix}</cameraName>
+        <plugin name="${prefix}_controller" filename="libgazebo_ros_openni_kinect.so">
+          <cameraName>${prefix}_camera</cameraName>
           <alwaysOn>true</alwaysOn>
           <updateRate>10</updateRate>

File: src/bulldog_simulator/bulldog_gazebo/urdf/bulldog.gazebo.xacro (robot description, xacro)
@@ -21,7 +21,14 @@
 ARISING IN ANY WAY OUT OF THE USE OF THIS SOFTWARE, EVEN IF ADVISED OF THE POSSIBILITY OF SUCH DAMAGE.
 -->
-<robot name="bulldog_robot_gazebo" xmlns:xacro="http://ros.org/wiki/xacro">
+<robot name="bulldog_gazebo_robot" xmlns:xacro="http://ros.org/wiki/xacro">
   <xacro:include filename="$(find bulldog_gazebo)/urdf/accessories/kinect_camera.gazebo.xacro"/>
-  <xacro:macro name="bulldog_robot_gazebo">
+  <xacro:include filename="$(find bulldog_gazebo)/urdf/accessories/realsense_d415_camera.gazebo.xacro"/>
+  <xacro:macro name="bulldog_gazebo_config">
+    <!-- ROS control -->
+    <gazebo>
+      <plugin name="gazebo_ros_control" filename="libgazebo_ros_control.so">
+        <robotNamespace>/</robotNamespace>
+      </plugin>
+    </gazebo>
     <!-- imu -->
     <gazebo>
@@ -53,25 +60,72 @@
     <!-- ur5 arm -->
     <!--Remove when https://github.com/ros-industrial/universal_robot/pull/168 is resolved -->
-    <gazebo reference="ur5_arm_shoulder_link">
-      <selfCollide>true</selfCollide>
-    </gazebo>
-    <gazebo reference="ur5_arm_upper_arm_link">
-      <selfCollide>true</selfCollide>
-    </gazebo>
-    <gazebo reference="ur5_arm_forearm_link">
-      <selfCollide>true</selfCollide>
-    </gazebo>
-    <gazebo reference="ur5_arm_wrist_1_link">
-      <selfCollide>true</selfCollide>
-    </gazebo>
-    <gazebo reference="ur5_arm_wrist_3_link">
-      <selfCollide>true</selfCollide>
-    </gazebo>
-    <gazebo reference="ur5_arm_wrist_2_link">
-      <selfCollide>true</selfCollide>
-    </gazebo>
-    <gazebo reference="ur5_arm_ee_link">
-      <selfCollide>true</selfCollide>
-    </gazebo>
+    <xacro:if value="$(arg ur5_enabled)">
+      <gazebo reference="ur5_arm_shoulder_link">
+        <selfCollide>true</selfCollide>
+      </gazebo>
+      <gazebo reference="ur5_arm_upper_arm_link">
+        <selfCollide>true</selfCollide>
+      </gazebo>
+      <gazebo reference="ur5_arm_forearm_link">
+        <selfCollide>true</selfCollide>
+      </gazebo>
+      <gazebo reference="ur5_arm_wrist_1_link">
+        <selfCollide>true</selfCollide>
+      </gazebo>
+      <gazebo reference="ur5_arm_wrist_3_link">
+        <selfCollide>true</selfCollide>
+      </gazebo>
+      <gazebo reference="ur5_arm_wrist_2_link">
+        <selfCollide>true</selfCollide>
+      </gazebo>
+      <gazebo reference="ur5_arm_ee_link">
+        <selfCollide>true</selfCollide>
+      </gazebo>
+    </xacro:if>
+    <xacro:if value="$(arg dual_ur5_enabled)">
+      <gazebo>
+        <plugin name="gazebo_grasp_fix" filename="libgazebo_grasp_fix.so">
+            <arm>
+              <arm_name>left_arm </arm_name>
+              <palm_link> left_arm_wrist_3_link </palm_link>
+              <gripper_link> left_gripper_finger_1_link_0 </gripper_link>
+              <gripper_link> left_gripper_finger_1_link_1 </gripper_link>
+              <gripper_link> left_gripper_finger_1_link_2 </gripper_link>
+              <gripper_link> left_gripper_finger_1_link_3 </gripper_link>
+              <gripper_link> left_gripper_finger_2_link_0 </gripper_link>
+              <gripper_link> left_gripper_finger_2_link_1 </gripper_link>
+              <gripper_link> left_gripper_finger_2_link_2 </gripper_link>
+              <gripper_link> left_gripper_finger_2_link_3 </gripper_link>
+              <gripper_link> left_gripper_finger_middle_link_0 </gripper_link>
+              <gripper_link> left_gripper_finger_middle_link_1 </gripper_link>
+              <gripper_link> left_gripper_finger_middle_link_2 </gripper_link>
+              <gripper_link> left_gripper_finger_middle_link_3 </gripper_link>
+            </arm>
+            <arm>
+              <arm_name>right_arm </arm_name>
+              <palm_link> right_arm_wrist_3_link  </palm_link>
+              <gripper_link> right_gripper_finger_1_link_0 </gripper_link>
+              <gripper_link> right_gripper_finger_1_link_1 </gripper_link>
+              <gripper_link> right_gripper_finger_1_link_2 </gripper_link>
+              <gripper_link> right_gripper_finger_1_link_3 </gripper_link>
+              <gripper_link> right_gripper_finger_2_link_0 </gripper_link>
+              <gripper_link> right_gripper_finger_2_link_1 </gripper_link>
+              <gripper_link> right_gripper_finger_2_link_2 </gripper_link>
+              <gripper_link> right_gripper_finger_2_link_3 </gripper_link>
+              <gripper_link> right_gripper_finger_middle_link_0 </gripper_link>
+              <gripper_link> right_gripper_finger_middle_link_1 </gripper_link>
+              <gripper_link> right_gripper_finger_middle_link_2 </gripper_link>
+              <gripper_link> right_gripper_finger_middle_link_3 </gripper_link>
+            </arm>
+          <forces_angle_tolerance>100</forces_angle_tolerance>
+          <update_rate>4</update_rate>
+          <grip_count_threshold>4</grip_count_threshold>
+          <max_grip_count>8</max_grip_count>
+          <release_tolerance>0.005</release_tolerance>
+          <disable_collisions_on_attach>false</disable_collisions_on_attach>
+          <contact_topic>__default_topic__</contact_topic>
+        </plugin>
+      </gazebo>
+    </xacro:if>
     <!-- robotiq grippers -->
     <xacro:if value="$(arg robotiq_grippers_enabled)">
@@ -88,82 +142,82 @@
               <kp_position>5.0</kp_position>
               <kd_position>0.5</kd_position>
-             </plugin>
-        </gazebo>
-        <gazebo reference="l_palm">
-            <material>Gazebo/Black</material>
-        </gazebo>
-        <gazebo reference="r_palm">
-            <material>Gazebo/Black</material>
-        </gazebo>
-        <gazebo reference="l_finger_1_link_0">
-            <material>Gazebo/Black</material>
-        </gazebo>
-        <gazebo reference="r_finger_1_link_0">
-            <material>Gazebo/Black</material>
-        </gazebo>
-        <gazebo reference="l_finger_1_link_1">
-            <material>Gazebo/Black</material>
-        </gazebo>
-        <gazebo reference="r_finger_1_link_1">
-            <material>Gazebo/Black</material>
-        </gazebo>
-        <gazebo reference="l_finger_1_link_2">
-            <material>Gazebo/Black</material>
-        </gazebo>
-        <gazebo reference="r_finger_1_link_2">
-            <material>Gazebo/Black</material>
-        </gazebo>
-        <gazebo reference="l_finger_1_link_3">
-            <material>Gazebo/Grey</material>
-        </gazebo>
-        <gazebo reference="r_finger_1_link_3">
-            <material>Gazebo/Grey</material>
-        </gazebo>
-        <gazebo reference="l_finger_2_link_0">
-            <material>Gazebo/Black</material>
-        </gazebo>
-        <gazebo reference="r_finger_2_link_0">
-            <material>Gazebo/Black</material>
-        </gazebo>
-        <gazebo reference="l_finger_2_link_1">
-            <material>Gazebo/Black</material>
-        </gazebo>
-        <gazebo reference="r_finger_2_link_1">
-            <material>Gazebo/Black</material>
-        </gazebo>
-        <gazebo reference="l_finger_2_link_2">
-            <material>Gazebo/Black</material>
-        </gazebo>
-        <gazebo reference="r_finger_2_link_2">
-            <material>Gazebo/Black</material>
-        </gazebo>
-        <gazebo reference="l_finger_2_link_3">
-            <material>Gazebo/Grey</material>
-        </gazebo>
-        <gazebo reference="r_finger_2_link_3">
-            <material>Gazebo/Grey</material>
-        </gazebo>
-        <gazebo reference="l_finger_middle_link_0">
-            <material>Gazebo/Black</material>
-        </gazebo>
-        <gazebo reference="r_finger_middle_link_0">
-            <material>Gazebo/Black</material>
-        </gazebo>
-        <gazebo reference="l_finger_middle_link_1">
-            <material>Gazebo/Black</material>
-        </gazebo>
-        <gazebo reference="r_finger_middle_link_1">
-            <material>Gazebo/Black</material>
-        </gazebo>
-        <gazebo reference="l_finger_middle_link_2">
-            <material>Gazebo/Black</material>
-        </gazebo>
-        <gazebo reference="r_finger_middle_link_2">
-            <material>Gazebo/Black</material>
-        </gazebo>
-        <gazebo reference="l_finger_middle_link_3">
-            <material>Gazebo/Grey</material>
-        </gazebo>
-        <gazebo reference="r_finger_middle_link_3">
+            </plugin>
+        </gazebo>
+        <gazebo reference="left_gripper">
+            <material>Gazebo/Black</material>
+        </gazebo>
+        <gazebo reference="right_gripper">
+            <material>Gazebo/Black</material>
+        </gazebo>
+        <gazebo reference="left_gripper_finger_1_link_0">
+            <material>Gazebo/Black</material>
+        </gazebo>
+        <gazebo reference="right_gripper_finger_1_link_0">
+            <material>Gazebo/Black</material>
+        </gazebo>
+        <gazebo reference="left_gripper_finger_1_link_1">
+            <material>Gazebo/Black</material>
+        </gazebo>
+        <gazebo reference="right_gripper_finger_1_link_1">
+            <material>Gazebo/Black</material>
+        </gazebo>
+        <gazebo reference="left_gripper_finger_1_link_2">
+            <material>Gazebo/Black</material>
+        </gazebo>
+        <gazebo reference="right_gripper_finger_1_link_2">
+            <material>Gazebo/Black</material>
+        </gazebo>
+        <gazebo reference="left_gripper_finger_1_link_3">
+            <material>Gazebo/Grey</material>
+        </gazebo>
+        <gazebo reference="right_gripper_finger_1_link_3">
+            <material>Gazebo/Grey</material>
+        </gazebo>
+        <gazebo reference="left_gripper_finger_2_link_0">
+            <material>Gazebo/Black</material>
+        </gazebo>
+        <gazebo reference="right_gripper_finger_2_link_0">
+            <material>Gazebo/Black</material>
+        </gazebo>
+        <gazebo reference="left_gripper_finger_2_link_1">
+            <material>Gazebo/Black</material>
+        </gazebo>
+        <gazebo reference="right_gripper_finger_2_link_1">
+            <material>Gazebo/Black</material>
+        </gazebo>
+        <gazebo reference="left_gripper_finger_2_link_2">
+            <material>Gazebo/Black</material>
+        </gazebo>
+        <gazebo reference="right_gripper_finger_2_link_2">
+            <material>Gazebo/Black</material>
+        </gazebo>
+        <gazebo reference="left_gripper_finger_2_link_3">
+            <material>Gazebo/Grey</material>
+        </gazebo>
+        <gazebo reference="right_gripper_finger_2_link_3">
+            <material>Gazebo/Grey</material>
+        </gazebo>
+        <gazebo reference="left_gripper_finger_middle_link_0">
+            <material>Gazebo/Black</material>
+        </gazebo>
+        <gazebo reference="right_gripper_finger_middle_link_0">
+            <material>Gazebo/Black</material>
+        </gazebo>
+        <gazebo reference="left_gripper_finger_middle_link_1">
+            <material>Gazebo/Black</material>
+        </gazebo>
+        <gazebo reference="right_gripper_finger_middle_link_1">
+            <material>Gazebo/Black</material>
+        </gazebo>
+        <gazebo reference="left_gripper_finger_middle_link_2">
+            <material>Gazebo/Black</material>
+        </gazebo>
+        <gazebo reference="right_gripper_finger_middle_link_2">
+            <material>Gazebo/Black</material>
+        </gazebo>
+        <gazebo reference="left_gripper_finger_middle_link_3">
+            <material>Gazebo/Grey</material>
+        </gazebo>
+        <gazebo reference="right_gripper_finger_middle_link_3">
             <material>Gazebo/Grey</material>
         </gazebo>
@@ -171,5 +225,10 @@
     <!-- kinect -->
     <xacro:if value="$(arg kinect_enabled)">
-      <xacro:kinect_camera_gazebo prefix="camera"/>
+      <xacro:kinect_camera_gazebo prefix="kinect"/>
+    </xacro:if>
+    <!-- realsense -->
+    <xacro:if value="$(arg realsense_enabled)">
+      <xacro:sensor_d415_gazebo prefix="left_gripper_sensor_d415_"/>
+      <xacro:sensor_d415_gazebo prefix="right_gripper_sensor_d415_"/>
     </xacro:if>
   </xacro:macro>
