Commit message: begin to merger server branch

File: src/bulldog_simulator/bulldog_gazebo/urdf/description.gazebo.xacro (robot description, xacro)
@@ -25,58 +25,10 @@
   <xacro:arg name="ur5_enabled" default="false" />
   <xacro:arg name="kinect_enabled" default="false" />
-  <xacro:arg name="dual_ur5_enabled" default="true"/>
-  <xacro:arg name="robotiq_grippers_enabled" default="true"/>
+  <xacro:arg name="realsense_enabled" default="true" />
+  <xacro:arg name="dual_ur5_enabled" default="true" />
+  <xacro:arg name="robotiq_grippers_enabled" default="true" />
   <xacro:include filename="$(find bulldog_description)/urdf/bulldog/bulldog.urdf.xacro" />
   <xacro:include filename="$(find bulldog_gazebo)/urdf/bulldog.gazebo.xacro" />
-  <!-- Gazebo plugin for ROS Control -->
-  <gazebo>
-    <plugin name="gazebo_ros_control" filename="libgazebo_ros_control.so">
-      <robotNamespace>/</robotNamespace>
-    </plugin>
-  </gazebo>
-  <gazebo>
-    <plugin name="gazebo_grasp_fix" filename="libgazebo_grasp_fix.so">
-        <arm>
-           <arm_name>left_arm </arm_name>
-           <palm_link> left_arm_wrist_3_link </palm_link>
-           <gripper_link> l_finger_1_link_0 </gripper_link>
-           <gripper_link> l_finger_1_link_1 </gripper_link>
-           <gripper_link> l_finger_1_link_2 </gripper_link>
-           <gripper_link> l_finger_1_link_3 </gripper_link>
-           <gripper_link> l_finger_2_link_0 </gripper_link>
-           <gripper_link> l_finger_2_link_1 </gripper_link>
-           <gripper_link> l_finger_2_link_2 </gripper_link>
-           <gripper_link> l_finger_2_link_3 </gripper_link>
-           <gripper_link> l_finger_middle_link_0 </gripper_link>
-           <gripper_link> l_finger_middle_link_1 </gripper_link>
-           <gripper_link> l_finger_middle_link_2 </gripper_link>
-           <gripper_link> l_finger_middle_link_3 </gripper_link>
-        </arm>
-        <arm>
-           <arm_name>right_arm </arm_name>
-           <palm_link> right_arm_wrist_3_link  </palm_link>
-           <gripper_link> r_finger_1_link_0 </gripper_link>
-           <gripper_link> r_finger_1_link_1 </gripper_link>
-           <gripper_link> r_finger_1_link_2 </gripper_link>
-           <gripper_link> r_finger_1_link_3 </gripper_link>
-           <gripper_link> r_finger_2_link_0 </gripper_link>
-           <gripper_link> r_finger_2_link_1 </gripper_link>
-           <gripper_link> r_finger_2_link_2 </gripper_link>
-           <gripper_link> r_finger_2_link_3 </gripper_link>
-           <gripper_link> r_finger_middle_link_0 </gripper_link>
-           <gripper_link> r_finger_middle_link_1 </gripper_link>
-           <gripper_link> r_finger_middle_link_2 </gripper_link>
-           <gripper_link> r_finger_middle_link_3 </gripper_link>
-        </arm>
-       <forces_angle_tolerance>100</forces_angle_tolerance>
-       <update_rate>4</update_rate>
-       <grip_count_threshold>4</grip_count_threshold>
-       <max_grip_count>8</max_grip_count>
-       <release_tolerance>0.005</release_tolerance>
-       <disable_collisions_on_attach>false</disable_collisions_on_attach>
-       <contact_topic>__default_topic__</contact_topic>
-    </plugin>
-  </gazebo>
+  <xacro:bulldog_gazebo_config />
   <xacro:bulldog_robot />
-  <xacro:bulldog_robot_gazebo />
 </robot>

Commit message: fix wheel jump bug

File: src/bulldog/bulldog_description/urdf/accessories/wheel.urdf.xacro (robot description, xacro)
@@ -1,10 +1,10 @@
 <?xml version="1.0"?>
 <robot name="wheel" xmlns:xacro="http://ros.org/wiki/xacro">
-  <xacro:macro name="bulldog_wheel" params="wheel_prefix *joint_pose">
+  <xacro:macro name="bulldog_wheel" params="wheel_prefix *joint_pose wheel_length:=0.142 wheel_radius:=0.183">
     <link name="${wheel_prefix}_wheel_link">
       <inertial>
-        <mass value="3" />
+        <mass value="3.0" />
         <origin xyz="0 0 0" />
-        <inertia  ixx="0.025" ixy="0" ixz="0" iyy="0.025" iyz="0" izz="0.045" />
+        <inertia  ixx="0.025" ixy="0" ixz="0" iyy="0.045" iyz="0" izz="0.025" />
       </inertial>
       <visual>
@@ -24,8 +24,8 @@
     <gazebo reference="${wheel_prefix}_wheel_link">
       <mu1 value="1.0"/>
-      <mu2 value="1.0"/>
-      <kp value="10000000.0" />
-      <kd value="1.0" />
-      <fdir1 value="1 0 0"/>
+			<mu2 value="0.05"/>
+			<kp value="10000000.0" />
+			<kd value="1.0" />
+			<fdir1 value="1 0 0"/>
       <material>Gazebo/DarkGrey</material>
     </gazebo>
@@ -40,5 +40,4 @@
       <actuator name="${wheel_prefix}_wheel_motor">
         <mechanicalReduction>1</mechanicalReduction>
-        <hardwareInterface>VelocityJointInterface</hardwareInterface>
       </actuator>
       <joint name="${wheel_prefix}_wheel_joint">

File: src/bulldog/bulldog_description/urdf/bulldog/bulldog.urdf.xacro (robot description, xacro)
@@ -10,6 +10,4 @@
   <xacro:include filename="$(find bulldog_description)/urdf/sensors/kinect_camera.urdf.xacro" />
   <xacro:include filename="$(find realsense2_description)/urdf/_d415.urdf.xacro" />
-  <xacro:property name="wheel_length" value="0.142" />
-  <xacro:property name="wheel_radius" value="0.183" />
   <xacro:property name="base_x_size" value="0.85" />
   <xacro:property name="base_y_size" value="0.42" />

File: src/bulldog/bulldog_description/urdf/bulldog/bulldog_gazebo.urdf.xacro (robot description, xacro)
@@ -9,6 +9,4 @@
   <xacro:include filename="$(find bulldog_description)/urdf/sensors/kinect_camera.urdf.xacro" />
   <xacro:include filename="$(find realsense2_description)/urdf/_d415.urdf.xacro" />
-  <xacro:property name="wheel_length" value="0.142" />
-  <xacro:property name="wheel_radius" value="0.183" />
   <xacro:property name="base_x_size" value="0.85" />
   <xacro:property name="base_y_size" value="0.42" />

Commit message: debugging bulldog_navigation

File: src/bulldog/bulldog_description/urdf/accessories/wheel.urdf.xacro (robot description, xacro)
@@ -1,5 +1,5 @@
 <?xml version="1.0"?>
 <robot name="wheel" xmlns:xacro="http://ros.org/wiki/xacro">
-  <xacro:macro name="bulldog_wheel" params="wheel_prefix *joint_pose wheel_length:=0.142 wheel_radius:=0.183">
+  <xacro:macro name="bulldog_wheel" params="wheel_prefix wheel_length wheel_radius *joint_pose">
     <link name="${wheel_prefix}_wheel_link">
       <inertial>

File: src/bulldog/bulldog_description/urdf/bulldog/bulldog.urdf.xacro (robot description, xacro)
@@ -10,9 +10,17 @@
   <xacro:include filename="$(find bulldog_description)/urdf/sensors/kinect_camera.urdf.xacro" />
   <xacro:include filename="$(find realsense2_description)/urdf/_d415.urdf.xacro" />
-  <xacro:property name="base_x_size" value="0.85" />
-  <xacro:property name="base_y_size" value="0.42" />
-  <xacro:property name="base_z_size" value="0.325" />
+  <!-- Base Size -->
+  <xacro:property name="base_x_size" value="0.85000000" />
+  <xacro:property name="base_y_size" value="0.42000000" />
+  <xacro:property name="base_z_size" value="0.32500000" />
+  <!-- Wheel Mounting Positions -->
+  <xacro:property name="wheelbase" value="0.5587" /> <!-- husky = 0.5120 -->
+  <xacro:property name="track" value="0.5708" /> <!-- husky = 0.5708 -->
+  <xacro:property name="wheel_vertical_offset" value="0.04352" /> <!-- husky = 0.3282 -->
+  <!-- Wheel Properties -->
+  <xacro:property name="wheel_length" value="0.1420" /> <!-- husky = 0.1143 -->
+  <xacro:property name="wheel_radius" value="0.1830" /> <!-- husky = 0.1651 -->
   <xacro:macro name="bulldog_robot">
-    <!-- base -->
+    <!-- Base -->
     <link name="base_link">
       <visual>
@@ -24,14 +32,27 @@
       </visual>
       <collision>
-        <origin xyz="0 0 ${base_z_size / 2.0}" rpy="0 0 0" />
+        <origin xyz="0 0 ${base_z_size / 4.0}" rpy="0 0 0" />
         <geometry>
-          <box size="${base_x_size} ${base_y_size} ${base_z_size}"/>
+          <box size="${base_x_size} ${base_y_size} ${base_z_size / 2}"/>
+        </geometry>
+      </collision>
+      <collision>
+        <origin xyz="0 0 ${base_z_size * 3 / 4 - 0.01}" rpy="0 0 0" />
+        <geometry>
+          <box size="${base_x_size * 4 / 5} ${base_y_size} ${base_z_siz / 2 - 0.02}"/>
         </geometry>
       </collision>
     </link>
-    <gazebo reference="base_link">
+    <!-- <gazebo reference="base_link">
       <material>Gazebo/FlatBlack</material>
-    </gazebo>
-    <!-- inertial -->
+    </gazebo> -->
+    <!-- Base footprint is on the ground under the robot -->
+    <link name="base_footprint"/>
+    <joint name="base_footprint_joint" type="fixed">
+      <origin xyz="0 0 ${wheel_vertical_offset - wheel_radius}" rpy="0 0 0" />
+      <parent link="base_link" />
+      <child link="base_footprint" />
+    </joint>
+    <!-- Inertial -->
     <link name="inertial_link">
       <inertial>
@@ -46,7 +67,7 @@
       <child link="inertial_link" />
     </joint>
-    <!-- top plate -->
+    <!-- Top Plate -->
     <xacro:top_plate />
-    <!-- imu -->
+    <!-- IMU -->
     <link name="imu_link"/>
     <joint name="imu_joint" type="fixed">
@@ -57,5 +78,5 @@
     <gazebo reference="imu_link" />
     <xacro:bulldog_wheel wheel_prefix="front_left">
-      <origin xyz="0.27937 0.285 0.0435" rpy="0 0 0" />
+      <origin xyz="${wheelbase / 2} ${track / 2} ${wheel_vertical_offset}" rpy="0 0 0" />
     </xacro:bulldog_wheel>
     <xacro:bulldog_wheel wheel_prefix="front_right">
@@ -68,7 +89,7 @@
       <origin xyz="-0.27937 -0.285 0.0435" rpy="0 0 0" />
     </xacro:bulldog_wheel>
-    <!-- installation plate -->
+    <!-- Installation Plate -->
     <xacro:installation_plate />
-    <!-- dual ur5 arms -->
+    <!-- Dual UR5 Arms -->
     <xacro:if value="$(arg dual_ur5_enabled)">
       <xacro:ur5_robot prefix="left_arm_" joint_limited="true"
@@ -95,8 +116,9 @@
       </xacro:robotiq_hand>
     </xacro:if>
-    <!-- laser -->
+    <!-- Sick LMS1xx LiDAR -->
     <xacro:if value="$(arg laser_enabled)">
       <xacro:laser_plate />
-      <sick_lms1xx frame="laser" topic="scan" visualize="true"/>
+      <sick_lms1xx frame="laser" topic="scan" visualize="true"
+        min_angle="-2.35619" max_angle="2.35619"/>
       <joint name="laser_mount_joint" type="fixed">
         <origin xyz="0.015 0 0.044" rpy="${pi} 0 0" />
@@ -105,9 +127,9 @@
       </joint>
     </xacro:if>
-    <!-- kinect -->
+    <!-- Kinect -->
     <xacro:if value="$(arg kinect_enabled)">
       <xacro:kinect_camera prefix="kinect" parent="installation_plate_link" />
     </xacro:if>
-    <!-- realsense d415 -->
+    <!-- RealSense D415 -->
     <xacro:if value="$(arg realsense_enabled)">
       <xacro:realsense_support prefix="left_gripper_sensor_support_"
