Commit message: Add tool0 link in robotiq hand URDF

File: src/robotiq/robotiq_3f_gripper_visualization/cfg/robotiq_hand_macro.urdf.xacro (robot description, xacro)
@@ -674,4 +674,12 @@
         <mu2>1.1</mu2>
       </gazebo>
+      <!-- Link tool0 -->
+      <link name="${prefix}tool0"/>
+      <!-- Link inertial -->
+      <inertial>
+        <origin xyz="0 0 0" rpy="0 0 0"/>
+        <mass value="1.3"/>
+        <inertia ixx="0.006012" ixy="0.000079" ixz="-0.00024" iyy="0.012892" iyz="0" izz="0.002435" />
+      </inertial>
     <!-- End of link list -->
     <!-- Joint list -->
@@ -714,4 +722,13 @@
       <implicitSpringDamper>1</implicitSpringDamper>
     </gazebo>
+    <!-- Joint palm_tool0 -->
+    <joint name="${prefix}palm_tool0" type="fixed">
+			<parent link="${prefix}palm"/>
+			<child link="${prefix}tool0"/>
+			<origin xyz="0.0 0.0875 0.0" rpy="0 0 1.5707"/>
+		</joint>
+    <gazebo reference="${prefix}palm_tool0">
+      <implicitSpringDamper>1</implicitSpringDamper>
+    </gazebo>
     <!-- end of joint list -->
   </xacro:macro>

Commit message: revert to original robotiq gripper model

File: src/robotiq/robotiq_3f_gripper_visualization/cfg/robotiq_hand_macro.urdf.xacro (robot description, xacro)
@@ -259,10 +259,10 @@
         </geometry>
       </visual>
-      <!-- <collision>
+      <collision>
         <origin rpy="0 0 0" xyz="0 0 0"/>
          <geometry>
           <box size=".02 .02 .002"/>
         </geometry>
-      </collision> -->
+      </collision>
       <inertial>
         <origin rpy="0 0 0" xyz="0.0092 0.00514 0"/>
@@ -317,10 +317,10 @@
         </geometry>
       </visual>
-      <!-- <collision>
+      <collision>
         <origin rpy="0 0 0" xyz="0 0 0"/>
          <geometry>
           <box size=".02 .02 .002"/>
         </geometry>
-      </collision> -->
+      </collision>
       <inertial>
         <origin rpy="0 0 0" xyz="-0.01025 0.00046 0"/>
@@ -375,10 +375,10 @@
         </geometry>
       </visual>
-      <!--  <collision>
+      <collision>
         <origin rpy="0 0 0" xyz="0 0 0"/>
          <geometry>
           <box size=".02 0.02 .002"/>
         </geometry>
-      </collision> -->
+      </collision>
       <inertial>
         <origin rpy="0 0 0" xyz="0.00548 0 0"/>

Commit message: rotate gripper tool0 frame

File: src/robotiq/robotiq_3f_gripper_visualization/cfg/robotiq_hand_macro.urdf.xacro (robot description, xacro)
@@ -726,5 +726,5 @@
 			<parent link="${prefix}palm"/>
 			<child link="${prefix}tool0"/>
-			<origin xyz="0.0 0.0875 0.0" rpy="0 0 1.5707"/>
+			<origin xyz="0.0 0.0875 0.0" rpy="-1.5707 0 0"/>
 		</joint>
     <gazebo reference="${prefix}palm_tool0">
