Commit message: debugging bulldog navigation

File: src/bulldog_description/urdf/accessories/wheel.urdf.xacro (robot description, xacro)
@@ -24,5 +24,5 @@
     <gazebo reference="${wheel_prefix}_wheel_link">
       <mu1 value="1.0"/>
-			<mu2 value="0.1"/>
+			<mu2 value="0.5"/>
 			<kp value="10000000.0" />
 			<kd value="1.0" />

File: src/bulldog_description/urdf/bulldog/bulldog.urdf.xacro (robot description, xacro)
@@ -59,11 +59,14 @@
         </geometry>
       </collision>
-      <collision>
+      <!-- <collision>
         <origin xyz="0 0 ${base_z_size * 3 / 4 - 0.01}" rpy="0 0 0" />
         <geometry>
           <box size="${base_x_size * 4 / 5} ${base_y_size} ${base_z_size / 2 - 0.02}"/>
         </geometry>
-      </collision>
+      </collision> -->
     </link>
+    <gazebo reference="base_link">
+      <material>Gazebo/FlatBlack</material>
+    </gazebo>
     <!-- Base footprint is on the ground under the robot -->
     <link name="base_footprint"/>
@@ -82,5 +85,5 @@
     </link> -->
     <!-- Dual UR5 Husky -->
-    <!-- <link name="inertial_link">
+    <link name="inertial_link">
       <inertial>
         <mass value="48.39054"/>
@@ -88,7 +91,7 @@
         <inertia ixx="2.1634275613800003" ixy="-0.055452352110000006" ixz="-0.41083822026" iyy="3.5314689495400002" iyz="-0.004366145530000001" izz="4.4759585875" />
       </inertial>
-    </link>  -->
+    </link>
     <!-- Husky -->
-    <link name="inertial_link">
+    <!-- <link name="inertial_link">
       <inertial>
         <mass value="46.034" />
@@ -96,5 +99,5 @@
         <inertia ixx="0.6022" ixy="-0.02364" ixz="-0.1197" iyy="1.7386" iyz="-0.001544" izz="2.0296" />
       </inertial>
-    </link>
+    </link> -->
     <joint name="inertial_joint" type="fixed">
       <origin xyz="0 0 0" rpy="0 0 0" />

Commit message: debugging bulldog_description

File: src/bulldog_description/urdf/accessories/wheel.urdf.xacro (robot description, xacro)
@@ -3,6 +3,11 @@
   <xacro:macro name="bulldog_wheel" params="wheel_prefix wheel_length wheel_radius *joint_pose">
     <link name="${wheel_prefix}_wheel_link">
+      <!-- <inertial>
+        <mass value="2.637" />
+				<origin xyz="0 0 0" />
+				<inertia  ixx="0.02467" ixy="0" ixz="0" iyy="0.04411" iyz="0" izz="0.02467" />
+      </inertial> -->
       <inertial>
-        <mass value="3.0" />
+        <mass value="3" />
         <origin xyz="0 0 0" />
         <inertia  ixx="0.025" ixy="0" ixz="0" iyy="0.045" iyz="0" izz="0.025" />
@@ -24,5 +29,5 @@
     <gazebo reference="${wheel_prefix}_wheel_link">
       <mu1 value="1.0"/>
-			<mu2 value="0.5"/>
+			<mu2 value="0.25"/>
 			<kp value="10000000.0" />
 			<kd value="1.0" />
@@ -37,12 +42,12 @@
     </joint>
     <transmission name="${wheel_prefix}_wheel_trans" type="SimpleTransmission">
-      <type>transmission_interface/SimpleTransmission</type>
-      <actuator name="${wheel_prefix}_wheel_motor">
-        <mechanicalReduction>1</mechanicalReduction>
-      </actuator>
-      <joint name="${wheel_prefix}_wheel_joint">
-        <hardwareInterface>hardware_interface/VelocityJointInterface</hardwareInterface>
-      </joint>
-    </transmission>
+			<type>transmission_interface/SimpleTransmission</type>
+			<actuator name="${wheel_prefix}_wheel_motor">
+				<mechanicalReduction>1</mechanicalReduction>
+			</actuator>
+			<joint name="${wheel_prefix}_wheel_joint">
+				<hardwareInterface>hardware_interface/VelocityJointInterface</hardwareInterface>
+			</joint>
+		</transmission>
   </xacro:macro>
 </robot>

File: src/bulldog_description/urdf/bulldog/bulldog.urdf.xacro (robot description, xacro)
@@ -77,5 +77,5 @@
     </joint>
     <!-- Interial link stores the robot's inertial information -->
-    <!-- <link name="inertial_link">
+    <link name="inertial_link">
       <inertial>
         <mass value="40" />
@@ -83,7 +83,7 @@
         <inertia ixx="0.7" ixy="-0.03" ixz="-0.15" iyy="2" iyz="-0.01" izz="4" />
       </inertial>
-    </link> -->
+    </link>
     <!-- Dual UR5 Husky -->
-    <link name="inertial_link">
+    <!-- <link name="inertial_link">
       <inertial>
         <mass value="48.39054"/>
@@ -91,5 +91,5 @@
         <inertia ixx="2.1634275613800003" ixy="-0.055452352110000006" ixz="-0.41083822026" iyy="3.5314689495400002" iyz="-0.004366145530000001" izz="4.4759585875" />
       </inertial>
-    </link>
+    </link> -->
     <!-- Husky -->
     <!-- <link name="inertial_link">

Commit message: acml begin to work!

File: src/bulldog_description/urdf/accessories/wheel.urdf.xacro (robot description, xacro)
@@ -29,5 +29,5 @@
     <gazebo reference="${wheel_prefix}_wheel_link">
       <mu1 value="1.0"/>
-			<mu2 value="0.25"/>
+			<mu2 value="0.5"/>
 			<kp value="10000000.0" />
 			<kd value="1.0" />

File: src/bulldog_description/urdf/bulldog/bulldog.urdf.xacro (robot description, xacro)
@@ -35,5 +35,5 @@
   <xacro:property name="right_robotiq_3f_gripper_rpy" value="${pi / 2} 0 ${pi * 3 / 4}" />
   <!-- LMS1xx LiDAR Angle Range and Mounting Positions -->
-  <xacro:property name="lms1xx_angle" value="${pi * 3 / 4}" />
+  <xacro:property name="lms1xx_angle" value="${pi * 2 / 4}" />
   <xacro:property name="lms1xx_xyz" value="0.015 0 0.044" />
   <xacro:property name="lms1xx_rpy" value="${pi} 0 0" />

Commit message: debugging wheel frictions

File: src/bulldog_description/urdf/accessories/wheel.urdf.xacro (robot description, xacro)
@@ -3,14 +3,14 @@
   <xacro:macro name="bulldog_wheel" params="wheel_prefix wheel_length wheel_radius *joint_pose">
     <link name="${wheel_prefix}_wheel_link">
-      <!-- <inertial>
+      <inertial>
         <mass value="2.637" />
 				<origin xyz="0 0 0" />
 				<inertia  ixx="0.02467" ixy="0" ixz="0" iyy="0.04411" iyz="0" izz="0.02467" />
-      </inertial> -->
-      <inertial>
+      </inertial>
+      <!-- <inertial>
         <mass value="3" />
         <origin xyz="0 0 0" />
         <inertia  ixx="0.025" ixy="0" ixz="0" iyy="0.045" iyz="0" izz="0.025" />
-      </inertial>
+      </inertial> -->
       <visual>
         <origin xyz="0 0 0" rpy="0 0 0" />
@@ -29,5 +29,5 @@
     <gazebo reference="${wheel_prefix}_wheel_link">
       <mu1 value="1.0"/>
-			<mu2 value="0.5"/>
+			<mu2 value="0.2"/>
 			<kp value="10000000.0" />
 			<kd value="1.0" />

File: src/bulldog_description/urdf/bulldog/bulldog.urdf.xacro (robot description, xacro)
@@ -16,5 +16,5 @@
   <!-- Wheel Mounting Positions -->
   <xacro:property name="wheelbase" value="0.5587" /> <!-- husky = 0.5120 -->
-  <xacro:property name="track" value="0.5708" /> <!-- husky = 0.5708 -->
+  <xacro:property name="track" value="0.5848" /> <!-- husky = 0.5708 -->
   <xacro:property name="wheel_vertical_offset" value="0.04352" /> <!-- husky = 0.3282 -->
   <!-- Wheel Properties -->
@@ -77,5 +77,5 @@
     </joint>
     <!-- Interial link stores the robot's inertial information -->
-    <link name="inertial_link">
+    <!-- <link name="inertial_link">
       <inertial>
         <mass value="40" />
@@ -83,5 +83,5 @@
         <inertia ixx="0.7" ixy="-0.03" ixz="-0.15" iyy="2" iyz="-0.01" izz="4" />
       </inertial>
-    </link>
+    </link> -->
     <!-- Dual UR5 Husky -->
     <!-- <link name="inertial_link">
@@ -93,5 +93,5 @@
     </link> -->
     <!-- Husky -->
-    <!-- <link name="inertial_link">
+    <link name="inertial_link">
       <inertial>
         <mass value="46.034" />
@@ -99,5 +99,5 @@
         <inertia ixx="0.6022" ixy="-0.02364" ixz="-0.1197" iyy="1.7386" iyz="-0.001544" izz="2.0296" />
       </inertial>
-    </link> -->
+    </link>
     <joint name="inertial_joint" type="fixed">
       <origin xyz="0 0 0" rpy="0 0 0" />
@@ -114,5 +114,5 @@
     </joint>
     <gazebo reference="imu_link" />
-    <!-- Wheel macros -->
+    <!-- Wheels -->
     <xacro:bulldog_wheel wheel_prefix="front_left" wheel_length="${wheel_length}" wheel_radius="${wheel_radius}">
       <origin xyz="${wheelbase / 2} ${track / 2} ${wheel_vertical_offset}" rpy="0 0 0" />

Commit message: tuning bulldog navigation

File: src/bulldog_description/urdf/accessories/wheel.urdf.xacro (robot description, xacro)
@@ -29,5 +29,5 @@
     <gazebo reference="${wheel_prefix}_wheel_link">
       <mu1 value="1.0"/>
-			<mu2 value="0.2"/>
+			<mu2 value="0.15"/>
 			<kp value="10000000.0" />
 			<kd value="1.0" />

File: src/bulldog_description/urdf/bulldog/bulldog.urdf.xacro (robot description, xacro)
@@ -35,5 +35,5 @@
   <xacro:property name="right_robotiq_3f_gripper_rpy" value="${pi / 2} 0 ${pi * 3 / 4}" />
   <!-- LMS1xx LiDAR Angle Range and Mounting Positions -->
-  <xacro:property name="lms1xx_angle" value="${pi * 2 / 4}" />
+  <xacro:property name="lms1xx_angle" value="${pi * 3 / 4}" />
   <xacro:property name="lms1xx_xyz" value="0.015 0 0.044" />
   <xacro:property name="lms1xx_rpy" value="${pi} 0 0" />
@@ -96,6 +96,5 @@
       <inertial>
         <mass value="46.034" />
-        <!-- <origin xyz="-0.00065 -0.085 0.062" /> -->
-        <origin xyz="-0.00065 0.0 0.062" />
+        <origin xyz="-0.00065 -0.085 0.062" />
         <inertia ixx="0.6022" ixy="-0.02364" ixz="-0.1197" iyy="1.7386" iyz="-0.001544" izz="2.0296" />
       </inertial>
